File: KLST_SHEEP/KLST_SHEEP.sch (KiCad schematic (older format))
At the start: 93 parts, among them J1 Micro_SD_Card_Card_Detect_SPI, J2 GPIO+AUDIO+ANALOG, J3 USB_A, J4 GPIO_EXT_A, J5 USB_B_Micro, J6 GPIO_EXT_B, J7 GPIO_EXT_C, J8 GMT028-05_V1.1, J9 ARM_JTAG_SWD(STDC14), Q1 AO3401A, SW1 BUTTON_BOOT_FLASH, SW2 BUTTON_RESET, U1 STM32H743VITx, U2 AMS1117-3.3, X1 KLST_SHEEP--graphics, X2 KLST_SHEEP--icon, X3 KLST_SHEEP--wolf, Y1 16MHz

Commit message: finished PIN assignment, cleaned up silkscreen
READY TO ROUTE :)
Parts:
- removed J2: GPIO+AUDIO+ANALOG, Connector_PinHeader_2.54mm:PinHeader_2x08_P2.54mm_Vertical, symbol Connector_Generic:Conn_02x08_Odd_Even
- removed J4: GPIO_EXT_A, Connector_PinHeader_2.54mm:PinHeader_2x04_P2.54mm_Vertical_SMD, symbol Connector_Generic:Conn_02x04_Odd_Even
- removed J6: GPIO_EXT_B, Connector_PinHeader_2.54mm:PinHeader_2x04_P2.54mm_Vertical_SMD, symbol Connector_Generic:Conn_02x04_Odd_Even
- removed J7: GPIO_EXT_C, Connector_PinHeader_2.54mm:PinHeader_2x04_P2.54mm_Vertical_SMD, symbol Connector_Generic:Conn_02x04_Odd_Even
- added J2: PERIPHERALS, Connector_PinHeader_2.54mm:PinHeader_2x24_P2.54mm_Vertical_SMD, symbol Connector_Generic:Conn_02x24_Odd_Even
- added R53, R54: 2.2K, Resistor_SMD:R_0402_1005Metric, symbol Device:R
Connections:
- net GPIO_EXT_A_00 is gone; now on net GPIO_02: U1.84 (PD3)
- net GPIO_EXT_A_01 is gone; now on net GPIO_03: U1.83 (PD2)
- net GPIO_EXT_B_00 is gone; now on net GPIO_04: U1.58 (PD11)
- net GPIO_EXT_B_01 is gone; now on net GPIO_05: U1.57 (PD10)
- net GPIO_EXT_B_02 is gone; now on net GPIO_06: U1.56 (PD9)
- net GPIO_EXT_B_03 is gone; now on net GPIO_07: U1.55 (PD8)
- net GPIO_EXT_C_00 is gone; now on net LED_11: U1.35 (PB1)
- net GPIO_EXT_C_01 is gone; now on net LED_12: U1.34 (PB0)
- net GPIO_EXT_C_07 is gone; now on net GPIO_00: U1.88 (PD7)
- net +3V3: now also J2.39 (Pin_39), J2.4 (Pin_4), J2.40 (Pin_40), J2.47 (Pin_47), J2.48 (Pin_48), R53.1, R54.1
- net +5V: now also J2.2 (Pin_2)
- net ADC_00: now also J2.21 (Pin_21)
- net ADC_01: now also J2.23 (Pin_23)
- net DAC_00: now also J2.22 (Pin_22)
- net DAC_01: now also J2.24 (Pin_24)
- net GND: now also J2.1 (Pin_1), J2.29 (Pin_29), J2.3 (Pin_3), J2.30 (Pin_30), J2.41 (Pin_41), J2.42 (Pin_42)
- net GPIO_00: now also J2.19 (Pin_19); no longer U1.66 (PC9)
- net GPIO_01: now also U1.85 (PD4), J2.20 (Pin_20); no longer U1.65 (PC8)
- net GPIO_02: now also J2.17 (Pin_17); no longer U1.64 (PC7)
- net GPIO_03: now also J2.18 (Pin_18); no longer U1.63 (PC6)
- net GPIO_04: now also J2.15 (Pin_15); no longer U1.62 (PD15)
- net GPIO_05: now also J2.16 (Pin_16); no longer U1.61 (PD14)
- net GPIO_06: now also J2.13 (Pin_13); no longer U1.60 (PD13)
- net GPIO_07: now also J2.14 (Pin_14); no longer U1.59 (PD12)
- net LED_00: now also U1.95 (PB8); no longer U1.30 (PA6)
- net LED_01: now also U1.91 (PB5); no longer U1.31 (PA7)
- net LED_02: now also U1.90 (PB4); no longer U1.24 (PA2)
- net LED_03: now also U1.66 (PC9)
- net LED_04: now also U1.65 (PC8)
- net LED_05: now also U1.64 (PC7)
- net LED_06: now also U1.63 (PC6)
- net LED_07: now also U1.62 (PD15)
- net LED_08: now also U1.61 (PD14)
- net LED_09: now also U1.60 (PD13)
- net LED_10: now also U1.59 (PD12)
- net LED_13: now also U1.31 (PA7)
- net LED_14: now also U1.30 (PA6)
- net LED_15: now also U1.24 (PA2)
- net LINE_IN_LEFT: now also J2.28 (Pin_28)
- net LINE_IN_RIGHT: now also J2.26 (Pin_26)
- net LINE_OUT_LEFT: now also J2.27 (Pin_27)
- net LINE_OUT_RIGHT: now also J2.25 (Pin_25)
- net SERIAL_DEBUG_RX: now also J2.45 (Pin_45)
- net SERIAL_DEBUG_TX: now also J2.43 (Pin_43)
- net SPI_DISPLAY_CS: now also J2.38 (Pin_38)
- net SPI_DISPLAY_MISO: now also J2.34 (Pin_34)
- net SPI_DISPLAY_MOSI: now also J2.32 (Pin_32)
- net SPI_DISPLAY_SCK: now also J2.36 (Pin_36)
- net GPIO_EXT_B_04 renamed GPIO_08
- net GPIO_08: now also J2.11 (Pin_11)
- net GPIO_EXT_B_05 renamed GPIO_09
- net GPIO_09: now also J2.12 (Pin_12)
- net GPIO_EXT_B_06 renamed GPIO_10
- net GPIO_10: now also J2.9 (Pin_9)
- net GPIO_EXT_B_07 renamed GPIO_11
- net GPIO_11: now also J2.10 (Pin_10)
- net GPIO_EXT_C_02 renamed GPIO_12
- net GPIO_12: now also J2.7 (Pin_7)
- net GPIO_EXT_C_03 renamed GPIO_13
- net GPIO_13: now also J2.8 (Pin_8)
- net GPIO_EXT_C_04 renamed GPIO_14
- net GPIO_14: now also J2.5 (Pin_5)
- net GPIO_EXT_C_05 renamed GPIO_15
- net GPIO_15: now also J2.6 (Pin_6)
- net GPIO_EXT_C_06 renamed BUTTON_PRG
- net I2C_00_SCL renamed I2C_USR_SCL
- net I2C_USR_SCL: now also J2.44 (Pin_44), R54.2
- net I2C_00_SDA renamed I2C_USR_SDA
- net I2C_USR_SDA: now also J2.46 (Pin_46), R53.2
- net SPI_00_CS renamed SPI_USR_CS
- net SPI_USR_CS: now also J2.37 (Pin_37)
- net SPI_00_MISO renamed SPI_USR_MISO
- net SPI_USR_MISO: now also J2.33 (Pin_33)
- net SPI_00_MOSI renamed SPI_USR_MOSI
- net SPI_USR_MOSI: now also J2.31 (Pin_31)
- net SPI_00_SCK renamed SPI_USR_SCK
- net SPI_USR_SCK: now also J2.35 (Pin_35)
- no-connect marks 9 -> 5
Other:
- note removed: "--------------------------------\nTODO\n--------------------------------\n- [ ] CHECK PINS\n- [ ] ADD SPIs TO *GPIO PORT*\n--------------------------------"
- moved on the sheet: C12, C3, C4, C5, C6, C7, C8, C9, D1, D10, D11, D12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
