File: KLST_SHEEP/audio_codec_WM8731.sch (KiCad schematic (older format))
At the start: 39 parts, among them J6 HEADPHONES+MIC, J7 LINE_IN, J8 LINE_OUT, U3 WM8731SEDS

Commit message: added NHD display
Parts:
- renumbered C16 to C27, C17 to C28, C18 to C29, C19 to C30, C20 to C31, C21 to C32, C22 to C33, C23 to C34, C24 to C35, C25 to C36, C26 to C37, C27 to C38, C28 to C39, C29 to C40, C30 to C41, C31 to C42, C32 to C43, C33 to C44, C34 to C45, C35 to C46, J7 to J10, J8 to J11, J6 to J9, R10 to R13, R11 to R14, R12 to R15, R13 to R16, R14 to R17, R15 to R18, R16 to R19, R17 to R20, R18 to R21, R19 to R22, R20 to R23, R21 to R24, R22 to R25, R23 to R26, R24 to R27

Commit message: added icons
Parts:
- renumbered J9 to J10, J10 to J11, J11 to J12, R13 to R26, R14 to R27, R15 to R28, R16 to R29, R17 to R30, R18 to R31, R19 to R32, R20 to R33, R21 to R34, R22 to R35, R23 to R36, R24 to R37, R25 to R38, R26 to R39, R27 to R40

Commit message: KLST_SHEEP-v0.1
Parts:
- C27, C28: JLCPCB Part # (none) -> C3345; LCSC Part # C3345 -> (none)
- C29, C33, C35, C37, C38: JLCPCB Part # (none) -> C7175; LCSC Part # C7175 -> (none)
- C30, C34, C36: JLCPCB Part # (none) -> C53172; LCSC Part # C53172 -> (none)
- C31, C40, C42, C44, C46: JLCPCB Part # (none) -> C7171; LCSC Part # C7171 -> (none)
- C32, C39, C41, C43, C45: JLCPCB Part # (none) -> C1525; LCSC Part # C1525 -> (none)
- J10, J11, J12: JLCPCB Part # (none) -> C128987; LCSC Part # C128987 -> (none)
- R26, R27, R32, R38, R40: JLCPCB Part # (none) -> C17713; LCSC Part # C17713 -> (none)
- R28: JLCPCB Part # (none) -> C17798; LCSC Part # C17798 -> (none)
- R29, R30: JLCPCB Part # (none) -> C25879; LCSC Part # C25879 -> (none)
- R31: JLCPCB Part # (none) -> C17630; LCSC Part # C17630 -> (none)
- R33, R34, R35, R36: JLCPCB Part # (none) -> C4382; LCSC Part # C4382 -> (none)
- R37, R39: JLCPCB Part # (none) -> C17408; LCSC Part # C17408 -> (none)
- U3: JLCPCB Part # (none) -> DNF; LCSC Part # C323837 -> (none)
