File: KLST_SHEEP/rotary_encoder__with_push_button.sch (KiCad schematic (older format))
At the start: 10 parts, among them SW3 ENCODER

Commit message: added NHD display
Parts:
- renumbered C36 to C47, C37 to C48, C38 to C49, R25 to R28, R26 to R29, R27 to R30, R28 to R31, R29 to R32, R30 to R33
Changed lines of the file:
@@
 $EndDescr
 $Comp
-L power:GND #PWR059
+L power:GND #PWR063
 U 1 1 606340DF
 P 5950 5200
-AR Path="/60628872/606340DF" Ref="#PWR059"  Part="1"
+AR Path="/60628872/606340DF" Ref="#PWR063"  Part="1"
 AR Path="/6067FDCF/606340DF" Ref="#PWR?"  Part="1"
 AR Path="/606B66E6/606340DF" Ref="#PWR?"  Part="1"
-AR Path="/6075A95B/606340DF" Ref="#PWR061"  Part="1"
-AR Path="/607910C2/606340DF" Ref="#PWR063"  Part="1"
-F 0 "#PWR063" H 5950 4950 50  0001 C CNN
+AR Path="/6075A95B/606340DF" Ref="#PWR065"  Part="1"
+AR Path="/607910C2/606340DF" Ref="#PWR067"  Part="1"
+F 0 "#PWR067" H 5950 4950 50  0001 C CNN
 F 1 "GND" H 5950 5050 50  0000 C CNN
 F 2 "" H 5950 5200 50  0001 C CNN
@@
 $EndComp
 $Comp
-L Device:C_Small C37
+L Device:C_Small C48
 U 1 1 606340E5
 P 5200 4900
-AR Path="/60628872/606340E5" Ref="C37"  Part="1"
+AR Path="/60628872/606340E5" Ref="C48"  Part="1"
 AR Path="/6067FDCF/606340E5" Ref="C?"  Part="1"
 AR Path="/606B66E6/606340E5" Ref="C?"  Part="1"
-AR Path="/6075A95B/606340E5" Ref="C40"  Part="1"
-AR Path="/607910C2/606340E5" Ref="C43"  Part="1"
-F 0 "C43" H 5292 4946 50  0000 L CNN
+AR Path="/6075A95B/606340E5" Ref="C51"  Part="1"
+AR Path="/607910C2/606340E5" Ref="C54"  Part="1"
+F 0 "C54" H 5292 4946 50  0000 L CNN
 F 1 "100nF" H 5292 4855 50  0000 L CNN
 F 2 "Capacitor_SMD:C_0402_1005Metric" H 5200 4900 50  0001 C CNN
@@
 $EndComp
 $Comp
-L Device:R R29
+L Device:R R32
 U 1 1 606340EB
 P 4900 4500
-AR Path="/60628872/606340EB" Ref="R29"  Part="1"
+AR Path="/60628872/606340EB" Ref="R32"  Part="1"
 AR Path="/6067FDCF/606340EB" Ref="R?"  Part="1"
 AR Path="/606B66E6/606340EB" Ref="R?"  Part="1"
-AR Path="/6075A95B/606340EB" Ref="R35"  Part="1"
-AR Path="/607910C2/606340EB" Ref="R41"  Part="1"
-F 0 "R41" V 4800 4500 50  0000 C CNN
+AR Path="/6075A95B/606340EB" Ref="R38"  Part="1"
+AR Path="/607910C2/606340EB" Ref="R44"  Part="1"
+F 0 "R44" V 4800 4500 50  0000 C CNN
 F 1 "10K" V 5000 4500 50  0000 C CNN
 F 2 "Resistor_SMD:R_0402_1005Metric" V 4830 4500 50  0001 C CNN
@@
 $EndComp
 $Comp
-L Device:C_Small C38
+L Device:C_Small C49
 U 1 1 606340F1
 P 6650 4900
-AR Path="/60628872/606340F1" Ref="C38"  Part="1"
+AR Path="/60628872/606340F1" Ref="C49"  Part="1"
 AR Path="/6067FDCF/606340F1" Ref="C?"  Part="1"
 AR Path="/606B66E6/606340F1" Ref="C?"  Part="1"
-AR Path="/6075A95B/606340F1" Ref="C41"  Part="1"
-AR Path="/607910C2/606340F1" Ref="C44"  Part="1"
-F 0 "C44" H 6742 4946 50  0000 L CNN
+AR Path="/6075A95B/606340F1" Ref="C52"  Part="1"
+AR Path="/607910C2/606340F1" Ref="C55"  Part="1"
+F 0 "C55" H 6742 4946 50  0000 L CNN
 F 1 "100nF" H 6742 4855 50  0000 L CNN
 F 2 "Capacitor_SMD:C_0402_1005Metric" H 6650 4900 50  0001 C CNN
@@
 $EndComp
 $Comp
-L Device:R R30
+L Device:R R33
 U 1 1 606340F7
 P 6950 4500
-AR Path="/60628872/606340F7" Ref="R30"  Part="1"
+AR Path="/60628872/606340F7" Ref="R33"  Part="1"
 AR Path="/6067FDCF/606340F7" Ref="R?"  Part="1"
 AR Path="/606B66E6/606340F7" Ref="R?"  Part="1"
-AR Path="/6075A95B/606340F7" Ref="R36"  Part="1"
-AR Path="/607910C2/606340F7" Ref="R42"  Part="1"
-F 0 "R42" V 6850 4500 50  0000 C CNN
+AR Path="/6075A95B/606340F7" Ref="R39"  Part="1"
+AR Path="/607910C2/606340F7" Ref="R45"  Part="1"
+F 0 "R45" V 6850 4500 50  0000 C CNN
 F 1 "10K" V 7050 4500 50  0000 C CNN
 F 2 "Resistor_SMD:R_0402_1005Metric" V 6880 4500 50  0001 C CNN
@@
 	5950 5100 5950 4500
 $Comp
-L Device:R R27
+L Device:R R30
 U 1 1 60634116
 P 6650 3900
-AR Path="/60628872/60634116" Ref="R27"  Part="1"
+AR Path="/60628872/60634116" Ref="R30"  Part="1"
 AR Path="/6067FDCF/60634116" Ref="R?"  Part="1"
 AR Path="/606B66E6/60634116" Ref="R?"  Part="1"
-AR Path="/6075A95B/60634116" Ref="R33"  Part="1"
-AR Path="/607910C2/60634116" Ref="R39"  Part="1"
-F 0 "R39" H 6580 3946 50  0000 R CNN
+AR Path="/6075A95B/60634116" Ref="R36"  Part="1"
+AR Path="/607910C2/60634116" Ref="R42"  Part="1"
+F 0 "R42" H 6580 3946 50  0000 R CNN
 F 1 "10K" H 6580 3855 50  0000 R CNN
 F 2 "Resistor_SMD:R_0402_1005Metric" V 6580 3900 50  0001 C CNN
@@
 	6650 4050 6650 4500
 $Comp
-L Device:R R28
+L Device:R R31
 U 1 1 6063411D
 P 5200 3950
-AR Path="/60628872/6063411D" Ref="R28"  Part="1"
+AR Path="/60628872/6063411D" Ref="R31"  Part="1"
 AR Path="/6067FDCF/6063411D" Ref="R?"  Part="1"
 AR Path="/606B66E6/6063411D" Ref="R?"  Part="1"
-AR Path="/6075A95B/6063411D" Ref="R34"  Part="1"
-AR Path="/607910C2/6063411D" Ref="R40"  Part="1"
-F 0 "R40" H 5130 3996 50  0000 R CNN
+AR Path="/6075A95B/6063411D" Ref="R37"  Part="1"
+AR Path="/607910C2/6063411D" Ref="R43"  Part="1"
+F 0 "R43" H 5130 3996 50  0000 R CNN
 F 1 "10K" H 5130 3905 50  0000 R CNN
 F 2 "Resistor_SMD:R_0402_1005Metric" V 5130 3950 50  0001 C CNN
@@
 Connection ~ 5850 2950
 $Comp
-L Device:R R25
+L Device:R R28
 U 1 1 60634126
 P 5850 3150
-AR Path="/60628872/60634126" Ref="R25"  Part="1"
+AR Path="/60628872/60634126" Ref="R28"  Part="1"
 AR Path="/6067FDCF/60634126" Ref="R?"  Part="1"
 AR Path="/606B66E6/60634126" Ref="R?"  Part="1"
-AR Path="/6075A95B/60634126" Ref="R31"  Part="1"
-AR Path="/607910C2/60634126" Ref="R37"  Part="1"
-F 0 "R37" H 5950 3100 50  0000 L CNN
+AR Path="/6075A95B/60634126" Ref="R34"  Part="1"
+AR Path="/607910C2/60634126" Ref="R40"  Part="1"
+F 0 "R40" H 5950 3100 50  0000 L CNN
 F 1 "10K" H 5950 3200 50  0000 L CNN
 F 2 "Resistor_SMD:R_0402_1005Metric" V 5780 3150 50  0001 C CNN
@@
 $EndComp
 $Comp
-L Device:C_Small C36
+L Device:C_Small C47
 U 1 1 6063412C
 P 6350 3700
-AR Path="/60628872/6063412C" Ref="C36"  Part="1"
+AR Path="/60628872/6063412C" Ref="C47"  Part="1"
 AR Path="/6067FDCF/6063412C" Ref="C?"  Part="1"
 AR Path="/606B66E6/6063412C" Ref="C?"  Part="1"
-AR Path="/6075A95B/6063412C" Ref="C39"  Part="1"
-AR Path="/607910C2/6063412C" Ref="C42"  Part="1"
-F 0 "C42" H 6442 3746 50  0000 L CNN
+AR Path="/6075A95B/6063412C" Ref="C50"  Part="1"
+AR Path="/607910C2/6063412C" Ref="C53"  Part="1"
+F 0 "C53" H 6442 3746 50  0000 L CNN
 F 1 "100nF" H 6442 3655 50  0000 L CNN
 F 2 "Capacitor_SMD:C_0402_1005Metric" H 6350 3700 50  0001 C CNN
@@
 	5850 3300 5850 3400
 $Comp
-L Device:R R26
+L Device:R R29
 U 1 1 60634138
 P 6100 3400
-AR Path="/60628872/60634138" Ref="R26"  Part="1"
+AR Path="/60628872/60634138" Ref="R29"  Part="1"
 AR Path="/6067FDCF/60634138" Ref="R?"  Part="1"
 AR Path="/606B66E6/60634138" Ref="R?"  Part="1"
-AR Path="/6075A95B/60634138" Ref="R32"  Part="1"
-AR Path="/607910C2/60634138" Ref="R38"  Part="1"
-F 0 "R38" V 6000 3400 50  0000 C CNN
+AR Path="/6075A95B/60634138" Ref="R35"  Part="1"
+AR Path="/607910C2/60634138" Ref="R41"  Part="1"
+F 0 "R41" V 6000 3400 50  0000 C CNN
 F 1 "1K" V 6200 3400 50  0000 C CNN
 F 2 "Resistor_SMD:R_0402_1005Metric" V 6030 3400 50  0001 C CNN
@@
 P 5950 2850
 AR Path="/615FFAB7" Ref="#PWR?"  Part="1"
-AR Path="/60628872/615FFAB7" Ref="#PWR058"  Part="1"
-AR Path="/6075A95B/615FFAB7" Ref="#PWR060"  Part="1"
-AR Path="/607910C2/615FFAB7" Ref="#PWR062"  Part="1"
-F 0 "#PWR062" H 5950 2700 50  0001 C CNN
+AR Path="/60628872/615FFAB7" Ref="#PWR062"  Part="1"
+AR Path="/6075A95B/615FFAB7" Ref="#PWR064"  Part="1"
+AR Path="/607910C2/615FFAB7" Ref="#PWR066"  Part="1"
+F 0 "#PWR066" H 5950 2700 50  0001 C CNN
 F 1 "+3V3" H 5965 3023 50  0000 C CNN
 F 2 "" H 5950 2850 50  0001 C CNN

Commit message: added screen, added icon
Changed lines of the file:
@@
 $Descr A4 11693 8268
 encoding utf-8
-Sheet 3 7
+Sheet 3 6
 Title "KLST_SHEEP"
 Date "2021-05-01"
@@
 AR Path="/6075A95B/606340DF" Ref="#PWR065"  Part="1"
 AR Path="/607910C2/606340DF" Ref="#PWR067"  Part="1"
-F 0 "#PWR067" H 5950 4950 50  0001 C CNN
+F 0 "#PWR065" H 5950 4950 50  0001 C CNN
 F 1 "GND" H 5950 5050 50  0000 C CNN
 F 2 "" H 5950 5200 50  0001 C CNN
@@
 AR Path="/6075A95B/606340E5" Ref="C51"  Part="1"
 AR Path="/607910C2/606340E5" Ref="C54"  Part="1"
-F 0 "C54" H 5292 4946 50  0000 L CNN
+F 0 "C51" H 5292 4946 50  0000 L CNN
 F 1 "100nF" H 5292 4855 50  0000 L CNN
 F 2 "Capacitor_SMD:C_0402_1005Metric" H 5200 4900 50  0001 C CNN
@@
 AR Path="/6075A95B/606340EB" Ref="R38"  Part="1"
 AR Path="/607910C2/606340EB" Ref="R44"  Part="1"
-F 0 "R44" V 4800 4500 50  0000 C CNN
+F 0 "R38" V 4800 4500 50  0000 C CNN
 F 1 "10K" V 5000 4500 50  0000 C CNN
 F 2 "Resistor_SMD:R_0402_1005Metric" V 4830 4500 50  0001 C CNN
@@
 AR Path="/6075A95B/606340F1" Ref="C52"  Part="1"
 AR Path="/607910C2/606340F1" Ref="C55"  Part="1"
-F 0 "C55" H 6742 4946 50  0000 L CNN
+F 0 "C52" H 6742 4946 50  0000 L CNN
 F 1 "100nF" H 6742 4855 50  0000 L CNN
 F 2 "Capacitor_SMD:C_0402_1005Metric" H 6650 4900 50  0001 C CNN
@@
 AR Path="/6075A95B/606340F7" Ref="R39"  Part="1"
 AR Path="/607910C2/606340F7" Ref="R45"  Part="1"
-F 0 "R45" V 6850 4500 50  0000 C CNN
+F 0 "R39" V 6850 4500 50  0000 C CNN
 F 1 "10K" V 7050 4500 50  0000 C CNN
 F 2 "Resistor_SMD:R_0402_1005Metric" V 6880 4500 50  0001 C CNN
@@
 AR Path="/6075A95B/606340FD" Ref="SW4"  Part="1"
 AR Path="/607910C2/606340FD" Ref="SW5"  Part="1"
-F 0 "SW5" V 5996 4430 50  0000 L CNN
+F 0 "SW4" V 5996 4430 50  0000 L CNN
 F 1 "ENCODER" V 5905 4430 50  0000 L CNN
 F 2 "Rotary_Encoder:RotaryEncoder_Alps_EC12E-Switch_Vertical_H20mm" H 5800 4360 50  0001 C CNN
@@
 AR Path="/6075A95B/60634116" Ref="R36"  Part="1"
 AR Path="/607910C2/60634116" Ref="R42"  Part="1"
-F 0 "R42" H 6580 3946 50  0000 R CNN
+F 0 "R36" H 6580 3946 50  0000 R CNN
 F 1 "10K" H 6580 3855 50  0000 R CNN
 F 2 "Resistor_SMD:R_0402_1005Metric" V 6580 3900 50  0001 C CNN
@@
 AR Path="/6075A95B/6063411D" Ref="R37"  Part="1"
 AR Path="/607910C2/6063411D" Ref="R43"  Part="1"
-F 0 "R43" H 5130 3996 50  0000 R CNN
+F 0 "R37" H 5130 3996 50  0000 R CNN
 F 1 "10K" H 5130 3905 50  0000 R CNN
 F 2 "Resistor_SMD:R_0402_1005Metric" V 5130 3950 50  0001 C CNN
@@
 AR Path="/6075A95B/60634126" Ref="R34"  Part="1"
 AR Path="/607910C2/60634126" Ref="R40"  Part="1"
-F 0 "R40" H 5950 3100 50  0000 L CNN
+F 0 "R34" H 5950 3100 50  0000 L CNN
 F 1 "10K" H 5950 3200 50  0000 L CNN
 F 2 "Resistor_SMD:R_0402_1005Metric" V 5780 3150 50  0001 C CNN
@@
 AR Path="/6075A95B/6063412C" Ref="C50"  Part="1"
 AR Path="/607910C2/6063412C" Ref="C53"  Part="1"
-F 0 "C53" H 6442 3746 50  0000 L CNN
+F 0 "C50" H 6442 3746 50  0000 L CNN
 F 1 "100nF" H 6442 3655 50  0000 L CNN
 F 2 "Capacitor_SMD:C_0402_1005Metric" H 6350 3700 50  0001 C CNN
@@
 AR Path="/6075A95B/60634138" Ref="R35"  Part="1"
 AR Path="/607910C2/60634138" Ref="R41"  Part="1"
-F 0 "R41" V 6000 3400 50  0000 C CNN
+F 0 "R35" V 6000 3400 50  0000 C CNN
 F 1 "1K" V 6200 3400 50  0000 C CNN
 F 2 "Resistor_SMD:R_0402_1005Metric" V 6030 3400 50  0001 C CNN
@@
 AR Path="/6075A95B/615FFAB7" Ref="#PWR064"  Part="1"
 AR Path="/607910C2/615FFAB7" Ref="#PWR066"  Part="1"
-F 0 "#PWR066" H 5950 2700 50  0001 C CNN
+F 0 "#PWR064" H 5950 2700 50  0001 C CNN
 F 1 "+3V3" H 5965 3023 50  0000 C CNN
 F 2 "" H 5950 2850 50  0001 C CNN

Commit message: added icons
Parts:
- renumbered R28 to R41, R29 to R42, R30 to R43, R31 to R44, R32 to R45, R33 to R46
Changed lines of the file:
@@
 $EndDescr
 $Comp
-L power:GND #PWR063
+L power:GND #PWR067
 U 1 1 606340DF
 P 5950 5200
-AR Path="/60628872/606340DF" Ref="#PWR063"  Part="1"
+AR Path="/60628872/606340DF" Ref="#PWR067"  Part="1"
 AR Path="/6067FDCF/606340DF" Ref="#PWR?"  Part="1"
 AR Path="/606B66E6/606340DF" Ref="#PWR?"  Part="1"
-AR Path="/6075A95B/606340DF" Ref="#PWR065"  Part="1"
-AR Path="/607910C2/606340DF" Ref="#PWR067"  Part="1"
-F 0 "#PWR065" H 5950 4950 50  0001 C CNN
+AR Path="/6075A95B/606340DF" Ref="#PWR069"  Part="1"
+AR Path="/607910C2/606340DF" Ref="#PWR?"  Part="1"
+F 0 "#PWR069" H 5950 4950 50  0001 C CNN
 F 1 "GND" H 5950 5050 50  0000 C CNN
 F 2 "" H 5950 5200 50  0001 C CNN
@@
 AR Path="/606B66E6/606340E5" Ref="C?"  Part="1"
 AR Path="/6075A95B/606340E5" Ref="C51"  Part="1"
-AR Path="/607910C2/606340E5" Ref="C54"  Part="1"
+AR Path="/607910C2/606340E5" Ref="C?"  Part="1"
 F 0 "C51" H 5292 4946 50  0000 L CNN
 F 1 "100nF" H 5292 4855 50  0000 L CNN
@@
 $EndComp
 $Comp
-L Device:R R32
+L Device:R R45
 U 1 1 606340EB
 P 4900 4500
-AR Path="/60628872/606340EB" Ref="R32"  Part="1"
+AR Path="/60628872/606340EB" Ref="R45"  Part="1"
 AR Path="/6067FDCF/606340EB" Ref="R?"  Part="1"
 AR Path="/606B66E6/606340EB" Ref="R?"  Part="1"
-AR Path="/6075A95B/606340EB" Ref="R38"  Part="1"
-AR Path="/607910C2/606340EB" Ref="R44"  Part="1"
-F 0 "R38" V 4800 4500 50  0000 C CNN
+AR Path="/6075A95B/606340EB" Ref="R51"  Part="1"
+AR Path="/607910C2/606340EB" Ref="R?"  Part="1"
+F 0 "R51" V 4800 4500 50  0000 C CNN
 F 1 "10K" V 5000 4500 50  0000 C CNN
 F 2 "Resistor_SMD:R_0402_1005Metric" V 4830 4500 50  0001 C CNN
@@
 AR Path="/606B66E6/606340F1" Ref="C?"  Part="1"
 AR Path="/6075A95B/606340F1" Ref="C52"  Part="1"
-AR Path="/607910C2/606340F1" Ref="C55"  Part="1"
+AR Path="/607910C2/606340F1" Ref="C?"  Part="1"
 F 0 "C52" H 6742 4946 50  0000 L CNN
 F 1 "100nF" H 6742 4855 50  0000 L CNN
@@
 $EndComp
 $Comp
-L Device:R R33
+L Device:R R46
 U 1 1 606340F7
 P 6950 4500
-AR Path="/60628872/606340F7" Ref="R33"  Part="1"
+AR Path="/60628872/606340F7" Ref="R46"  Part="1"
 AR Path="/6067FDCF/606340F7" Ref="R?"  Part="1"
 AR Path="/606B66E6/606340F7" Ref="R?"  Part="1"
-AR Path="/6075A95B/606340F7" Ref="R39"  Part="1"
-AR Path="/607910C2/606340F7" Ref="R45"  Part="1"
-F 0 "R39" V 6850 4500 50  0000 C CNN
+AR Path="/6075A95B/606340F7" Ref="R52"  Part="1"
+AR Path="/607910C2/606340F7" Ref="R?"  Part="1"
+F 0 "R52" V 6850 4500 50  0000 C CNN
 F 1 "10K" V 7050 4500 50  0000 C CNN
 F 2 "Resistor_SMD:R_0402_1005Metric" V 6880 4500 50  0001 C CNN
@@
 AR Path="/606B66E6/606340FD" Ref="SW?"  Part="1"
 AR Path="/6075A95B/606340FD" Ref="SW4"  Part="1"
-AR Path="/607910C2/606340FD" Ref="SW5"  Part="1"
+AR Path="/607910C2/606340FD" Ref="SW?"  Part="1"
 F 0 "SW4" V 5996 4430 50  0000 L CNN
 F 1 "ENCODER" V 5905 4430 50  0000 L CNN
@@
 	5950 5100 5950 4500
 $Comp
-L Device:R R30
+L Device:R R43
 U 1 1 60634116
 P 6650 3900
-AR Path="/60628872/60634116" Ref="R30"  Part="1"
+AR Path="/60628872/60634116" Ref="R43"  Part="1"
 AR Path="/6067FDCF/60634116" Ref="R?"  Part="1"
 AR Path="/606B66E6/60634116" Ref="R?"  Part="1"
-AR Path="/6075A95B/60634116" Ref="R36"  Part="1"
-AR Path="/607910C2/60634116" Ref="R42"  Part="1"
-F 0 "R36" H 6580 3946 50  0000 R CNN
+AR Path="/6075A95B/60634116" Ref="R49"  Part="1"
+AR Path="/607910C2/60634116" Ref="R?"  Part="1"
+F 0 "R49" H 6580 3946 50  0000 R CNN
 F 1 "10K" H 6580 3855 50  0000 R CNN
 F 2 "Resistor_SMD:R_0402_1005Metric" V 6580 3900 50  0001 C CNN
@@
 	6650 4050 6650 4500
 $Comp
-L Device:R R31
+L Device:R R44
 U 1 1 6063411D
 P 5200 3950
-AR Path="/60628872/6063411D" Ref="R31"  Part="1"
+AR Path="/60628872/6063411D" Ref="R44"  Part="1"
 AR Path="/6067FDCF/6063411D" Ref="R?"  Part="1"
 AR Path="/606B66E6/6063411D" Ref="R?"  Part="1"
-AR Path="/6075A95B/6063411D" Ref="R37"  Part="1"
-AR Path="/607910C2/6063411D" Ref="R43"  Part="1"
-F 0 "R37" H 5130 3996 50  0000 R CNN
+AR Path="/6075A95B/6063411D" Ref="R50"  Part="1"
+AR Path="/607910C2/6063411D" Ref="R?"  Part="1"
+F 0 "R50" H 5130 3996 50  0000 R CNN
 F 1 "10K" H 5130 3905 50  0000 R CNN
 F 2 "Resistor_SMD:R_0402_1005Metric" V 5130 3950 50  0001 C CNN
@@
 Connection ~ 5850 2950
 $Comp
-L Device:R R28
+L Device:R R41
 U 1 1 60634126
 P 5850 3150
-AR Path="/60628872/60634126" Ref="R28"  Part="1"
+AR Path="/60628872/60634126" Ref="R41"  Part="1"
 AR Path="/6067FDCF/60634126" Ref="R?"  Part="1"
 AR Path="/606B66E6/60634126" Ref="R?"  Part="1"
-AR Path="/6075A95B/60634126" Ref="R34"  Part="1"
-AR Path="/607910C2/60634126" Ref="R40"  Part="1"
-F 0 "R34" H 5950 3100 50  0000 L CNN
+AR Path="/6075A95B/60634126" Ref="R47"  Part="1"
+AR Path="/607910C2/60634126" Ref="R?"  Part="1"
+F 0 "R47" H 5950 3100 50  0000 L CNN
 F 1 "10K" H 5950 3200 50  0000 L CNN
 F 2 "Resistor_SMD:R_0402_1005Metric" V 5780 3150 50  0001 C CNN
@@
 AR Path="/606B66E6/6063412C" Ref="C?"  Part="1"
 AR Path="/6075A95B/6063412C" Ref="C50"  Part="1"
-AR Path="/607910C2/6063412C" Ref="C53"  Part="1"
+AR Path="/607910C2/6063412C" Ref="C?"  Part="1"
 F 0 "C50" H 6442 3746 50  0000 L CNN
 F 1 "100nF" H 6442 3655 50  0000 L CNN
@@
 	5850 3300 5850 3400
 $Comp
-L Device:R R29
+L Device:R R42
 U 1 1 60634138
 P 6100 3400
-AR Path="/60628872/60634138" Ref="R29"  Part="1"
+AR Path="/60628872/60634138" Ref="R42"  Part="1"
 AR Path="/6067FDCF/60634138" Ref="R?"  Part="1"
 AR Path="/606B66E6/60634138" Ref="R?"  Part="1"
-AR Path="/6075A95B/60634138" Ref="R35"  Part="1"
-AR Path="/607910C2/60634138" Ref="R41"  Part="1"
-F 0 "R35" V 6000 3400 50  0000 C CNN
+AR Path="/6075A95B/60634138" Ref="R48"  Part="1"
+AR Path="/607910C2/60634138" Ref="R?"  Part="1"
+F 0 "R48" V 6000 3400 50  0000 C CNN
 F 1 "1K" V 6200 3400 50  0000 C CNN
 F 2 "Resistor_SMD:R_0402_1005Metric" V 6030 3400 50  0001 C CNN
@@
 P 5950 2850
 AR Path="/615FFAB7" Ref="#PWR?"  Part="1"
-AR Path="/60628872/615FFAB7" Ref="#PWR062"  Part="1"
-AR Path="/6075A95B/615FFAB7" Ref="#PWR064"  Part="1"
-AR Path="/607910C2/615FFAB7" Ref="#PWR066"  Part="1"
-F 0 "#PWR064" H 5950 2700 50  0001 C CNN
+AR Path="/60628872/615FFAB7" Ref="#PWR066"  Part="1"
+AR Path="/6075A95B/615FFAB7" Ref="#PWR068"  Part="1"
+AR Path="/607910C2/615FFAB7" Ref="#PWR?"  Part="1"
+F 0 "#PWR068" H 5950 2700 50  0001 C CNN
 F 1 "+3V3" H 5965 3023 50  0000 C CNN
 F 2 "" H 5950 2850 50  0001 C CNN

Commit message: started routing GPIOs + LEDs
Changed lines of the file:
@@
 $Descr A4 11693 8268
 encoding utf-8
-Sheet 3 6
+Sheet 5 6
 Title "KLST_SHEEP"
 Date "2021-05-01"
@@
 AR Path="/6075A95B/606340E5" Ref="C51"  Part="1"
 AR Path="/607910C2/606340E5" Ref="C?"  Part="1"
-F 0 "C51" H 5292 4946 50  0000 L CNN
+F 0 "C48" H 5292 4946 50  0000 L CNN
 F 1 "100nF" H 5292 4855 50  0000 L CNN
 F 2 "Capacitor_SMD:C_0402_1005Metric" H 5200 4900 50  0001 C CNN
@@
 AR Path="/6075A95B/606340EB" Ref="R51"  Part="1"
 AR Path="/607910C2/606340EB" Ref="R?"  Part="1"
-F 0 "R51" V 4800 4500 50  0000 C CNN
+F 0 "R45" V 4800 4500 50  0000 C CNN
 F 1 "10K" V 5000 4500 50  0000 C CNN
 F 2 "Resistor_SMD:R_0402_1005Metric" V 4830 4500 50  0001 C CNN
@@
 AR Path="/6075A95B/606340F1" Ref="C52"  Part="1"
 AR Path="/607910C2/606340F1" Ref="C?"  Part="1"
-F 0 "C52" H 6742 4946 50  0000 L CNN
+F 0 "C49" H 6742 4946 50  0000 L CNN
 F 1 "100nF" H 6742 4855 50  0000 L CNN
 F 2 "Capacitor_SMD:C_0402_1005Metric" H 6650 4900 50  0001 C CNN
@@
 AR Path="/6075A95B/606340F7" Ref="R52"  Part="1"
 AR Path="/607910C2/606340F7" Ref="R?"  Part="1"
-F 0 "R52" V 6850 4500 50  0000 C CNN
+F 0 "R46" V 6850 4500 50  0000 C CNN
 F 1 "10K" V 7050 4500 50  0000 C CNN
 F 2 "Resistor_SMD:R_0402_1005Metric" V 6880 4500 50  0001 C CNN
@@
 AR Path="/6075A95B/606340FD" Ref="SW4"  Part="1"
 AR Path="/607910C2/606340FD" Ref="SW?"  Part="1"
-F 0 "SW4" V 5996 4430 50  0000 L CNN
+F 0 "SW3" V 5996 4430 50  0000 L CNN
 F 1 "ENCODER" V 5905 4430 50  0000 L CNN
 F 2 "Rotary_Encoder:RotaryEncoder_Alps_EC12E-Switch_Vertical_H20mm" H 5800 4360 50  0001 C CNN
@@
 AR Path="/6075A95B/60634116" Ref="R49"  Part="1"
 AR Path="/607910C2/60634116" Ref="R?"  Part="1"
-F 0 "R49" H 6580 3946 50  0000 R CNN
+F 0 "R43" H 6580 3946 50  0000 R CNN
 F 1 "10K" H 6580 3855 50  0000 R CNN
 F 2 "Resistor_SMD:R_0402_1005Metric" V 6580 3900 50  0001 C CNN
@@
 AR Path="/6075A95B/6063411D" Ref="R50"  Part="1"
 AR Path="/607910C2/6063411D" Ref="R?"  Part="1"
-F 0 "R50" H 5130 3996 50  0000 R CNN
+F 0 "R44" H 5130 3996 50  0000 R CNN
 F 1 "10K" H 5130 3905 50  0000 R CNN
 F 2 "Resistor_SMD:R_0402_1005Metric" V 5130 3950 50  0001 C CNN
@@
 AR Path="/6075A95B/60634126" Ref="R47"  Part="1"
 AR Path="/607910C2/60634126" Ref="R?"  Part="1"
-F 0 "R47" H 5950 3100 50  0000 L CNN
+F 0 "R41" H 5950 3100 50  0000 L CNN
 F 1 "10K" H 5950 3200 50  0000 L CNN
 F 2 "Resistor_SMD:R_0402_1005Metric" V 5780 3150 50  0001 C CNN
@@
 AR Path="/6075A95B/6063412C" Ref="C50"  Part="1"
 AR Path="/607910C2/6063412C" Ref="C?"  Part="1"
-F 0 "C50" H 6442 3746 50  0000 L CNN
+F 0 "C47" H 6442 3746 50  0000 L CNN
 F 1 "100nF" H 6442 3655 50  0000 L CNN
 F 2 "Capacitor_SMD:C_0402_1005Metric" H 6350 3700 50  0001 C CNN
@@
 AR Path="/6075A95B/60634138" Ref="R48"  Part="1"
 AR Path="/607910C2/60634138" Ref="R?"  Part="1"
-F 0 "R48" V 6000 3400 50  0000 C CNN
+F 0 "R42" V 6000 3400 50  0000 C CNN
 F 1 "1K" V 6200 3400 50  0000 C CNN
 F 2 "Resistor_SMD:R_0402_1005Metric" V 6030 3400 50  0001 C CNN
