File: KLST_SHEEP/rotary_encoder__with_push_button.sch (KiCad schematic (older format))
At the start: 10 parts, among them SW3 ENCODER

Commit message: finalized PCB design (v0.1)
Changed lines of the file:
@@
 AR Path="/6075A95B/606340E5" Ref="C51"  Part="1"
 AR Path="/607910C2/606340E5" Ref="C?"  Part="1"
-F 0 "C48" H 5292 4946 50  0000 L CNN
+F 0 "C51" H 5292 4946 50  0000 L CNN
 F 1 "100nF" H 5292 4855 50  0000 L CNN
 F 2 "Capacitor_SMD:C_0402_1005Metric" H 5200 4900 50  0001 C CNN
@@
 AR Path="/6075A95B/606340EB" Ref="R51"  Part="1"
 AR Path="/607910C2/606340EB" Ref="R?"  Part="1"
-F 0 "R45" V 4800 4500 50  0000 C CNN
+F 0 "R51" V 4800 4500 50  0000 C CNN
 F 1 "10K" V 5000 4500 50  0000 C CNN
 F 2 "Resistor_SMD:R_0402_1005Metric" V 4830 4500 50  0001 C CNN
@@
 AR Path="/6075A95B/606340F1" Ref="C52"  Part="1"
 AR Path="/607910C2/606340F1" Ref="C?"  Part="1"
-F 0 "C49" H 6742 4946 50  0000 L CNN
+F 0 "C52" H 6742 4946 50  0000 L CNN
 F 1 "100nF" H 6742 4855 50  0000 L CNN
 F 2 "Capacitor_SMD:C_0402_1005Metric" H 6650 4900 50  0001 C CNN
@@
 AR Path="/6075A95B/606340F7" Ref="R52"  Part="1"
 AR Path="/607910C2/606340F7" Ref="R?"  Part="1"
-F 0 "R46" V 6850 4500 50  0000 C CNN
+F 0 "R52" V 6850 4500 50  0000 C CNN
 F 1 "10K" V 7050 4500 50  0000 C CNN
 F 2 "Resistor_SMD:R_0402_1005Metric" V 6880 4500 50  0001 C CNN
@@
 AR Path="/6075A95B/606340FD" Ref="SW4"  Part="1"
 AR Path="/607910C2/606340FD" Ref="SW?"  Part="1"
-F 0 "SW3" V 5996 4430 50  0000 L CNN
+F 0 "SW4" V 5996 4430 50  0000 L CNN
 F 1 "ENCODER" V 5905 4430 50  0000 L CNN
 F 2 "Rotary_Encoder:RotaryEncoder_Alps_EC12E-Switch_Vertical_H20mm" H 5800 4360 50  0001 C CNN
@@
 AR Path="/6075A95B/60634116" Ref="R49"  Part="1"
 AR Path="/607910C2/60634116" Ref="R?"  Part="1"
-F 0 "R43" H 6580 3946 50  0000 R CNN
+F 0 "R49" H 6580 3946 50  0000 R CNN
 F 1 "10K" H 6580 3855 50  0000 R CNN
 F 2 "Resistor_SMD:R_0402_1005Metric" V 6580 3900 50  0001 C CNN
@@
 AR Path="/6075A95B/6063411D" Ref="R50"  Part="1"
 AR Path="/607910C2/6063411D" Ref="R?"  Part="1"
-F 0 "R44" H 5130 3996 50  0000 R CNN
+F 0 "R50" H 5130 3996 50  0000 R CNN
 F 1 "10K" H 5130 3905 50  0000 R CNN
 F 2 "Resistor_SMD:R_0402_1005Metric" V 5130 3950 50  0001 C CNN
@@
 AR Path="/6075A95B/60634126" Ref="R47"  Part="1"
 AR Path="/607910C2/60634126" Ref="R?"  Part="1"
-F 0 "R41" H 5950 3100 50  0000 L CNN
+F 0 "R47" H 5950 3100 50  0000 L CNN
 F 1 "10K" H 5950 3200 50  0000 L CNN
 F 2 "Resistor_SMD:R_0402_1005Metric" V 5780 3150 50  0001 C CNN
@@
 AR Path="/6075A95B/6063412C" Ref="C50"  Part="1"
 AR Path="/607910C2/6063412C" Ref="C?"  Part="1"
-F 0 "C47" H 6442 3746 50  0000 L CNN
+F 0 "C50" H 6442 3746 50  0000 L CNN
 F 1 "100nF" H 6442 3655 50  0000 L CNN
 F 2 "Capacitor_SMD:C_0402_1005Metric" H 6350 3700 50  0001 C CNN
@@
 AR Path="/6075A95B/60634138" Ref="R48"  Part="1"
 AR Path="/607910C2/60634138" Ref="R?"  Part="1"
-F 0 "R42" V 6000 3400 50  0000 C CNN
+F 0 "R48" V 6000 3400 50  0000 C CNN
 F 1 "1K" V 6200 3400 50  0000 C CNN
 F 2 "Resistor_SMD:R_0402_1005Metric" V 6030 3400 50  0001 C CNN

Commit message: KLST_SHEEP-v0.1
Parts:
- C47, C48, C49: JLCPCB Part # (none) -> C1525; LCSC Part # C1525 -> (none)
- R41, R43, R44, R45, R46: JLCPCB Part # (none) -> C25744; LCSC Part # C25744 -> (none)
- R42: JLCPCB Part # (none) -> C11702; LCSC Part # C11702 -> (none)
- SW3: JLCPCB Part # (none) -> DNF; LCSC Part # DNF -> (none)
Changed lines of the file:
@@
 F 3 "~" H 5200 4900 50  0001 C CNN
 F 4 "CL05B104KO5NNNC" H 5200 4900 50  0001 C CNN "MFR.Part #"
-F 5 "C1525" H 5200 4900 50  0001 C CNN "LCSC Part #"
+F 5 "" H 5200 4900 50  0001 C CNN "LCSC Part #"
 F 6 "-" H 5200 4900 50  0001 C CNN "Extended Part"
+F 7 "C1525" H 5200 4900 50  0001 C CNN "JLCPCB Part #"
 	1    5200 4900
 	1    0    0    -1
@@
 F 3 "~" H 4900 4500 50  0001 C CNN
 F 4 "0402WGF1002TCE" V 4900 4500 50  0001 C CNN "MFR.Part #"
-F 5 "C25744" H 4900 4500 50  0001 C CNN "LCSC Part #"
+F 5 "" H 4900 4500 50  0001 C CNN "LCSC Part #"
 F 6 "-" H 4900 4500 50  0001 C CNN "Extended Part"
+F 7 "C25744" H 4900 4500 50  0001 C CNN "JLCPCB Part #"
 	1    4900 4500
 	0    1    1    0
@@
 F 3 "~" H 6650 4900 50  0001 C CNN
 F 4 "CL05B104KO5NNNC" H 6650 4900 50  0001 C CNN "MFR.Part #"
-F 5 "C1525" H 6650 4900 50  0001 C CNN "LCSC Part #"
+F 5 "" H 6650 4900 50  0001 C CNN "LCSC Part #"
 F 6 "-" H 6650 4900 50  0001 C CNN "Extended Part"
+F 7 "C1525" H 6650 4900 50  0001 C CNN "JLCPCB Part #"
 	1    6650 4900
 	1    0    0    -1
@@
 F 3 "~" H 6950 4500 50  0001 C CNN
 F 4 "0402WGF1002TCE" V 6950 4500 50  0001 C CNN "MFR.Part #"
-F 5 "C25744" H 6950 4500 50  0001 C CNN "LCSC Part #"
+F 5 "" H 6950 4500 50  0001 C CNN "LCSC Part #"
 F 6 "-" H 6950 4500 50  0001 C CNN "Extended Part"
+F 7 "C25744" H 6950 4500 50  0001 C CNN "JLCPCB Part #"
 	1    6950 4500
 	0    1    1    0
@@
 F 4 "DNF" V 5950 4200 50  0001 C CNN "MFR.Part #"
 F 5 "-" H 5950 4200 50  0001 C CNN "Extended Part"
-F 6 "DNF" H 5950 4200 50  0001 C CNN "LCSC Part #"
+F 6 "" H 5950 4200 50  0001 C CNN "LCSC Part #"
+F 7 "DNF" H 5950 4200 50  0001 C CNN "JLCPCB Part #"
 	1    5950 4200
 	0    -1   -1   0
@@
 F 3 "~" H 6650 3900 50  0001 C CNN
 F 4 "0402WGF1002TCE" H 6650 3900 50  0001 C CNN "MFR.Part #"
-F 5 "C25744" H 6650 3900 50  0001 C CNN "LCSC Part #"
+F 5 "" H 6650 3900 50  0001 C CNN "LCSC Part #"
 F 6 "-" H 6650 3900 50  0001 C CNN "Extended Part"
+F 7 "C25744" H 6650 3900 50  0001 C CNN "JLCPCB Part #"
 	1    6650 3900
 	-1   0    0    -1
@@
 F 3 "~" H 5200 3950 50  0001 C CNN
 F 4 "0402WGF1002TCE" H 5200 3950 50  0001 C CNN "MFR.Part #"
-F 5 "C25744" H 5200 3950 50  0001 C CNN "LCSC Part #"
+F 5 "" H 5200 3950 50  0001 C CNN "LCSC Part #"
 F 6 "-" H 5200 3950 50  0001 C CNN "Extended Part"
+F 7 "C25744" H 5200 3950 50  0001 C CNN "JLCPCB Part #"
 	1    5200 3950
 	-1   0    0    -1
@@
 F 3 "~" H 5850 3150 50  0001 C CNN
 F 4 "0402WGF1002TCE" H 5850 3150 50  0001 C CNN "MFR.Part #"
-F 5 "C25744" H 5850 3150 50  0001 C CNN "LCSC Part #"
+F 5 "" H 5850 3150 50  0001 C CNN "LCSC Part #"
 F 6 "-" H 5850 3150 50  0001 C CNN "Extended Part"
+F 7 "C25744" H 5850 3150 50  0001 C CNN "JLCPCB Part #"
 	1    5850 3150
 	-1   0    0    1
@@
 F 3 "~" H 6350 3700 50  0001 C CNN
 F 4 "CL05B104KO5NNNC" H 6350 3700 50  0001 C CNN "MFR.Part #"
-F 5 "C1525" H 6350 3700 50  0001 C CNN "LCSC Part #"
+F 5 "" H 6350 3700 50  0001 C CNN "LCSC Part #"
 F 6 "-" H 6350 3700 50  0001 C CNN "Extended Part"
+F 7 "C1525" H 6350 3700 50  0001 C CNN "JLCPCB Part #"
 	1    6350 3700
 	-1   0    0    -1
@@
 F 3 "~" H 6100 3400 50  0001 C CNN
 F 4 "0402WGF1001TCE" V 6100 3400 50  0001 C CNN "MFR.Part #"
-F 5 "C11702" H 6100 3400 50  0001 C CNN "LCSC Part #"
+F 5 "" H 6100 3400 50  0001 C CNN "LCSC Part #"
 F 6 "-" H 6100 3400 50  0001 C CNN "Extended Part"
+F 7 "C11702" H 6100 3400 50  0001 C CNN "JLCPCB Part #"
 	1    6100 3400
 	0    1    1    0
