File: KLST_OCTOPUS/KLST_OCTOPUS.kicad_pcb (KiCad board)
At the start: 2 copper layers, 135 x 44.5 mm, 37 parts, among them J1 MIDI IN, J10 UART, J11 UART, J12 UART, J13 UART, J2 MIDI OUT, J3 MIDI THRU, J4 UART, J5 UART, J6 UART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

Commit message: finished PCB routing
Parts:
- X1: value KLST_SHEEP--graphics -> KLST_ICON
- moved D1 0.50 mm to (196.5, 81.0)
Routing:
- net +3V3: track 161.1 -> 155.9 mm
- net /UART_RX: track 231.8 -> 234.0 mm
- net /PWR: track 160.5 -> 159.4 mm
- net Net-(D1-Pad1): track 6.56 -> 5.85 mm
- net Net-(D1-Pad2): track 40.4 -> 39.9 mm

Commit message: finalized PCB
Parts:
- moved JP1 16.0 mm to (191.0, 108.5)
- moved D10 4.12 mm to (121.0, 96.0), turned to 180 degrees
- moved D2 4.12 mm to (159.5, 105.5), turned to 180 degrees
- moved D3 4.12 mm to (143.0, 105.5), turned to 180 degrees
- moved D4 4.12 mm to (126.5, 105.5), turned to 180 degrees
- moved D5 4.12 mm to (110.0, 105.5), turned to 180 degrees
- moved D6 4.12 mm to (187.0, 96.0), turned to 180 degrees
- moved D7 4.12 mm to (170.5, 96.0), turned to 180 degrees
- moved D8 4.12 mm to (154.0, 96.0), turned to 180 degrees
- moved D9 4.12 mm to (137.5, 96.0), turned to 180 degrees
Connections:
- R4 pad 2: unconnected-(R4-Pad2) -> Net-(R4-Pad2)
- R5 pad 2: unconnected-(R5-Pad2) -> Net-(R5-Pad2)
- U2 pad 4: unconnected-(R4-Pad2) -> Net-(R4-Pad2)
- U3 pad 4: unconnected-(R5-Pad2) -> Net-(R5-Pad2)
Routing:
- net /PWR: track 159.4 -> 145.0 mm, vias 18 -> 12
- net Net-(D6-Pad1): track 9.90 -> 14.9 mm
- net Net-(D8-Pad1): track 9.90 -> 14.8 mm
- net Net-(D7-Pad1): track 9.90 -> 14.7 mm
- net Net-(D10-Pad1): track 9.90 -> 14.7 mm
- net Net-(D9-Pad1): track 9.90 -> 14.6 mm
- net Net-(D3-Pad1): track 9.96 -> 13.2 mm
- net +3V3: track 155.9 -> 152.8 mm
- net Net-(D5-Pad1): track 9.96 -> 12.9 mm
- net Net-(D2-Pad1): track 9.96 -> 12.9 mm
- net Net-(D4-Pad1): track 9.96 -> 12.8 mm
- net unconnected-(R4-Pad2): track 2.17 -> 0.00 mm
- net Net-(R4-Pad2): track 0.00 -> 2.17 mm
- net unconnected-(R5-Pad2): track 2.17 -> 0.00 mm
- net Net-(R5-Pad2): track 0.00 -> 2.17 mm
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