File: KLST_OCTOPUS/KLST_OCTOPUS.kicad_sch (KiCad schematic)
At the start: 16 parts

Commit message: renamed project, routed traces
Parts:
- added H1, H2: MountingHole_Pad, MountingHole:MountingHole_3.2mm_M3_Pad_Via, symbol Mechanical:MountingHole_Pad
- added X1: KLST_SHEEP--graphics, DIN-5:KLST--icon, symbol KLST_SHEEP--graphics:KLST_SHEEP--graphics
- C1: value (none) -> 100uF; footprint (none) -> Capacitor_SMD:C_0805_2012Metric_Pad1.18x1.45mm_HandSolder
- D1: value (none) -> 1N914WT; footprint (none) -> Diode_SMD:D_SOD-523
- J1: value (none) -> MIDI_IN; footprint (none) -> DIN-5:DIN5-RA-PTH
- J2: value (none) -> MIDI_OUT; footprint (none) -> DIN-5:DIN5-RA-PTH
- J3: value (none) -> MIDI_THRU; footprint (none) -> DIN-5:DIN5-RA-PTH
- J4: value (none) -> UART; footprint (none) -> Connector_IDC:IDC-Header_2x03_P2.54mm_Horizontal
- JP1: value (none) -> PWR; footprint (none) -> Jumper:SolderJumper-2_P1.3mm_Bridged_RoundedPad1.0x1.5mm
- R1, R2, R4, R5: value (none) -> 47; footprint (none) -> Resistor_SMD:R_0805_2012Metric_Pad1.20x1.40mm_HandSolder
- R3: value (none) -> 220; footprint (none) -> Resistor_SMD:R_0805_2012Metric_Pad1.20x1.40mm_HandSolder
- R6: value (none) -> 470; footprint (none) -> Resistor_SMD:R_0805_2012Metric_Pad1.20x1.40mm_HandSolder
- U1: value (none) -> H11L1SR2M; footprint (none) -> Package_DIP:SMDIP-6_W9.53mm
- U2, U3: value (none) -> 74AHC1G125; footprint (none) -> Package_TO_SOT_SMD:SOT-23-5_HandSoldering
Connections:
- no-connect marks 17 -> 19

Commit message: finished PCB routing
Parts:
- J1: value MIDI_IN -> MIDI IN
- J2: value MIDI_OUT -> MIDI OUT
- J3: value MIDI_THRU -> MIDI THRU
- X1: value KLST_SHEEP--graphics -> KLST_ICON
Connections:
- no-connect marks 19 -> 15
Other:
- note added: "@NOTE(symbol is *looking* onto cable connector e.g PIN4 is on right side, looking into to socket )"
- note removed: "@NOTE(looking into the plug)"
- note removed: "if no BUFFER is used ( e.g 74AHC1G125 ) just connect 'UART_TX' here. @TODO(DECIDE ON BUFFER)"
Changed lines of the file:
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@@
   (junction (at 140.97 104.14) (diameter 0) (color 0 0 0 0)
-  )
-  (junction (at 49.53 85.09) (diameter 0) (color 0 0 0 0)
-  )
-  (junction (at 49.53 138.43) (diameter 0) (color 0 0 0 0)
   )
   (junction (at 137.16 118.11) (diameter 0) (color 0 0 0 0)
@@
   (no_connect (at 26.67 48.26))
   (no_connect (at 30.48 148.59))
-  (no_connect (at 49.53 140.97))
   (no_connect (at 25.4 33.02))
   (no_connect (at 30.48 95.25))
@@
   (no_connect (at 21.59 87.63))
   (no_connect (at 21.59 140.97))
-  (no_connect (at 49.53 90.17))
   (no_connect (at 36.83 140.97))
-  (no_connect (at 49.53 87.63))
   (no_connect (at 24.13 48.26))
   (no_connect (at 27.94 148.59))
   (no_connect (at 27.94 95.25))
-  (no_connect (at 49.53 143.51))
   (wire (pts (xy 187.96 92.71) (xy 187.96 81.28))
     (stroke (width 0) (type default) (color 0 0 0 0))
@@
     (stroke (width 0) (type default) (color 0 0 0 0))
   )
-  (polyline (pts (xy 48.26 154.94) (xy 48.26 139.7))
-    (stroke (width 0) (type default) (color 0 0 0 0))
-  )
   (wire (pts (xy 140.97 104.14) (xy 140.97 92.71))
     (stroke (width 0) (type default) (color 0 0 0 0))
@@
     (stroke (width 0) (type default) (color 0 0 0 0))
   )
-  (polyline (pts (xy 54.61 139.7) (xy 77.47 139.7))
-    (stroke (width 0) (type default) (color 0 0 0 0))
-  )
   (wire (pts (xy 67.31 25.4) (xy 67.31 27.94))
     (stroke (width 0) (type default) (color 0 0 0 0))
@@
     (stroke (width 0) (type default) (color 0 0 0 0))
   )
-  (polyline (pts (xy 77.47 139.7) (xy 77.47 154.94))
-    (stroke (width 0) (type default) (color 0 0 0 0))
-  )
   (wire (pts (xy 81.28 143.51) (xy 81.28 149.86))
     (stroke (width 0) (type default) (color 0 0 0 0))
@@
     (stroke (width 0) (type default) (color 0 0 0 0))
   )
-  (wire (pts (xy 44.45 85.09) (xy 49.53 85.09))
-    (stroke (width 0) (type default) (color 0 0 0 0))
-  )
   (wire (pts (xy 171.45 129.54) (xy 184.15 129.54))
     (stroke (width 0) (type default) (color 0 0 0 0))
@@
     (stroke (width 0) (type default) (color 0 0 0 0))
   )
-  (polyline (pts (xy 48.26 101.6) (xy 48.26 86.36))
-    (stroke (width 0) (type default) (color 0 0 0 0))
-  )
   (wire (pts (xy 161.29 40.64) (xy 161.29 41.91))
     (stroke (width 0) (type default) (color 0 0 0 0))
@@
     (stroke (width 0) (type default) (color 0 0 0 0))
   )
-  (wire (pts (xy 49.53 138.43) (xy 49.53 140.97))
-    (stroke (width 0) (type default) (color 0 0 0 0))
-  )
   (wire (pts (xy 184.15 72.39) (xy 184.15 83.82))
     (stroke (width 0) (type default) (color 0 0 0 0))
@@
     (stroke (width 0) (type default) (color 0 0 0 0))
   )
-  (polyline (pts (xy 48.26 139.7) (xy 54.61 139.7))
-    (stroke (width 0) (type default) (color 0 0 0 0))
-  )
   (wire (pts (xy 43.18 27.94) (xy 52.07 27.94))
     (stroke (width 0) (type default) (color 0 0 0 0))
@@
     (stroke (width 0) (type default) (color 0 0 0 0))
   )
-  (wire (pts (xy 44.45 138.43) (xy 49.53 138.43))
+  (wire (pts (xy 44.45 138.43) (xy 74.93 138.43))
     (stroke (width 0) (type default) (color 0 0 0 0))
   )
@@
     (stroke (width 0) (type default) (color 0 0 0 0))
   )
-  (polyline (pts (xy 48.26 86.36) (xy 54.61 86.36))
-    (stroke (width 0) (type default) (color 0 0 0 0))
-  )
   (polyline (pts (xy 13.97 57.15) (xy 16.51 57.15))
     (stroke (width 0) (type default) (color 0 0 0 0))
@@
     (stroke (width 0) (type default) (color 0 0 0 0))
   )
-  (polyline (pts (xy 54.61 86.36) (xy 77.47 86.36))
-    (stroke (width 0) (type default) (color 0 0 0 0))
-  )
   (polyline (pts (xy 214.63 13.97) (xy 214.63 161.29))
     (stroke (width 0) (type default) (color 0 0 0 0))
   )
-  (polyline (pts (xy 77.47 86.36) (xy 77.47 101.6))
-    (stroke (width 0) (type default) (color 0 0 0 0))
-  )
   (wire (pts (xy 171.45 81.28) (xy 187.96 81.28))
     (stroke (width 0) (type default) (color 0 0 0 0))
   )
-  (wire (pts (xy 49.53 138.43) (xy 74.93 138.43))
-    (stroke (width 0) (type default) (color 0 0 0 0))
-  )
   (wire (pts (xy 137.16 152.4) (xy 153.67 152.4))
     (stroke (width 0) (type default) (color 0 0 0 0))
@@
     (stroke (width 0) (type default) (color 0 0 0 0))
   )
-  (wire (pts (xy 49.53 85.09) (xy 49.53 87.63))
-    (stroke (width 0) (type default) (color 0 0 0 0))
-  )
   (wire (pts (xy 29.21 80.01) (xy 29.21 78.74))
     (stroke (width 0) (type default) (color 0 0 0 0))
@@
     (stroke (width 0) (type default) (color 0 0 0 0))
   )
-  (wire (pts (xy 49.53 85.09) (xy 74.93 85.09))
-    (stroke (width 0) (type default) (color 0 0 0 0))
-  )
-  (polyline (pts (xy 77.47 101.6) (xy 48.26 101.6))
-    (stroke (width 0) (type default) (color 0 0 0 0))
-  )
-  (polyline (pts (xy 77.47 154.94) (xy 48.26 154.94))
+  (wire (pts (xy 44.45 85.09) (xy 74.93 85.09))
     (stroke (width 0) (type default) (color 0 0 0 0))
   )
@@
     (effects (font (size 1.27 1.27)) (justify left bottom))
   )
-  (text "if no BUFFER is used \n( e.g 74AHC1G125 ) just \nconnect 'UART_TX' here.\n@TODO(DECIDE ON BUFFER)"
-    (at 49.53 152.4 0)
-    (effects (font (size 1.27 1.27)) (justify left bottom))
-  )
   (text "KLST SATELLITES" (at 116.84 53.34 0)
     (effects (font (size 1.27 1.27)) (justify left bottom))
@@
     (effects (font (size 1.27 1.27)) (justify left bottom))
   )
-  (text "if no BUFFER is used \n( e.g 74AHC1G125 ) just \nconnect 'UART_TX' here.\n@TODO(DECIDE ON BUFFER)"
-    (at 49.53 99.06 0)
-    (effects (font (size 1.27 1.27)) (justify left bottom))
-  )
   (text "KLST MAIN" (at 116.84 17.78 0)
     (effects (font (size 1.27 1.27)) (justify left bottom))
   )
-  (text "@NOTE(looking into the plug)" (at 29.21 46.99 0)
+  (text "@NOTE(symbol is *looking* onto cable connector\ne.g PIN4 is on right side, looking into to socket )"
+    (at 15.24 53.34 0)
     (effects (font (size 1.27 1.27)) (justify left bottom))
   )
@@
     (effects (font (size 1.27 1.27)) (justify right bottom))
   )
-  (label "UART_TX" (at 49.53 90.17 0)
-    (effects (font (size 1.27 1.27)) (justify left bottom))
-  )
   (label "UART_TX" (at 171.45 36.83 0)
     (effects (font (size 1.27 1.27)) (justify left bottom))
@@
   (label "UART_RX" (at 151.13 31.75 180)
     (effects (font (size 1.27 1.27)) (justify right bottom))
-  )
-  (label "UART_TX" (at 49.53 143.51 0)
-    (effects (font (size 1.27 1.27)) (justify left bottom))
   )
   (symbol (lib_id "Mechanical:MountingHole_Pad") (at 229.87 43.18 0) (unit 1)
@@
       (effects (font (size 1.27 1.27)) (justify left))
     )
-    (property "Value" "KLST_SHEEP--graphics" (id 1) (at 231.775 22.733 0)
+    (property "Value" "KLST_ICON" (id 1) (at 231.775 22.733 0)
       (effects (font (size 1.27 1.27)) (justify left))
     )
@@
       (effects (font (size 1.27 1.27)) (justify left))
     )
-    (property "Value" "MIDI_OUT" (id 1) (at 30.8611 80.01 0)
+    (property "Value" "MIDI OUT" (id 1) (at 30.8611 80.01 0)
       (effects (font (size 1.27 1.27)) (justify left))
     )
@@
       (effects (font (size 1.27 1.27)) (justify left))
     )
-    (property "Value" "MIDI_IN" (id 1) (at 27.0511 33.02 0)
+    (property "Value" "MIDI IN" (id 1) (at 27.0511 33.02 0)
       (effects (font (size 1.27 1.27)) (justify left))
     )
@@
       (effects (font (size 1.27 1.27)) (justify left))
     )
-    (property "Value" "MIDI_THRU" (id 1) (at 30.8611 133.35 0)
+    (property "Value" "MIDI THRU" (id 1) (at 30.8611 133.35 0)
       (effects (font (size 1.27 1.27)) (justify left))
     )
@@
     )
     (path "/b96aec94-25ef-4764-8e35-cc0574a76f94"
-      (reference "J1") (unit 1) (value "MIDI_IN") (footprint "DIN-5:DIN5-RA-PTH")
+      (reference "J1") (unit 1) (value "MIDI IN") (footprint "DIN-5:DIN5-RA-PTH")
     )
     (path "/86771a88-aa95-4c5b-9d61-c96f546382ac"
-      (reference "J2") (unit 1) (value "MIDI_OUT") (footprint "DIN-5:DIN5-RA-PTH")
+      (reference "J2") (unit 1) (value "MIDI OUT") (footprint "DIN-5:DIN5-RA-PTH")
     )
     (path "/d875e0c9-a433-4a5d-80fd-824539ee071e"
-      (reference "J3") (unit 1) (value "MIDI_THRU") (footprint "DIN-5:DIN5-RA-PTH")
+      (reference "J3") (unit 1) (value "MIDI THRU") (footprint "DIN-5:DIN5-RA-PTH")
     )
     (path "/3fd02374-7d7f-4117-8b30-31486dac145e"
@@
     )
     (path "/20194246-20e6-4817-bebf-2d40fda41fa7"
-      (reference "X1") (unit 1) (value "KLST_SHEEP--graphics") (footprint "DIN-5:KLST--icon")
-    )
-  )
+      (reference "X1") (unit 1) (value "KLST_ICON") (footprint "DIN-5:KLST--icon")
+    )
+  )

Commit message: finalized PCB
Parts:
- C1: MFR.Part # (none) -> T529P106M010AAE200; MPN F380G107MSALZT -> (none)
- D1: MFR.Part # (none) -> 1N914BWT; MPN 1N914BWT -> (none)
- H1, H2, X1: JLCPCB Part # (none) -> -
- J1, J2, J3: MFR.Part # (none) -> DIN-504-M10; MPN FM6725 -> (none)
- J4: MFR.Part # 300R-6P -> B-3000R06P-0110
- R1, R2, R4, R5: MFR.Part # (none) -> AECR0805F47R0K9
- R3: MFR.Part # (none) -> PTFR0805B220RP9
- R6: MFR.Part # (none) -> AECR0805F470RK9
- U1: MFR.Part # (none) -> H11L1SR2M
- U2, U3: MFR.Part # (none) -> SN74AHC1G125DBVR
Changed lines of the file:
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@@
+      (effects (font (size 1.27 1.27)) hide)
+    )
+    (property "JLCPCB Part #" "-" (id 4) (at 229.87 43.18 0)
       (effects (font (size 1.27 1.27)) hide)
     )
@@
       (effects (font (size 2.54 2.54)) hide)
     )
+    (property "JLCPCB Part #" "-" (id 4) (at 231.14 21.59 0)
+      (effects (font (size 1.27 1.27)) hide)
+    )
   )
   (symbol (lib_id "power:+3V3") (at 20.32 71.12 0) (unit 1)
@@
       (effects (font (size 1.27 1.27)) hide)
     )
+    (property "MFR.Part #" "AECR0805F47R0K9" (id 6) (at 20.32 74.93 0)
+      (effects (font (size 1.27 1.27)) hide)
+    )
     (pin "1")
     (pin "2")
@@
       (effects (font (size 1.27 1.27)) hide)
     )
-    (property "MPN" "1N914BWT" (id 4) (at 52.07 33.02 0)
+    (property "MPN" "" (id 4) (at 52.07 33.02 0)
       (effects (font (size 1.27 1.27)) hide)
     )
@@
     )
     (property "JLCPCB Part #" "C896167" (id 6) (at 52.07 33.02 0)
+      (effects (font (size 1.27 1.27)) hide)
+    )
+    (property "MFR.Part #" "1N914BWT" (id 7) (at 52.07 33.02 0)
       (effects (font (size 1.27 1.27)) hide)
     )
@@
       (effects (font (size 1.27 1.27)) hide)
     )
-    (property "MFR.Part #" "300R-6P" (id 4) (at 162.56 34.29 0)
+    (property "MFR.Part #" "B-3000R06P-0110" (id 4) (at 162.56 34.29 0)
       (effects (font (size 1.27 1.27)) hide)
     )
@@
       (effects (font (size 1.27 1.27)) hide)
     )
+    (property "MFR.Part #" "AECR0805F47R0K9" (id 6) (at 20.32 128.27 0)
+      (effects (font (size 1.27 1.27)) hide)
+    )
     (pin "1")
     (pin "2")
@@
       (effects (font (size 1.27 1.27)) hide)
     )
+    (property "MFR.Part #" "SN74AHC1G125DBVR" (id 6) (at 81.28 85.09 0)
+      (effects (font (size 1.27 1.27)) hide)
+    )
     (pin "1")
     (pin "2")
@@
       (effects (font (size 1.27 1.27)) hide)
     )
-    (property "MPN" "FM6725" (id 4) (at 29.21 87.63 0)
+    (property "MPN" "" (id 4) (at 29.21 87.63 0)
       (effects (font (size 1.27 1.27)) hide)
     )
@@
     )
     (property "JLCPCB Part #" "C2939344" (id 6) (at 29.21 87.63 0)
+      (effects (font (size 1.27 1.27)) hide)
+    )
+    (property "MFR.Part #" "DIN-504-M10" (id 7) (at 29.21 87.63 0)
       (effects (font (size 1.27 1.27)) hide)
     )
@@
     )
     (property "Extended Part" "-" (id 5) (at 67.31 35.56 0)
+      (effects (font (size 1.27 1.27)) hide)
+    )
+    (property "MFR.Part #" "H11L1SR2M" (id 6) (at 67.31 35.56 0)
       (effects (font (size 1.27 1.27)) hide)
     )
@@
       (effects (font (size 1.27 1.27)) hide)
     )
+    (property "MFR.Part #" "SN74AHC1G125DBVR" (id 6) (at 81.28 138.43 0)
+      (effects (font (size 1.27 1.27)) hide)
+    )
     (pin "1")
     (pin "2")
@@
       (effects (font (size 1.27 1.27)) hide)
     )
-    (property "MPN" "FM6725" (id 4) (at 25.4 40.64 0)
+    (property "MPN" "" (id 4) (at 25.4 40.64 0)
       (effects (font (size 1.27 1.27)) hide)
     )
@@
     )
     (property "JLCPCB Part #" "C2939344" (id 6) (at 25.4 40.64 0)
+      (effects (font (size 1.27 1.27)) hide)
+    )
+    (property "MFR.Part #" "DIN-504-M10" (id 7) (at 25.4 40.64 0)
       (effects (font (size 1.27 1.27)) hide)
     )
@@
       (effects (font (size 1.27 1.27)) hide)
     )
+    (property "MFR.Part #" "AECR0805F47R0K9" (id 6) (at 41.91 138.43 0)
+      (effects (font (size 1.27 1.27)) hide)
+    )
     (pin "1")
     (pin "2")
@@
       (effects (font (size 1.27 1.27)) hide)
     )
+    (property "MFR.Part #" "PTFR0805B220RP9" (id 6) (at 40.64 27.94 0)
+      (effects (font (size 1.27 1.27)) hide)
+    )
     (pin "1")
     (pin "2")
@@
       (effects (font (size 1.27 1.27)) hide)
     )
-    (property "MPN" "F380G107MSALZT" (id 4) (at 99.06 34.29 0)
+    (property "MPN" "" (id 4) (at 99.06 34.29 0)
       (effects (font (size 1.27 1.27)) hide)
     )
@@
       (effects (font (size 1.27 1.27)) hide)
     )
+    (property "MFR.Part #" "T529P106M010AAE200" (id 7) (at 99.06 34.29 0)
+      (effects (font (size 1.27 1.27)) hide)
+    )
     (pin "1")
     (pin "2")
@@
     )
     (property "Datasheet" "~" (id 3) (at 229.87 35.56 0)
+      (effects (font (size 1.27 1.27)) hide)
+    )
+    (property "JLCPCB Part #" "-" (id 4) (at 229.87 35.56 0)
       (effects (font (size 1.27 1.27)) hide)
     )
@@
       (effects (font (size 1.27 1.27)) hide)
     )
-    (property "MPN" "FM6725" (id 4) (at 29.21 140.97 0)
+    (property "MPN" "" (id 4) (at 29.21 140.97 0)
       (effects (font (size 1.27 1.27)) hide)
     )
@@
     )
     (property "JLCPCB Part #" "C2939344" (id 6) (at 29.21 140.97 0)
+      (effects (font (size 1.27 1.27)) hide)
+    )
+    (property "MFR.Part #" "DIN-504-M10" (id 7) (at 29.21 140.97 0)
       (effects (font (size 1.27 1.27)) hide)
     )
@@
       (effects (font (size 1.27 1.27)) hide)
     )
+    (property "MFR.Part #" "AECR0805F470RK9" (id 6) (at 77.47 30.48 0)
+      (effects (font (size 1.27 1.27)) hide)
+    )
     (pin "1")
     (pin "2")
@@
     )
     (property "JLCPCB Part #" "C328398" (id 5) (at 41.91 85.09 0)
+      (effects (font (size 1.27 1.27)) hide)
+    )
+    (property "MFR.Part #" "AECR0805F47R0K9" (id 6) (at 41.91 85.09 0)
       (effects (font (size 1.27 1.27)) hide)
     )
@@
     )
     (path "/d8e2a12b-31be-47f1-8115-76d754dc9bd2/56b7259e-6208-4e67-ad75-da378c45e298"
-      (reference "D2") (unit 1) (value "Schottky") (footprint "Diode_SMD:D_SOD-123")
+      (reference "D2") (unit 1) (value "Schottky") (footprint "")
     )
     (path "/f3531ba1-f7e9-41d2-a32e-05e17fbdb6b6/56b7259e-6208-4e67-ad75-da378c45e298"
-      (reference "D3") (unit 1) (value "Schottky") (footprint "Diode_SMD:D_SOD-123")
+      (reference "D3") (unit 1) (value "Schottky") (footprint "")
     )
     (path "/27ca45b9-c275-4628-856d-ae0261f758e0/56b7259e-6208-4e67-ad75-da378c45e298"
-      (reference "D4") (unit 1) (value "Schottky") (footprint "Diode_SMD:D_SOD-123")
+      (reference "D4") (unit 1) (value "Schottky") (footprint "")
     )
     (path "/a1718a90-de27-4640-8a78-6c2834ef780e/56b7259e-6208-4e67-ad75-da378c45e298"
-      (reference "D5") (unit 1) (value "Schottky") (footprint "Diode_SMD:D_SOD-123")
+      (reference "D5") (unit 1) (value "Schottky") (footprint "")
     )
     (path "/c7cce935-268b-4ca7-bcc6-d4c3407696e4/56b7259e-6208-4e67-ad75-da378c45e298"
-      (reference "D6") (unit 1) (value "Schottky") (footprint "Diode_SMD:D_SOD-123")
+      (reference "D6") (unit 1) (value "Schottky") (footprint "")
     )
     (path "/739ea1f8-cdea-420a-8d3a-4b30fb9859c1/56b7259e-6208-4e67-ad75-da378c45e298"
-      (reference "D7") (unit 1) (value "Schottky") (footprint "Diode_SMD:D_SOD-123")
+      (reference "D7") (unit 1) (value "Schottky") (footprint "")
     )
     (path "/12e2e5c2-f4b0-4246-b746-b5954e2505f0/56b7259e-6208-4e67-ad75-da378c45e298"
-      (reference "D8") (unit 1) (value "Schottky") (footprint "Diode_SMD:D_SOD-123")
+      (reference "D8") (unit 1) (value "Schottky") (footprint "")
     )
     (path "/9ff9e472-5d9b-4cd1-ae9f-d409e958cd01/56b7259e-6208-4e67-ad75-da378c45e298"
-      (reference "D9") (unit 1) (value "Schottky") (footprint "Diode_SMD:D_SOD-123")
+      (reference "D9") (unit 1) (value "Schottky") (footprint "")
     )
     (path "/feed83e7-fe35-45c3-b938-143fa9d139d9/56b7259e-6208-4e67-ad75-da378c45e298"
-      (reference "D10") (unit 1) (value "Schottky") (footprint "Diode_SMD:D_SOD-123")
+      (reference "D10") (unit 1) (value "Schottky") (footprint "")
     )
     (path "/ce631169-40e5-44ad-95a8-46fd5f8c17a5"

Commit message: updated LCSC #
Parts:
- C1: LCSC Part # (none) -> C696821
- D1: LCSC Part # (none) -> C896167
- J1, J2, J3: LCSC Part # (none) -> C2939344
- J4: LCSC Part # (none) -> C146629
- R1, R2, R4, R5: LCSC Part # (none) -> C328398
- R3: LCSC Part # (none) -> C479094
- R6: LCSC Part # (none) -> C328396
- U1: LCSC Part # (none) -> C20082
- U2, U3: LCSC Part # (none) -> C7468
Changed lines of the file:
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@@
+      (effects (font (size 1.27 1.27)) hide)
+    )
+    (property "LCSC Part #" "C328398" (id 7) (at 20.32 74.93 0)
       (effects (font (size 1.27 1.27)) hide)
     )
@@
     )
     (property "MFR.Part #" "1N914BWT" (id 7) (at 52.07 33.02 0)
+      (effects (font (size 1.27 1.27)) hide)
+    )
+    (property "LCSC Part #" "C896167" (id 8) (at 52.07 33.02 0)
       (effects (font (size 1.27 1.27)) hide)
     )
@@
       (effects (font (size 1.27 1.27)) hide)
     )
-    (property "LCSC Part #" "" (id 5) (at 162.56 34.29 0)
+    (property "LCSC Part #" "C146629" (id 5) (at 162.56 34.29 0)
       (effects (font (size 1.27 1.27)) hide)
     )
@@
       (effects (font (size 1.27 1.27)) hide)
     )
+    (property "LCSC Part #" "C328398" (id 7) (at 20.32 128.27 0)
+      (effects (font (size 1.27 1.27)) hide)
+    )
     (pin "1")
     (pin "2")
@@
       (effects (font (size 1.27 1.27)) hide)
     )
+    (property "LCSC Part #" "C7468" (id 7) (at 81.28 85.09 0)
+      (effects (font (size 1.27 1.27)) hide)
+    )
     (pin "1")
     (pin "2")
@@
       (effects (font (size 1.27 1.27)) hide)
     )
+    (property "LCSC Part #" "C2939344" (id 8) (at 29.21 87.63 0)
+      (effects (font (size 1.27 1.27)) hide)
+    )
     (pin "6")
     (pin "7")
@@
     )
     (property "MFR.Part #" "H11L1SR2M" (id 6) (at 67.31 35.56 0)
+      (effects (font (size 1.27 1.27)) hide)
+    )
+    (property "LCSC Part #" "C20082" (id 7) (at 67.31 35.56 0)
       (effects (font (size 1.27 1.27)) hide)
     )
@@
       (effects (font (size 1.27 1.27)) hide)
     )
+    (property "LCSC Part #" "C7468" (id 7) (at 81.28 138.43 0)
+      (effects (font (size 1.27 1.27)) hide)
+    )
     (pin "1")
     (pin "2")
@@
       (effects (font (size 1.27 1.27)) hide)
     )
+    (property "LCSC Part #" "C2939344" (id 8) (at 25.4 40.64 0)
+      (effects (font (size 1.27 1.27)) hide)
+    )
     (pin "6")
     (pin "7")
@@
       (effects (font (size 1.27 1.27)) hide)
     )
+    (property "LCSC Part #" "C328398" (id 7) (at 41.91 138.43 0)
+      (effects (font (size 1.27 1.27)) hide)
+    )
     (pin "1")
     (pin "2")
@@
       (effects (font (size 1.27 1.27)) hide)
     )
+    (property "LCSC Part #" "C479094" (id 7) (at 40.64 27.94 0)
+      (effects (font (size 1.27 1.27)) hide)
+    )
     (pin "1")
     (pin "2")
@@
     )
     (property "MFR.Part #" "T529P106M010AAE200" (id 7) (at 99.06 34.29 0)
+      (effects (font (size 1.27 1.27)) hide)
+    )
+    (property "LCSC Part #" "C696821" (id 8) (at 99.06 34.29 0)
       (effects (font (size 1.27 1.27)) hide)
     )
@@
     )
     (property "MFR.Part #" "DIN-504-M10" (id 7) (at 29.21 140.97 0)
+      (effects (font (size 1.27 1.27)) hide)
+    )
+    (property "LCSC Part #" "C2939344" (id 8) (at 29.21 140.97 0)
       (effects (font (size 1.27 1.27)) hide)
     )
@@
       (effects (font (size 1.27 1.27)) hide)
     )
+    (property "LCSC Part #" "C328396" (id 7) (at 77.47 30.48 0)
+      (effects (font (size 1.27 1.27)) hide)
+    )
     (pin "1")
     (pin "2")
@@
       (effects (font (size 1.27 1.27)) hide)
     )
+    (property "LCSC Part #" "C328398" (id 7) (at 41.91 85.09 0)
+      (effects (font (size 1.27 1.27)) hide)
+    )
