File: KLST_PANDA/USB.kicad_sch (KiCad schematic)
At the start: 11 parts, among them J16 DEVICE+CHARGE(UFP), J17 HOST(DFP)

Commit message: cleaned up main sheet
Parts:
- added R74, R75, R76, R77: 0R, symbol Device:R_Small
Connections:
- net _USB_DEVICE_HOST_MINUS: now also R74.2, R77.1; no longer D11.3 (K), J16.A7 (D-), J16.B7 (D-), J17.A7 (D-), J17.B7 (D-)
- net _USB_DEVICE_HOST_PLUS: now also R75.1, R76.2; no longer D11.4 (K), J16.A6 (D+), J16.B6 (D+), J17.A6 (D+), J17.B6 (D+)
- new net: D11.4 (K), J16.A6 (D+), J16.B6 (D+), R76.1
- new net: J17.A6 (D+), J17.B6 (D+), R75.2
- new net: D11.3 (K), J16.A7 (D-), J16.B7 (D-), R77.2
- new net: J17.A7 (D-), J17.B7 (D-), R74.1
Other:
- note added: "@TODO( are 22R necessary?! )"
- note added: "DEVICE+CHARGE"
- note added: "HOST"
- note removed: "Rd: pull-down resistor ( fixed at 5.1K )"
- note removed: "Rp: pull-up resisitor ( 56K to VBUS(5V) for default USB power )"
- moved on the sheet: C62, D11, D12, F1, F2, J16, J17, R67, R70, R72, R73

Commit message: improved GPIO, updated schematics
Parts:
- renumbered C62 to C71, J16 to J12, J17 to J13, R70 to R68, R77 to R69, R76 to R70, R74 to R71, R75 to R72, R72 to R73, R73 to R74
Changed lines of the file:
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@@
   (symbol (lib_id "Device:R_Small") (at 116.84 99.06 270) (unit 1)
     (in_bom yes) (on_board yes) (dnp no)
-    (property "Reference" "R76" (at 116.84 104.14 90)
+    (property "Reference" "R70" (at 116.84 104.14 90)
       (effects (font (size 1.27 1.27)))
     )
@@
       (project "KLST_PANDA"
         (path "/b4513875-4c57-4720-bcc5-43ead67fe18f/c1368b5a-3c14-4f80-b962-228aee9202ba"
-          (reference "R76") (unit 1)
+          (reference "R70") (unit 1)
         )
       )
@@
   (symbol (lib_id "Device:R_Small") (at 227.33 81.28 180) (unit 1)
     (in_bom yes) (on_board yes) (dnp no)
-    (property "Reference" "R73" (at 229.87 80.645 0)
+    (property "Reference" "R74" (at 229.87 80.645 0)
       (effects (font (size 1.27 1.27)) (justify right))
     )
@@
       (project "KLST_PANDA"
         (path "/b4513875-4c57-4720-bcc5-43ead67fe18f/c1368b5a-3c14-4f80-b962-228aee9202ba"
-          (reference "R73") (unit 1)
+          (reference "R74") (unit 1)
         )
       )
@@
   (symbol (lib_id "Device:R_Small") (at 205.74 99.06 270) (unit 1)
     (in_bom yes) (on_board yes) (dnp no)
-    (property "Reference" "R75" (at 205.74 104.14 90)
+    (property "Reference" "R72" (at 205.74 104.14 90)
       (effects (font (size 1.27 1.27)))
     )
@@
       (project "KLST_PANDA"
         (path "/b4513875-4c57-4720-bcc5-43ead67fe18f/c1368b5a-3c14-4f80-b962-228aee9202ba"
-          (reference "R75") (unit 1)
+          (reference "R72") (unit 1)
         )
       )
@@
   (symbol (lib_id "Device:R_Small") (at 116.84 96.52 90) (unit 1)
     (in_bom yes) (on_board yes) (dnp no)
-    (property "Reference" "R77" (at 116.84 91.44 90)
+    (property "Reference" "R69" (at 116.84 91.44 90)
       (effects (font (size 1.27 1.27)))
     )
@@
       (project "KLST_PANDA"
         (path "/b4513875-4c57-4720-bcc5-43ead67fe18f/c1368b5a-3c14-4f80-b962-228aee9202ba"
-          (reference "R77") (unit 1)
+          (reference "R69") (unit 1)
         )
       )
@@
   (symbol (lib_id "Device:R_Small") (at 83.82 114.3 180) (unit 1)
     (in_bom yes) (on_board yes) (dnp no)
-    (property "Reference" "R70" (at 86.36 113.665 0)
+    (property "Reference" "R68" (at 86.36 113.665 0)
       (effects (font (size 1.27 1.27)) (justify right))
     )
@@
       (project "KLST_PANDA"
         (path "/b4513875-4c57-4720-bcc5-43ead67fe18f/c1368b5a-3c14-4f80-b962-228aee9202ba"
-          (reference "R70") (unit 1)
+          (reference "R68") (unit 1)
         )
       )
@@
   (symbol (lib_id "Connector:USB_C_Receptacle_USB2.0") (at 146.05 96.52 0) (mirror y) (unit 1)
     (in_bom yes) (on_board yes) (dnp no)
-    (property "Reference" "J16" (at 146.05 74.93 0)
+    (property "Reference" "J12" (at 146.05 74.93 0)
       (effects (font (size 1.27 1.27)))
     )
@@
       (project "KLST_PANDA"
         (path "/b4513875-4c57-4720-bcc5-43ead67fe18f/c1368b5a-3c14-4f80-b962-228aee9202ba"
-          (reference "J16") (unit 1)
+          (reference "J12") (unit 1)
         )
       )
@@
   (symbol (lib_id "Device:R_Small") (at 205.74 96.52 90) (unit 1)
     (in_bom yes) (on_board yes) (dnp no) (fields_autoplaced)
-    (property "Reference" "R74" (at 205.74 91.44 90)
+    (property "Reference" "R71" (at 205.74 91.44 90)
       (effects (font (size 1.27 1.27)))
     )
@@
       (project "KLST_PANDA"
         (path "/b4513875-4c57-4720-bcc5-43ead67fe18f/c1368b5a-3c14-4f80-b962-228aee9202ba"
-          (reference "R74") (unit 1)
+          (reference "R71") (unit 1)
         )
       )
@@
         )
         (path "/b4513875-4c57-4720-bcc5-43ead67fe18f/c1368b5a-3c14-4f80-b962-228aee9202ba"
-          (reference "#PWR050") (unit 1)
+          (reference "#PWR084") (unit 1)
         )
       )
@@
         )
         (path "/b4513875-4c57-4720-bcc5-43ead67fe18f/c1368b5a-3c14-4f80-b962-228aee9202ba"
-          (reference "#PWR022") (unit 1)
+          (reference "#PWR085") (unit 1)
         )
       )
@@
   (symbol (lib_id "Device:R_Small") (at 224.79 81.28 0) (mirror x) (unit 1)
     (in_bom yes) (on_board yes) (dnp no)
-    (property "Reference" "R72" (at 222.25 80.645 0)
+    (property "Reference" "R73" (at 222.25 80.645 0)
       (effects (font (size 1.27 1.27)) (justify right))
     )
@@
       (project "KLST_PANDA"
         (path "/b4513875-4c57-4720-bcc5-43ead67fe18f/c1368b5a-3c14-4f80-b962-228aee9202ba"
-          (reference "R72") (unit 1)
+          (reference "R73") (unit 1)
         )
       )
@@
   (symbol (lib_id "Connector:USB_C_Receptacle_USB2.0") (at 179.07 96.52 0) (unit 1)
     (in_bom yes) (on_board yes) (dnp no) (fields_autoplaced)
-    (property "Reference" "J17" (at 179.07 74.93 0)
+    (property "Reference" "J13" (at 179.07 74.93 0)
       (effects (font (size 1.27 1.27)))
     )
@@
       (project "KLST_PANDA"
         (path "/b4513875-4c57-4720-bcc5-43ead67fe18f/c1368b5a-3c14-4f80-b962-228aee9202ba"
-          (reference "J17") (unit 1)
+          (reference "J13") (unit 1)
         )
       )
@@
   (symbol (lib_id "Device:C_Small") (at 73.66 95.25 0) (unit 1)
     (in_bom yes) (on_board yes) (dnp no)
-    (property "Reference" "C62" (at 71.12 94.6213 0)
+    (property "Reference" "C71" (at 71.12 94.6213 0)
       (effects (font (size 1.27 1.27)) (justify right))
     )
@@
       (project "KLST_PANDA"
         (path "/b4513875-4c57-4720-bcc5-43ead67fe18f/c1368b5a-3c14-4f80-b962-228aee9202ba"
-          (reference "C62") (unit 1)
+          (reference "C71") (unit 1)
         )
       )
@@
         )
         (path "/b4513875-4c57-4720-bcc5-43ead67fe18f/c1368b5a-3c14-4f80-b962-228aee9202ba"
-          (reference "#PWR042") (unit 1)
-        )
-      )
+          (reference "#PWR083") (unit 1)
+        )
+      )

Commit message: added mechanical keys, updated audio jacks, minor changes
Other:
- note added: "@TODO(replace with proper footprint)"
Changed lines of the file:
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@@
     (effects (font (size 1.27 1.27)) (justify right bottom))
+  )
+  (text "@TODO(replace with proper footprint)" (at 146.685 70.485 0)
+    (effects (font (size 1.27 1.27)) (justify left bottom))
   )
   (text "e.g\nJLCPCB Part # :: C3040626\nPackage :: SOT-143" (at 237.49 116.84 0)

Commit message: moved core (MCU) to sheet, cleaned up sheets
Parts:
- renumbered C71 to C68, J12 to J11, J13 to J12, R67 to R56, R68 to R57, R69 to R58, R70 to R59, R71 to R60, R72 to R61, R73 to R62, R74 to R63
Other:
- moved on the sheet: C68, D11, D12, F1, F2, J11, J12, R56, R57, R58, R59, R60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

Commit message: added battery clip, updated to new KiCad version
Parts:
- renumbered J11 to J13, J12 to J14
Changed lines of the file:
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@@
   (symbol (lib_id "Connector:USB_C_Receptacle_USB2.0") (at 127 55.88 0) (mirror y) (unit 1)
     (in_bom yes) (on_board yes) (dnp no)
-    (property "Reference" "J11" (at 127 34.29 0)
+    (property "Reference" "J13" (at 127 34.29 0)
       (effects (font (size 1.27 1.27)))
     )
@@
       (project "KLST_PANDA"
         (path "/b4513875-4c57-4720-bcc5-43ead67fe18f/c1368b5a-3c14-4f80-b962-228aee9202ba"
-          (reference "J11") (unit 1)
+          (reference "J13") (unit 1)
         )
       )
@@
   (symbol (lib_id "Connector:USB_C_Receptacle_USB2.0") (at 160.02 55.88 0) (unit 1)
     (in_bom yes) (on_board yes) (dnp no) (fields_autoplaced)
-    (property "Reference" "J12" (at 160.02 34.29 0)
+    (property "Reference" "J14" (at 160.02 34.29 0)
       (effects (font (size 1.27 1.27)))
     )
@@
       (project "KLST_PANDA"
         (path "/b4513875-4c57-4720-bcc5-43ead67fe18f/c1368b5a-3c14-4f80-b962-228aee9202ba"
-          (reference "J12") (unit 1)
-        )
-      )
+          (reference "J14") (unit 1)
+        )
+      )

Commit message: removed DRC warnings and error, added power page
Parts:
- renumbered C68 to C44, J14 to J10, J13 to J9, R56 to R42, R57 to R43, R58 to R44, R59 to R45, R60 to R46, R61 to R47, R62 to R48, R63 to R49

Commit message: changed I2C label, display can now be switched on and off
Parts:
- renumbered D11 to D12, D12 to D13
Changed lines of the file:
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@@
+    (stroke (width 0) (type default))
+  )
+  (wire (pts (xy 54.61 40.64) (xy 101.6 40.64))
     (stroke (width 0) (type default))
   )
@@
     (stroke (width 0) (type default))
   )
+  (wire (pts (xy 208.28 48.26) (xy 208.28 43.18))
+    (stroke (width 0) (type default))
+  )
+  (wire (pts (xy 198.12 55.88) (xy 207.01 55.88))
+    (stroke (width 0) (type default))
+  )
+  (wire (pts (xy 175.26 53.34) (xy 176.53 53.34))
+    (stroke (width 0) (type default))
+  )
+  (wire (pts (xy 160.02 80.01) (xy 160.02 78.74))
+    (stroke (width 0) (type default))
+  )
+  (wire (pts (xy 156.21 81.28) (xy 156.21 80.01))
+    (stroke (width 0) (type default))
+  )
+  (wire (pts (xy 111.76 55.88) (xy 110.49 55.88))
+    (stroke (width 0) (type default))
+  )
+  (wire (pts (xy 64.77 76.2) (xy 64.77 80.01))
+    (stroke (width 0) (type default))
+  )
+  (wire (pts (xy 106.68 58.42) (xy 106.68 67.31))
+    (stroke (width 0) (type default))
+  )
+  (wire (pts (xy 156.21 80.01) (xy 160.02 80.01))
+    (stroke (width 0) (type default))
+  )
+  (wire (pts (xy 62.23 80.01) (xy 64.77 80.01))
+    (stroke (width 0) (type default))
+  )
+  (wire (pts (xy 101.6 40.64) (xy 111.76 40.64))
+    (stroke (width 0) (type default))
+  )
+  (wire (pts (xy 111.76 53.34) (xy 110.49 53.34))
+    (stroke (width 0) (type default))
+  )
+  (wire (pts (xy 198.12 55.88) (xy 198.12 67.31))
+    (stroke (width 0) (type default))
+  )
+  (wire (pts (xy 95.25 58.42) (xy 92.71 58.42))
+    (stroke (width 0) (type default))
+  )
+  (wire (pts (xy 134.62 78.74) (xy 134.62 80.01))
+    (stroke (width 0) (type default))
+  )
+  (wire (pts (xy 176.53 53.34) (xy 176.53 55.88))
+    (stroke (width 0) (type default))
+  )
+  (wire (pts (xy 205.74 34.29) (xy 201.93 34.29))
+    (stroke (width 0) (type default))
+  )
+  (wire (pts (xy 95.25 55.88) (xy 92.71 55.88))
+    (stroke (width 0) (type default))
+  )
+  (wire (pts (xy 110.49 53.34) (xy 110.49 55.88))
+    (stroke (width 0) (type default))
+  )
+  (wire (pts (xy 104.14 80.01) (xy 127 80.01))
+    (stroke (width 0) (type default))
+  )
+  (wire (pts (xy 175.26 60.96) (xy 176.53 60.96))
+    (stroke (width 0) (type default))
+  )
+  (wire (pts (xy 186.69 40.64) (xy 195.58 40.64))
+    (stroke (width 0) (type default))
+  )
   (wire (pts (xy 44.45 40.64) (xy 46.99 40.64))
-    (stroke (width 0) (type default))
-  )
-  (wire (pts (xy 208.28 48.26) (xy 208.28 43.18))
-    (stroke (width 0) (type default))
-  )
-  (wire (pts (xy 198.12 55.88) (xy 207.01 55.88))
-    (stroke (width 0) (type default))
-  )
-  (wire (pts (xy 175.26 53.34) (xy 176.53 53.34))
-    (stroke (width 0) (type default))
-  )
-  (wire (pts (xy 160.02 80.01) (xy 160.02 78.74))
-    (stroke (width 0) (type default))
-  )
-  (wire (pts (xy 156.21 81.28) (xy 156.21 80.01))
-    (stroke (width 0) (type default))
-  )
-  (wire (pts (xy 111.76 55.88) (xy 110.49 55.88))
-    (stroke (width 0) (type default))
-  )
-  (wire (pts (xy 64.77 76.2) (xy 64.77 80.01))
-    (stroke (width 0) (type default))
-  )
-  (wire (pts (xy 106.68 58.42) (xy 106.68 67.31))
-    (stroke (width 0) (type default))
-  )
-  (wire (pts (xy 156.21 80.01) (xy 160.02 80.01))
-    (stroke (width 0) (type default))
-  )
-  (wire (pts (xy 54.61 40.64) (xy 101.6 40.64))
-    (stroke (width 0) (type default))
-  )
-  (wire (pts (xy 62.23 80.01) (xy 64.77 80.01))
-    (stroke (width 0) (type default))
-  )
-  (wire (pts (xy 101.6 40.64) (xy 111.76 40.64))
-    (stroke (width 0) (type default))
-  )
-  (wire (pts (xy 111.76 53.34) (xy 110.49 53.34))
-    (stroke (width 0) (type default))
-  )
-  (wire (pts (xy 198.12 55.88) (xy 198.12 67.31))
-    (stroke (width 0) (type default))
-  )
-  (wire (pts (xy 95.25 58.42) (xy 92.71 58.42))
-    (stroke (width 0) (type default))
-  )
-  (wire (pts (xy 134.62 78.74) (xy 134.62 80.01))
-    (stroke (width 0) (type default))
-  )
-  (wire (pts (xy 176.53 53.34) (xy 176.53 55.88))
-    (stroke (width 0) (type default))
-  )
-  (wire (pts (xy 205.74 34.29) (xy 201.93 34.29))
-    (stroke (width 0) (type default))
-  )
-  (wire (pts (xy 95.25 55.88) (xy 92.71 55.88))
-    (stroke (width 0) (type default))
-  )
-  (wire (pts (xy 110.49 53.34) (xy 110.49 55.88))
-    (stroke (width 0) (type default))
-  )
-  (wire (pts (xy 104.14 80.01) (xy 127 80.01))
-    (stroke (width 0) (type default))
-  )
-  (wire (pts (xy 175.26 60.96) (xy 176.53 60.96))
-    (stroke (width 0) (type default))
-  )
-  (wire (pts (xy 186.69 40.64) (xy 195.58 40.64))
     (stroke (width 0) (type default))
   )
@@
   (symbol (lib_id "Power_Protection:SP0503BAHT") (at 198.12 72.39 0) (mirror y) (unit 1)
     (in_bom yes) (on_board yes) (dnp no)
-    (property "Reference" "D12" (at 204.47 71.755 0)
+    (property "Reference" "D13" (at 204.47 71.755 0)
       (effects (font (size 1.27 1.27)) (justify right))
     )
@@
       (project "KLST_PANDA"
         (path "/b4513875-4c57-4720-bcc5-43ead67fe18f/c1368b5a-3c14-4f80-b962-228aee9202ba"
-          (reference "D12") (unit 1)
+          (reference "D13") (unit 1)
         )
       )
@@
         )
         (path "/b4513875-4c57-4720-bcc5-43ead67fe18f/c1368b5a-3c14-4f80-b962-228aee9202ba"
-          (reference "#PWR071") (unit 1)
+          (reference "#PWR070") (unit 1)
         )
       )
@@
         )
         (path "/b4513875-4c57-4720-bcc5-43ead67fe18f/c1368b5a-3c14-4f80-b962-228aee9202ba"
-          (reference "#PWR072") (unit 1)
+          (reference "#PWR071") (unit 1)
         )
       )
@@
   (symbol (lib_id "Power_Protection:SP0503BAHT") (at 104.14 72.39 0) (unit 1)
     (in_bom yes) (on_board yes) (dnp no)
-    (property "Reference" "D11" (at 97.79 71.755 0)
+    (property "Reference" "D12" (at 97.79 71.755 0)
       (effects (font (size 1.27 1.27)) (justify right))
     )
@@
       (project "KLST_PANDA"
         (path "/b4513875-4c57-4720-bcc5-43ead67fe18f/c1368b5a-3c14-4f80-b962-228aee9202ba"
-          (reference "D11") (unit 1)
+          (reference "D12") (unit 1)
         )
       )
@@
         )
         (path "/b4513875-4c57-4720-bcc5-43ead67fe18f/c1368b5a-3c14-4f80-b962-228aee9202ba"
-          (reference "#PWR070") (unit 1)
-        )
-      )
+          (reference "#PWR069") (unit 1)
+        )
+      )
