File: KLST_PANDA/audio_codec.kicad_sch (KiCad schematic)
At the start: 43 parts, among them J16 MIC_IN, J17 LINE_IN, J18 HEADPHONE_OUT+MIC, J19 LINE_OUT, U12 WM8904CGEFL/V

Commit message: assigned footprints
Parts:
- R18, R19, R20, R23: footprint (none) -> Resistor_SMD:R_0603_1608Metric; JLCPCB (none) -> C417107
- R21, R22: footprint (none) -> Resistor_SMD:R_0603_1608Metric; JLCPCB (none) -> C101304
- R24, R25: footprint Resistor_SMD:R_0805_2012Metric_Pad1.20x1.40mm_HandSolder -> Resistor_SMD:R_0603_1608Metric; JLCPCB C103914 -> C2924143
- R28, R29, R30, R31: footprint (none) -> Resistor_SMD:R_0603_1608Metric; JLCPCB (none) -> C544033
Changed lines of the file:
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@@
       (effects (font (size 1.27 1.27)) (justify left))
     )
-    (property "Footprint" "" (at 331.47 90.17 0)
+    (property "Footprint" "Resistor_SMD:R_0603_1608Metric" (at 331.47 90.17 0)
       (effects (font (size 1.27 1.27)) hide)
     )
     (property "Datasheet" "~" (at 331.47 90.17 0)
+      (effects (font (size 1.27 1.27)) hide)
+    )
+    (property "Description" "250mW" (at 331.47 90.17 0)
+      (effects (font (size 1.27 1.27)) hide)
+    )
+    (property "JLCPCB" "C544033" (at 331.47 90.17 0)
       (effects (font (size 1.27 1.27)) hide)
     )
@@
       (effects (font (size 1.27 1.27)) (justify left))
     )
-    (property "Footprint" "" (at 86.36 33.02 0)
+    (property "Footprint" "Resistor_SMD:R_0603_1608Metric" (at 86.36 33.02 0)
       (effects (font (size 1.27 1.27)) hide)
     )
     (property "Datasheet" "~" (at 86.36 33.02 0)
+      (effects (font (size 1.27 1.27)) hide)
+    )
+    (property "Description" "100mW" (at 86.36 33.02 0)
+      (effects (font (size 1.27 1.27)) hide)
+    )
+    (property "JLCPCB" "C101304" (at 86.36 33.02 0)
       (effects (font (size 1.27 1.27)) hide)
     )
@@
       (effects (font (size 1.27 1.27)) (justify left))
     )
-    (property "Footprint" "" (at 306.07 90.17 0)
+    (property "Footprint" "Resistor_SMD:R_0603_1608Metric" (at 306.07 90.17 0)
       (effects (font (size 1.27 1.27)) hide)
     )
@@
       (effects (font (size 1.27 1.27)) hide)
     )
+    (property "Description" "250mW" (at 306.07 90.17 0)
+      (effects (font (size 1.27 1.27)) hide)
+    )
+    (property "JLCPCB" "C544033" (at 306.07 90.17 0)
+      (effects (font (size 1.27 1.27)) hide)
+    )
     (pin "1")
     (pin "2")
@@
       (effects (font (size 1.27 1.27)) (justify left))
     )
-    (property "Footprint" "" (at 318.77 90.17 0)
+    (property "Footprint" "Resistor_SMD:R_0603_1608Metric" (at 318.77 90.17 0)
       (effects (font (size 1.27 1.27)) hide)
     )
     (property "Datasheet" "~" (at 318.77 90.17 0)
+      (effects (font (size 1.27 1.27)) hide)
+    )
+    (property "Description" "250mW" (at 318.77 90.17 0)
+      (effects (font (size 1.27 1.27)) hide)
+    )
+    (property "JLCPCB" "C544033" (at 318.77 90.17 0)
       (effects (font (size 1.27 1.27)) hide)
     )
@@
       (effects (font (size 1.27 1.27)) (justify left))
     )
-    (property "Footprint" "" (at 64.77 100.33 0)
+    (property "Footprint" "Resistor_SMD:R_0603_1608Metric" (at 64.77 100.33 0)
       (effects (font (size 1.27 1.27)) hide)
     )
     (property "Datasheet" "~" (at 64.77 100.33 0)
+      (effects (font (size 1.27 1.27)) hide)
+    )
+    (property "Description" "100mW" (at 64.77 100.33 0)
+      (effects (font (size 1.27 1.27)) hide)
+    )
+    (property "JLCPCB" "C417107" (at 64.77 100.33 0)
       (effects (font (size 1.27 1.27)) hide)
     )
@@
       (effects (font (size 1.27 1.27)))
     )
-    (property "Footprint" "" (at 50.8 83.82 0)
+    (property "Footprint" "Resistor_SMD:R_0603_1608Metric" (at 50.8 83.82 0)
       (effects (font (size 1.27 1.27)) hide)
     )
     (property "Datasheet" "~" (at 50.8 83.82 0)
+      (effects (font (size 1.27 1.27)) hide)
+    )
+    (property "Description" "100mW" (at 50.8 83.82 0)
+      (effects (font (size 1.27 1.27)) hide)
+    )
+    (property "JLCPCB" "C417107" (at 50.8 83.82 0)
       (effects (font (size 1.27 1.27)) hide)
     )
@@
       (effects (font (size 1.27 1.27)) (justify right))
     )
-    (property "Footprint" "Resistor_SMD:R_0805_2012Metric_Pad1.20x1.40mm_HandSolder" (at 115.57 100.33 0)
+    (property "Footprint" "Resistor_SMD:R_0603_1608Metric" (at 115.57 100.33 0)
       (effects (font (size 1.27 1.27)) hide)
     )
@@
       (effects (font (size 1.27 1.27)) hide)
     )
-    (property "JLCPCB" "C103914" (at 115.57 100.33 0)
+    (property "JLCPCB" "C2924143" (at 115.57 100.33 0)
+      (effects (font (size 1.27 1.27)) hide)
+    )
+    (property "Description" "100mW" (at 115.57 100.33 0)
       (effects (font (size 1.27 1.27)) hide)
     )
@@
       (effects (font (size 1.27 1.27)) (justify right))
     )
-    (property "Footprint" "" (at 82.55 33.02 0)
+    (property "Footprint" "Resistor_SMD:R_0603_1608Metric" (at 82.55 33.02 0)
       (effects (font (size 1.27 1.27)) hide)
     )
     (property "Datasheet" "~" (at 82.55 33.02 0)
+      (effects (font (size 1.27 1.27)) hide)
+    )
+    (property "Description" "100mW" (at 82.55 33.02 0)
+      (effects (font (size 1.27 1.27)) hide)
+    )
+    (property "JLCPCB" "C101304" (at 82.55 33.02 0)
       (effects (font (size 1.27 1.27)) hide)
     )
@@
       (effects (font (size 1.27 1.27)) (justify left))
     )
-    (property "Footprint" "" (at 86.36 100.33 0)
+    (property "Footprint" "Resistor_SMD:R_0603_1608Metric" (at 86.36 100.33 0)
       (effects (font (size 1.27 1.27)) hide)
     )
     (property "Datasheet" "~" (at 86.36 100.33 0)
+      (effects (font (size 1.27 1.27)) hide)
+    )
+    (property "Description" "100mW" (at 86.36 100.33 0)
+      (effects (font (size 1.27 1.27)) hide)
+    )
+    (property "JLCPCB" "C417107" (at 86.36 100.33 0)
       (effects (font (size 1.27 1.27)) hide)
     )
@@
       (effects (font (size 1.27 1.27)))
     )
-    (property "Footprint" "" (at 50.8 93.98 0)
+    (property "Footprint" "Resistor_SMD:R_0603_1608Metric" (at 50.8 93.98 0)
       (effects (font (size 1.27 1.27)) hide)
     )
@@
       (effects (font (size 1.27 1.27)) hide)
     )
+    (property "Description" "100mW" (at 50.8 93.98 0)
+      (effects (font (size 1.27 1.27)) hide)
+    )
+    (property "JLCPCB" "C417107" (at 50.8 93.98 0)
+      (effects (font (size 1.27 1.27)) hide)
+    )
     (pin "1")
     (pin "2")
@@
       (effects (font (size 1.27 1.27)) (justify left))
     )
-    (property "Footprint" "" (at 344.17 90.17 0)
+    (property "Footprint" "Resistor_SMD:R_0603_1608Metric" (at 344.17 90.17 0)
       (effects (font (size 1.27 1.27)) hide)
     )
     (property "Datasheet" "~" (at 344.17 90.17 0)
+      (effects (font (size 1.27 1.27)) hide)
+    )
+    (property "Description" "250mW" (at 344.17 90.17 0)
+      (effects (font (size 1.27 1.27)) hide)
+    )
+    (property "JLCPCB" "C544033" (at 344.17 90.17 0)
       (effects (font (size 1.27 1.27)) hide)
     )
@@
       (effects (font (size 1.27 1.27)) (justify left))
     )
-    (property "Footprint" "Resistor_SMD:R_0805_2012Metric_Pad1.20x1.40mm_HandSolder" (at 119.38 100.33 0)
+    (property "Footprint" "Resistor_SMD:R_0603_1608Metric" (at 119.38 100.33 0)
       (effects (font (size 1.27 1.27)) hide)
     )
@@
       (effects (font (size 1.27 1.27)) hide)
     )
-    (property "JLCPCB" "C103914" (at 119.38 100.33 0)
-      (effects (font (size 1.27 1.27)) hide)
-    )
+    (property "JLCPCB" "C2924143" (at 119.38 100.33 0)
+      (effects (font (size 1.27 1.27)) hide)
+    )
+    (property "Description" "100mW" (at 119.38 100.33 0)
+      (effects (font (size 1.27 1.27)) hide)
+    )

Commit message: cleaned up footprint assignment
Parts:
- C11, C13, C25, C26, C27, C28, C5, C7, C9: Extended Part - -> (none)
- U12: MANUFACTURER Cirrus Logic Inc -> (none); MAXIMUM_PACKAGE_HEIGHT 0.8mm -> (none); PARTREV 4.1 -> (none); STANDARD IPC-7351B -> (none)
Changed lines of the file:
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@@
-      (effects (font (size 1.27 1.27)) hide)
-    )
-    (property "JLCPCB Part #" "" (at 33.02 91.44 0)
       (effects (font (size 1.27 1.27)) hide)
     )
@@
       (effects (font (size 1.27 1.27)) hide)
     )
-    (property "LCSC" "" (at 280.035 30.48 0)
-      (effects (font (size 1.27 1.27)) hide)
-    )
-    (property "Extended Part" "-" (at 280.035 30.48 0)
-      (effects (font (size 1.27 1.27)) hide)
-    )
     (property "JLCPCB" "C1525" (at 280.035 30.48 0)
       (effects (font (size 1.27 1.27)) hide)
@@
       (effects (font (size 1.27 1.27)) hide)
     )
-    (property "LCSC" "" (at 304.165 30.48 0)
-      (effects (font (size 1.27 1.27)) hide)
-    )
-    (property "Extended Part" "-" (at 304.165 30.48 0)
-      (effects (font (size 1.27 1.27)) hide)
-    )
     (property "JLCPCB" "C1525" (at 304.165 30.48 0)
       (effects (font (size 1.27 1.27)) hide)
@@
     )
     (property "Datasheet" "~" (at 256.54 97.79 0)
-      (effects (font (size 1.27 1.27)) hide)
-    )
-    (property "LCSC" "" (at 256.54 97.79 0)
-      (effects (font (size 1.27 1.27)) hide)
-    )
-    (property "Extended Part" "" (at 256.54 97.79 0)
       (effects (font (size 1.27 1.27)) hide)
     )
@@
     )
     (property "Datasheet" "https://datasheet.lcsc.com/szlcsc/1810121710_Korean-Hroparts-Elec-PJ-316A-6A_C128987.pdf" (at 363.22 69.85 0)
-      (effects (font (size 1.27 1.27)) hide)
-    )
-    (property "JLCPCB Part #" "" (at 361.95 69.85 0)
       (effects (font (size 1.27 1.27)) hide)
     )
@@
       (effects (font (size 1.27 1.27)) hide)
     )
-    (property "LCSC" "" (at 269.24 97.79 0)
-      (effects (font (size 1.27 1.27)) hide)
-    )
-    (property "Extended Part" "" (at 269.24 97.79 0)
-      (effects (font (size 1.27 1.27)) hide)
-    )
     (property "Description" "10V" (at 269.24 97.79 0)
       (effects (font (size 1.27 1.27)) hide)
@@
       (effects (font (size 1.27 1.27)) hide)
     )
-    (property "LCSC" "" (at 281.94 97.79 0)
-      (effects (font (size 1.27 1.27)) hide)
-    )
-    (property "Extended Part" "" (at 281.94 97.79 0)
-      (effects (font (size 1.27 1.27)) hide)
-    )
     (property "Description" "10V" (at 281.94 97.79 0)
       (effects (font (size 1.27 1.27)) hide)
@@
     )
     (property "Datasheet" "~" (at 92.71 52.07 0)
-      (effects (font (size 1.27 1.27)) hide)
-    )
-    (property "JLCPCB Part #" "" (at 92.71 52.07 0)
       (effects (font (size 1.27 1.27)) hide)
     )
@@
       (effects (font (size 1.27 1.27)) hide)
     )
-    (property "LCSC" "" (at 331.47 81.28 0)
-      (effects (font (size 1.27 1.27)) hide)
-    )
-    (property "Extended Part" "-" (at 331.47 81.28 0)
-      (effects (font (size 1.27 1.27)) hide)
-    )
     (property "JLCPCB" "C1525" (at 331.47 81.28 0)
       (effects (font (size 1.27 1.27)) hide)
@@
     )
     (property "Datasheet" "~" (at 231.14 97.79 0)
-      (effects (font (size 1.27 1.27)) hide)
-    )
-    (property "LCSC" "" (at 231.14 97.79 0)
-      (effects (font (size 1.27 1.27)) hide)
-    )
-    (property "Extended Part" "" (at 231.14 97.79 0)
       (effects (font (size 1.27 1.27)) hide)
     )
@@
       (effects (font (size 1.27 1.27)) hide)
     )
-    (property "JLCPCB Part #" "" (at 92.71 41.91 0)
-      (effects (font (size 1.27 1.27)) hide)
-    )
     (property "JLCPCB" "C52923" (at 92.71 41.91 0)
       (effects (font (size 1.27 1.27)) hide)
@@
       (effects (font (size 1.27 1.27)) hide)
     )
-    (property "JLCPCB Part #" "" (at 101.6 83.82 0)
-      (effects (font (size 1.27 1.27)) hide)
-    )
     (property "JLCPCB" "C52923" (at 101.6 83.82 0)
       (effects (font (size 1.27 1.27)) hide)
@@
     )
     (property "Datasheet" "~" (at 254.635 30.48 0)
-      (effects (font (size 1.27 1.27)) hide)
-    )
-    (property "LCSC" "" (at 254.635 30.48 0)
-      (effects (font (size 1.27 1.27)) hide)
-    )
-    (property "Extended Part" "-" (at 254.635 30.48 0)
       (effects (font (size 1.27 1.27)) hide)
     )
@@
       (effects (font (size 1.27 1.27)) hide)
     )
-    (property "LCSC" "" (at 291.465 30.48 0)
-      (effects (font (size 1.27 1.27)) hide)
-    )
-    (property "Extended Part" "-" (at 291.465 30.48 0)
-      (effects (font (size 1.27 1.27)) hide)
-    )
     (property "JLCPCB" "C1525" (at 291.465 30.48 0)
       (effects (font (size 1.27 1.27)) hide)
@@
     )
     (property "Datasheet" "~" (at 101.6 93.98 0)
-      (effects (font (size 1.27 1.27)) hide)
-    )
-    (property "JLCPCB Part #" "" (at 101.6 93.98 0)
       (effects (font (size 1.27 1.27)) hide)
     )
@@
     )
     (property "Datasheet" "https://datasheet.lcsc.com/szlcsc/1810121710_Korean-Hroparts-Elec-PJ-316A-6A_C128987.pdf" (at 31.75 49.53 0)
-      (effects (font (size 1.27 1.27)) hide)
-    )
-    (property "JLCPCB Part #" "" (at 33.02 49.53 0)
       (effects (font (size 1.27 1.27)) hide)
     )
@@
       (effects (font (size 1.27 1.27)) hide)
     )
-    (property "LCSC" "" (at 318.77 81.28 0)
-      (effects (font (size 1.27 1.27)) hide)
-    )
-    (property "Extended Part" "-" (at 318.77 81.28 0)
-      (effects (font (size 1.27 1.27)) hide)
-    )
     (property "JLCPCB" "C1525" (at 318.77 81.28 0)
       (effects (font (size 1.27 1.27)) hide)
@@
       (effects (font (size 1.27 1.27)) hide)
     )
-    (property "LCSC" "" (at 243.84 97.79 0)
-      (effects (font (size 1.27 1.27)) hide)
-    )
-    (property "Extended Part" "" (at 243.84 97.79 0)
-      (effects (font (size 1.27 1.27)) hide)
-    )
     (property "JLCPCB" "C12530" (at 243.84 97.79 0)
       (effects (font (size 1.27 1.27)) hide)
@@
       (effects (font (size 1.27 1.27)) hide)
     )
-    (property "LCSC" "" (at 306.07 81.28 0)
-      (effects (font (size 1.27 1.27)) hide)
-    )
-    (property "Extended Part" "-" (at 306.07 81.28 0)
-      (effects (font (size 1.27 1.27)) hide)
-    )
     (property "JLCPCB" "C1525" (at 306.07 81.28 0)
       (effects (font (size 1.27 1.27)) hide)
@@
     )
     (property "Datasheet" "~" (at 76.2 52.07 0)
-      (effects (font (size 1.27 1.27)) hide)
-    )
-    (property "LCSC" "" (at 76.2 52.07 90)
       (effects (font (size 1.27 1.27)) hide)
     )
@@
       (effects (font (size 1.27 1.27)) hide)
     )
-    (property "LCSC" "" (at 76.2 41.91 90)
-      (effects (font (size 1.27 1.27)) hide)
-    )
     (property "JLCPCB" "C160969" (at 76.2 41.91 0)
       (effects (font (size 1.27 1.27)) hide)
@@
     )
     (property "Datasheet" "" (at 194.31 64.77 0)
-      (effects (font (size 1.27 1.27)) (justify left bottom) hide)
-    )
-    (property "MANUFACTURER" "Cirrus Logic Inc" (at 194.31 64.77 0)
-      (effects (font (size 1.27 1.27)) (justify left bottom) hide)
-    )
-    (property "PARTREV" "4.1" (at 194.31 64.77 0)
-      (effects (font (size 1.27 1.27)) (justify left bottom) hide)
-    )
-    (property "STANDARD" "IPC-7351B" (at 194.31 64.77 0)
-      (effects (font (size 1.27 1.27)) (justify left bottom) hide)
-    )
-    (property "MAXIMUM_PACKAGE_HEIGHT" "0.8mm" (at 194.31 64.77 0)
       (effects (font (size 1.27 1.27)) (justify left bottom) hide)
     )
@@
       (effects (font (size 1.27 1.27)) hide)
     )
-    (property "JLCPCB Part #" "" (at 361.95 49.53 0)
-      (effects (font (size 1.27 1.27)) hide)
-    )
     (property "JLCPCB" "C128987" (at 361.95 49.53 0)
       (effects (font (size 1.27 1.27)) hide)
@@
       (effects (font (size 1.27 1.27)) hide)
     )
-    (property "LCSC" "" (at 344.17 81.28 0)
-      (effects (font (size 1.27 1.27)) hide)
-    )
-    (property "Extended Part" "-" (at 344.17 81.28 0)
-      (effects (font (size 1.27 1.27)) hide)
-    )
     (property "JLCPCB" "C1525" (at 344.17 81.28 0)
       (effects (font (size 1.27 1.27)) hide)
@@
       (effects (font (size 1.27 1.27)) hide)
     )
-    (property "LCSC" "" (at 267.335 30.48 0)
-      (effects (font (size 1.27 1.27)) hide)
-    )
-    (property "Extended Part" "-" (at 267.335 30.48 0)
-      (effects (font (size 1.27 1.27)) hide)
-    )
