File: KLST_PANDA/power.kicad_sch (KiCad schematic)
At the start: 10 parts, among them Q1 AO3401A, U1 AMS1117-3.3

Commit message: removed GDNA
Parts:
- removed NT2: NetTie_2, symbol Device:NetTie_2

Commit message: started spec'ing components
Parts:
- C1, C3: JLCPCB (none) -> C15850; JLCPCB Part # C15850 -> (none)
- C4: footprint Capacitor_SMD:C_0402_1005Metric -> Capacitor_SMD:C_0805_2012Metric; JLCPCB (none) -> C28323; JLCPCB Part # C52923 -> (none)
- C5: footprint Capacitor_SMD:C_0402_1005Metric -> Capacitor_SMD:C_0805_2012Metric; JLCPCB (none) -> C1710; JLCPCB Part # C15195 -> (none)
- FB1: JLCPCB (none) -> C73732; JLCPCB Part # C73732 -> (none)
- L1: JLCPCB (none) -> C26443; JLCPCB Part # C26443 -> (none)
- NT1: footprint (none) -> NetTie-2_SMD_Pad2.0mm; JLCPCB (none) -> DNF
- Q1: JLCPCB (none) -> C15127; JLCPCB Part # C15127 -> (none)
Other:
- note added: "@TODO(check im 200mA is OK)"
Changed lines of the file:
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@@
     (fill (type none))
   )
-  (text_box "VDDA can be connected to VDD through a ferrite bead."
-    (at 111.76 46.99 0) (size 27.94 13.97)
+  (text_box "VDDA can be connected to VDD through a ferrite bead. see AN5419"
+    (at 111.76 46.99 0) (size 24.13 13.97)
     (stroke (width 0) (type default))
     (fill (type none))
@@
     (effects (font (size 1.27 1.27)) (justify left bottom))
   )
+  (text "@TODO(check im 200mA is OK)" (at 120.015 26.67 0)
+    (effects (font (size 1.27 1.27)) (justify left bottom))
+  )
   (text "POWER FLAGS" (at 15.24 67.945 0)
     (effects (font (size 1.27 1.27)) (justify left bottom))
@@
       (effects (font (size 1.27 1.27)) hide)
     )
-    (property "JLCPCB Part #" "C15850" (at 92.075 45.085 0)
+    (property "JLCPCB Part #" "" (at 92.075 45.085 0)
+      (effects (font (size 1.27 1.27)) hide)
+    )
+    (property "Description" "25V" (at 92.075 45.085 0)
+      (effects (font (size 1.27 1.27)) hide)
+    )
+    (property "JLCPCB" "C15850" (at 92.075 45.085 0)
       (effects (font (size 1.27 1.27)) hide)
     )
@@
       (effects (font (size 1.27 1.27)) hide)
     )
-    (property "JLCPCB Part #" "C73732" (at 53.34 38.735 90)
+    (property "JLCPCB Part #" "" (at 53.34 38.735 90)
+      (effects (font (size 1.27 1.27)) hide)
+    )
+    (property "JLCPCB" "C73732" (at 53.34 38.735 0)
       (effects (font (size 1.27 1.27)) hide)
     )
@@
       (effects (font (size 1.27 1.27)) (justify left))
     )
-    (property "Footprint" "Capacitor_SMD:C_0402_1005Metric" (at 135.89 34.29 0)
+    (property "Footprint" "Capacitor_SMD:C_0805_2012Metric" (at 135.89 34.29 0)
       (effects (font (size 1.27 1.27)) hide)
     )
@@
       (effects (font (size 1.27 1.27)) hide)
     )
-    (property "JLCPCB Part #" "C15195" (at 135.89 34.29 0)
+    (property "JLCPCB Part #" "" (at 135.89 34.29 0)
+      (effects (font (size 1.27 1.27)) hide)
+    )
+    (property "JLCPCB" "C1710" (at 135.89 34.29 0)
+      (effects (font (size 1.27 1.27)) hide)
+    )
+    (property "Description" "50V" (at 135.89 34.29 0)
       (effects (font (size 1.27 1.27)) hide)
     )
@@
       (effects (font (size 1.27 1.27)) (justify left))
     )
-    (property "Footprint" "Capacitor_SMD:C_0402_1005Metric" (at 125.73 34.29 0)
+    (property "Footprint" "Capacitor_SMD:C_0805_2012Metric" (at 125.73 34.29 0)
       (effects (font (size 1.27 1.27)) hide)
     )
@@
       (effects (font (size 1.27 1.27)) hide)
     )
-    (property "JLCPCB Part #" "C52923" (at 125.73 34.29 0)
+    (property "JLCPCB Part #" "" (at 125.73 34.29 0)
+      (effects (font (size 1.27 1.27)) hide)
+    )
+    (property "JLCPCB" "C28323" (at 125.73 34.29 0)
+      (effects (font (size 1.27 1.27)) hide)
+    )
+    (property "Description" "50V" (at 125.73 34.29 0)
       (effects (font (size 1.27 1.27)) hide)
     )
@@
       (effects (font (size 1.27 1.27)) hide)
     )
-    (property "JLCPCB Part #" "C26443" (at 120.65 30.48 0)
+    (property "JLCPCB Part #" "" (at 120.65 30.48 0)
+      (effects (font (size 1.27 1.27)) hide)
+    )
+    (property "JLCPCB" "C26443" (at 120.65 30.48 0)
+      (effects (font (size 1.27 1.27)) hide)
+    )
+    (property "Description" "200mA" (at 120.65 30.48 0)
       (effects (font (size 1.27 1.27)) hide)
     )
@@
       (effects (font (size 1.27 1.27)) hide)
     )
-    (property "JLCPCB Part #" "C15850" (at 62.23 45.085 0)
+    (property "JLCPCB Part #" "" (at 62.23 45.085 0)
+      (effects (font (size 1.27 1.27)) hide)
+    )
+    (property "Description" "25V" (at 62.23 45.085 0)
+      (effects (font (size 1.27 1.27)) hide)
+    )
+    (property "JLCPCB" "C15850" (at 62.23 45.085 0)
       (effects (font (size 1.27 1.27)) hide)
     )
@@
       (effects (font (size 1.27 1.27)) hide)
     )
-    (property "JLCPCB Part #" "C15127" (at 38.1 41.275 0)
+    (property "JLCPCB Part #" "" (at 38.1 41.275 0)
+      (effects (font (size 1.27 1.27)) hide)
+    )
+    (property "JLCPCB" "C15127" (at 38.1 41.275 0)
       (effects (font (size 1.27 1.27)) hide)
     )
@@
       (effects (font (size 1.27 1.27)) (justify left))
     )
-    (property "Footprint" "" (at 92.075 30.48 0)
+    (property "Footprint" "NetTie-2_SMD_Pad2.0mm" (at 92.075 30.48 0)
       (effects (font (size 1.27 1.27)) hide)
     )
@@
       (effects (font (size 1.27 1.27)) hide)
     )
+    (property "JLCPCB" "DNF" (at 92.075 30.48 0)
+      (effects (font (size 1.27 1.27)) hide)
+    )

Commit message: assigned footprints
Parts:
- NT1: footprint NetTie-2_SMD_Pad2.0mm -> NetTie:NetTie-2_SMD_Pad2.0mm
- U1: JLCPCB (none) -> C6186; JLCPCB Part # C6186 -> (none)
Changed lines of the file:
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@@
       (effects (font (size 1.27 1.27)) hide)
     )
-    (property "JLCPCB Part #" "C6186" (at 76.2 38.735 0)
+    (property "JLCPCB Part #" "" (at 76.2 38.735 0)
+      (effects (font (size 1.27 1.27)) hide)
+    )
+    (property "JLCPCB" "C6186" (at 76.2 38.735 0)
       (effects (font (size 1.27 1.27)) hide)
     )
@@
       (effects (font (size 1.27 1.27)) (justify left))
     )
-    (property "Footprint" "NetTie-2_SMD_Pad2.0mm" (at 92.075 30.48 0)
+    (property "Footprint" "NetTie:NetTie-2_SMD_Pad2.0mm" (at 92.075 30.48 0)
       (effects (font (size 1.27 1.27)) hide)
     )

Commit message: cleaned up footprint assignment
Parts:
- C1, C3: Extended Part - -> (none); MFR.Part # CL21A106KAYNNNE -> (none)
- C4: Extended Part - -> (none); MFR.Part # CL05A105KA5NQNC -> (none)
- C5: Extended Part - -> (none); MFR.Part # CL05B103KB5NNNC -> (none)
- L1: Extended Part - -> (none); MFR.Part # SDCL1005C39NJTDF -> (none)
- Q1: Extended Part - -> (none); MFR.Part # AO3401A -> (none)
- U1: Extended Part - -> (none); MFR.Part # AMS1117-3.3 -> (none)
Changed lines of the file:
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@@
-      (effects (font (size 1.27 1.27)) hide)
-    )
-    (property "MFR.Part #" "CL21A106KAYNNNE" (at 92.075 45.085 0)
-      (effects (font (size 1.27 1.27)) hide)
-    )
-    (property "LCSC Part #" "" (at 92.075 45.085 0)
-      (effects (font (size 1.27 1.27)) hide)
-    )
-    (property "Extended Part" "-" (at 92.075 45.085 0)
-      (effects (font (size 1.27 1.27)) hide)
-    )
-    (property "JLCPCB Part #" "" (at 92.075 45.085 0)
       (effects (font (size 1.27 1.27)) hide)
     )
@@
     )
     (property "Datasheet" "~" (at 53.34 38.735 0)
-      (effects (font (size 1.27 1.27)) hide)
-    )
-    (property "JLCPCB Part #" "" (at 53.34 38.735 90)
       (effects (font (size 1.27 1.27)) hide)
     )
@@
       (effects (font (size 1.27 1.27)) hide)
     )
-    (property "MFR.Part #" "CL05B103KB5NNNC" (at 135.89 34.29 0)
-      (effects (font (size 1.27 1.27)) hide)
-    )
-    (property "LCSC Part #" "" (at 135.89 34.29 0)
-      (effects (font (size 1.27 1.27)) hide)
-    )
-    (property "Extended Part" "-" (at 135.89 34.29 0)
-      (effects (font (size 1.27 1.27)) hide)
-    )
-    (property "JLCPCB Part #" "" (at 135.89 34.29 0)
-      (effects (font (size 1.27 1.27)) hide)
-    )
     (property "JLCPCB" "C1710" (at 135.89 34.29 0)
       (effects (font (size 1.27 1.27)) hide)
@@
       (effects (font (size 1.27 1.27)) hide)
     )
-    (property "MFR.Part #" "CL05A105KA5NQNC" (at 125.73 34.29 0)
-      (effects (font (size 1.27 1.27)) hide)
-    )
-    (property "LCSC Part #" "" (at 125.73 34.29 0)
-      (effects (font (size 1.27 1.27)) hide)
-    )
-    (property "Extended Part" "-" (at 125.73 34.29 0)
-      (effects (font (size 1.27 1.27)) hide)
-    )
-    (property "JLCPCB Part #" "" (at 125.73 34.29 0)
-      (effects (font (size 1.27 1.27)) hide)
-    )
     (property "JLCPCB" "C28323" (at 125.73 34.29 0)
       (effects (font (size 1.27 1.27)) hide)
@@
       (effects (font (size 1.27 1.27)) hide)
     )
-    (property "MFR.Part #" "SDCL1005C39NJTDF" (at 120.65 30.48 90)
-      (effects (font (size 1.27 1.27)) hide)
-    )
-    (property "LCSC Part #" "" (at 120.65 30.48 90)
-      (effects (font (size 1.27 1.27)) hide)
-    )
-    (property "Extended Part" "-" (at 120.65 30.48 0)
-      (effects (font (size 1.27 1.27)) hide)
-    )
-    (property "JLCPCB Part #" "" (at 120.65 30.48 0)
-      (effects (font (size 1.27 1.27)) hide)
-    )
     (property "JLCPCB" "C26443" (at 120.65 30.48 0)
       (effects (font (size 1.27 1.27)) hide)
@@
       (effects (font (size 1.27 1.27)) hide)
     )
-    (property "MFR.Part #" "CL21A106KAYNNNE" (at 62.23 45.085 0)
-      (effects (font (size 1.27 1.27)) hide)
-    )
-    (property "LCSC Part #" "" (at 62.23 45.085 0)
-      (effects (font (size 1.27 1.27)) hide)
-    )
-    (property "Extended Part" "-" (at 62.23 45.085 0)
-      (effects (font (size 1.27 1.27)) hide)
-    )
-    (property "JLCPCB Part #" "" (at 62.23 45.085 0)
-      (effects (font (size 1.27 1.27)) hide)
-    )
     (property "Description" "25V" (at 62.23 45.085 0)
       (effects (font (size 1.27 1.27)) hide)
@@
       (effects (font (size 1.27 1.27)) (justify left) hide)
     )
-    (property "MFR.Part #" "AO3401A" (at 38.1 41.275 90)
-      (effects (font (size 1.27 1.27)) hide)
-    )
-    (property "LCSC Part #" "" (at 38.1 41.275 90)
-      (effects (font (size 1.27 1.27)) hide)
-    )
-    (property "Extended Part" "-" (at 38.1 41.275 0)
-      (effects (font (size 1.27 1.27)) hide)
-    )
-    (property "JLCPCB Part #" "" (at 38.1 41.275 0)
-      (effects (font (size 1.27 1.27)) hide)
-    )
     (property "JLCPCB" "C15127" (at 38.1 41.275 0)
       (effects (font (size 1.27 1.27)) hide)
@@
       (effects (font (size 1.27 1.27)) hide)
     )
-    (property "MFR.Part #" "AMS1117-3.3" (at 76.2 38.735 0)
-      (effects (font (size 1.27 1.27)) hide)
-    )
-    (property "Extended Part" "-" (at 76.2 38.735 0)
-      (effects (font (size 1.27 1.27)) hide)
-    )
-    (property "JLCPCB Part #" "" (at 76.2 38.735 0)
-      (effects (font (size 1.27 1.27)) hide)
-    )

Commit message: distributed modules
Connections:
- net (PWR_3.3V): now reaches C3.1, NT1.2, U1.2 (VO)
- net (PWR_5V): now reaches C1.1, FB1.1, U1.3 (VI)
Other:
- moved on the sheet: C1, C3, C4, C5, FB1, L1, NT1, Q1, U1

Commit message: added resistor and capacitor, cleaned up TODOs
Other:
- note added: "@NOTE(200mA rating)"
- note removed: "@TODO(check im 200mA is OK)"
Changed lines of the file:
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@@
   )
   (text_box "VDDA can be connected to VDD through a ferrite bead. see AN5419"
-    (at 112.395 48.26 0) (size 24.13 13.97)
+    (at 110.49 51.435 0) (size 31.75 7.62)
     (stroke (width 0) (type default))
     (fill (type none))
@@
     (effects (font (size 1.27 1.27)) (justify left bottom))
   )
-  (text "@TODO(check im 200mA is OK)" (at 120.65 27.94 0)
+  (text "@NOTE(200mA rating)" (at 114.3 27.305 0)
     (effects (font (size 1.27 1.27)) (justify left bottom))
   )
@@
         )
         (path "/b4513875-4c57-4720-bcc5-43ead67fe18f/efc23d99-04cc-4530-a8d8-9c096b510f30"
-          (reference "#PWR010") (unit 1)
+          (reference "#PWR011") (unit 1)
         )
       )
@@
         )
         (path "/b4513875-4c57-4720-bcc5-43ead67fe18f/efc23d99-04cc-4530-a8d8-9c096b510f30"
-          (reference "#PWR04") (unit 1)
+          (reference "#PWR05") (unit 1)
         )
       )
@@
         )
         (path "/b4513875-4c57-4720-bcc5-43ead67fe18f/efc23d99-04cc-4530-a8d8-9c096b510f30"
-          (reference "#PWR08") (unit 1)
+          (reference "#PWR09") (unit 1)
         )
       )
@@
         )
         (path "/b4513875-4c57-4720-bcc5-43ead67fe18f/efc23d99-04cc-4530-a8d8-9c096b510f30"
-          (reference "#PWR011") (unit 1)
+          (reference "#PWR012") (unit 1)
         )
       )
@@
         )
         (path "/b4513875-4c57-4720-bcc5-43ead67fe18f/efc23d99-04cc-4530-a8d8-9c096b510f30"
-          (reference "#PWR05") (unit 1)
+          (reference "#PWR06") (unit 1)
         )
       )
@@
         )
         (path "/b4513875-4c57-4720-bcc5-43ead67fe18f/efc23d99-04cc-4530-a8d8-9c096b510f30"
-          (reference "#PWR012") (unit 1)
+          (reference "#PWR013") (unit 1)
         )
       )
@@
         )
         (path "/b4513875-4c57-4720-bcc5-43ead67fe18f/efc23d99-04cc-4530-a8d8-9c096b510f30"
-          (reference "#PWR09") (unit 1)
+          (reference "#PWR010") (unit 1)
         )
       )
@@
         )
         (path "/b4513875-4c57-4720-bcc5-43ead67fe18f/efc23d99-04cc-4530-a8d8-9c096b510f30"
-          (reference "#PWR07") (unit 1)
+          (reference "#PWR08") (unit 1)
         )
       )
@@
         )
         (path "/b4513875-4c57-4720-bcc5-43ead67fe18f/efc23d99-04cc-4530-a8d8-9c096b510f30"
-          (reference "#PWR06") (unit 1)
+          (reference "#PWR07") (unit 1)
         )
       )
@@
       (effects (font (size 1.27 1.27)) hide)
     )
-    (property "Value" "+3.3VA" (at 136.525 20.32 0)
-      (effects (font (size 1.27 1.27)))
+    (property "Value" "+3.3VA" (at 138.43 24.13 0)
+      (effects (font (size 1.27 1.27)) (justify left))
     )
     (property "Footprint" "" (at 136.525 25.4 0)
@@
         )
         (path "/b4513875-4c57-4720-bcc5-43ead67fe18f/efc23d99-04cc-4530-a8d8-9c096b510f30"
-          (reference "#PWR013") (unit 1)
-        )
-      )
+          (reference "#PWR014") (unit 1)
+        )
+      )
