File: KLST_PANDA/ADC_DAC.kicad_sch (KiCad schematic)
At the start: 7 parts, among them J3 ADC, J3 DAC, U6 TLV9001IDCK

Commit message: removed GDNA
Parts:
- renumbered R50 to R46, R51 to R47, R52 to R48, U6 to U7
Changed lines of the file:
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@@
         )
         (path "/b4513875-4c57-4720-bcc5-43ead67fe18f/98dcce4c-cc8c-420d-bfb6-73762da3b881"
-          (reference "#PWR076") (unit 1)
+          (reference "#PWR074") (unit 1)
         )
       )
@@
         )
         (path "/b4513875-4c57-4720-bcc5-43ead67fe18f/98dcce4c-cc8c-420d-bfb6-73762da3b881"
-          (reference "#PWR074") (unit 1)
+          (reference "#PWR072") (unit 1)
         )
       )
@@
         )
         (path "/b4513875-4c57-4720-bcc5-43ead67fe18f/98dcce4c-cc8c-420d-bfb6-73762da3b881"
-          (reference "#PWR073") (unit 1)
+          (reference "#PWR071") (unit 1)
         )
       )
@@
   (symbol (lib_id "Device:R_Small") (at 87.63 78.105 90) (unit 1)
     (in_bom yes) (on_board yes) (dnp no)
-    (property "Reference" "R51" (at 87.63 74.295 90)
+    (property "Reference" "R47" (at 87.63 74.295 90)
       (effects (font (size 1.27 1.27)))
     )
@@
       (project "KLST_PANDA"
         (path "/b4513875-4c57-4720-bcc5-43ead67fe18f/98dcce4c-cc8c-420d-bfb6-73762da3b881"
-          (reference "R51") (unit 1)
+          (reference "R47") (unit 1)
         )
       )
@@
   (symbol (lib_id "Amplifier_Operational:TLV9001IDCK") (at 98.425 80.645 0) (unit 1)
     (in_bom yes) (on_board yes) (dnp no) (fields_autoplaced)
-    (property "Reference" "U6" (at 114.3 77.2161 0)
+    (property "Reference" "U7" (at 114.3 77.2161 0)
       (effects (font (size 1.27 1.27)))
     )
@@
       (project "KLST_PANDA"
         (path "/b4513875-4c57-4720-bcc5-43ead67fe18f/98dcce4c-cc8c-420d-bfb6-73762da3b881"
-          (reference "U6") (unit 1)
+          (reference "U7") (unit 1)
         )
       )
@@
   (symbol (lib_id "power:+3.3V") (at 98.425 66.04 0) (unit 1)
     (in_bom yes) (on_board yes) (dnp no) (fields_autoplaced)
-    (property "Reference" "#PWR075" (at 98.425 69.85 0)
+    (property "Reference" "#PWR073" (at 98.425 69.85 0)
       (effects (font (size 1.27 1.27)) hide)
     )
@@
       (project "KLST_PANDA"
         (path "/b4513875-4c57-4720-bcc5-43ead67fe18f/98dcce4c-cc8c-420d-bfb6-73762da3b881"
-          (reference "#PWR075") (unit 1)
+          (reference "#PWR073") (unit 1)
         )
       )
@@
   (symbol (lib_id "Device:R_Small") (at 81.915 85.09 0) (mirror y) (unit 1)
     (in_bom yes) (on_board yes) (dnp no)
-    (property "Reference" "R50" (at 80.645 83.82 0)
+    (property "Reference" "R46" (at 80.645 83.82 0)
       (effects (font (size 1.27 1.27)) (justify left))
     )
@@
       (project "KLST_PANDA"
         (path "/b4513875-4c57-4720-bcc5-43ead67fe18f/98dcce4c-cc8c-420d-bfb6-73762da3b881"
-          (reference "R50") (unit 1)
+          (reference "R46") (unit 1)
         )
       )
@@
   (symbol (lib_id "Device:R_Small") (at 106.68 69.85 90) (unit 1)
     (in_bom yes) (on_board yes) (dnp no)
-    (property "Reference" "R52" (at 106.68 66.04 90)
+    (property "Reference" "R48" (at 106.68 66.04 90)
       (effects (font (size 1.27 1.27)))
     )
@@
       (project "KLST_PANDA"
         (path "/b4513875-4c57-4720-bcc5-43ead67fe18f/98dcce4c-cc8c-420d-bfb6-73762da3b881"
-          (reference "R52") (unit 1)
-        )
-      )
+          (reference "R48") (unit 1)
+        )
+      )

Commit message: resolved TODOs
Parts:
- renumbered U7 to U8
Changed lines of the file:
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@@
   (symbol (lib_id "Amplifier_Operational:TLV9001IDCK") (at 98.425 80.645 0) (unit 1)
     (in_bom yes) (on_board yes) (dnp no) (fields_autoplaced)
-    (property "Reference" "U7" (at 114.3 77.2161 0)
+    (property "Reference" "U8" (at 114.3 77.2161 0)
       (effects (font (size 1.27 1.27)))
     )
@@
       (project "KLST_PANDA"
         (path "/b4513875-4c57-4720-bcc5-43ead67fe18f/98dcce4c-cc8c-420d-bfb6-73762da3b881"
-          (reference "U7") (unit 1)
+          (reference "U8") (unit 1)
         )
       )

Commit message: started spec'ing components
Parts:
- D18: value D_Schottky -> SS14; footprint Diode_SMD:D_SOD-123 -> Diode_SMD:D_SMA; JLCPCB (none) -> C2480; JLCPCB Part # C8598 -> (none)
- J3: JLCPCB (none) -> C128987; JLCPCB Part # C128987 -> (none)
Changed lines of the file:
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@@
       (effects (font (size 1.27 1.27)))
     )
-    (property "Value" "D_Schottky" (at 102.235 31.115 0)
+    (property "Value" "SS14" (at 102.235 31.115 0)
       (effects (font (size 1.27 1.27)))
     )
-    (property "Footprint" "Diode_SMD:D_SOD-123" (at 102.235 33.655 90)
+    (property "Footprint" "Diode_SMD:D_SMA" (at 102.235 33.655 90)
       (effects (font (size 1.27 1.27)) hide)
     )
@@
       (effects (font (size 1.27 1.27)) hide)
     )
-    (property "JLCPCB Part #" "C8598" (at 102.235 33.655 0)
+    (property "JLCPCB Part #" "" (at 102.235 33.655 0)
+      (effects (font (size 1.27 1.27)) hide)
+    )
+    (property "JLCPCB" "C2480" (at 102.235 33.655 0)
       (effects (font (size 1.27 1.27)) hide)
     )
@@
       (effects (font (size 1.27 1.27)) hide)
     )
-    (property "JLCPCB Part #" "C128987" (at 29.845 83.185 0)
+    (property "JLCPCB Part #" "" (at 29.845 83.185 0)
+      (effects (font (size 1.27 1.27)) hide)
+    )
+    (property "JLCPCB" "C128987" (at 29.845 83.185 0)
       (effects (font (size 1.27 1.27)) hide)
     )
@@
       (effects (font (size 1.27 1.27)) hide)
     )
-    (property "JLCPCB Part #" "C128987" (at 29.845 38.735 0)
+    (property "JLCPCB Part #" "" (at 29.845 38.735 0)
       (effects (font (size 1.27 1.27)) hide)
     )
+    (property "JLCPCB" "C128987" (at 29.845 38.735 0)
+      (effects (font (size 1.27 1.27)) hide)
+    )

Commit message: assigned footprints
Parts:
- R46: footprint (none) -> Resistor_SMD:R_0805_2012Metric; JLCPCB (none) -> C25611
- R47, R48: footprint (none) -> Resistor_SMD:R_0805_2012Metric; JLCPCB (none) -> C4328
- U8: JLCPCB (none) -> C398362
Changed lines of the file:
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@@
       (effects (font (size 1.27 1.27)))
     )
-    (property "Footprint" "" (at 87.63 78.105 0)
+    (property "Footprint" "Resistor_SMD:R_0805_2012Metric" (at 87.63 78.105 0)
       (effects (font (size 1.27 1.27)) hide)
     )
     (property "Datasheet" "~" (at 87.63 78.105 0)
+      (effects (font (size 1.27 1.27)) hide)
+    )
+    (property "Description" "125mW" (at 87.63 78.105 0)
+      (effects (font (size 1.27 1.27)) hide)
+    )
+    (property "JLCPCB" "C4328" (at 87.63 78.105 0)
       (effects (font (size 1.27 1.27)) hide)
     )
@@
     )
     (property "Datasheet" "https://www.ti.com/lit/ds/symlink/tlv9001.pdf" (at 98.425 80.645 0)
+      (effects (font (size 1.27 1.27)) hide)
+    )
+    (property "JLCPCB" "C398362" (at 98.425 80.645 0)
       (effects (font (size 1.27 1.27)) hide)
     )
@@
       (effects (font (size 1.27 1.27)) (justify left))
     )
-    (property "Footprint" "" (at 81.915 85.09 0)
+    (property "Footprint" "Resistor_SMD:R_0805_2012Metric" (at 81.915 85.09 0)
       (effects (font (size 1.27 1.27)) hide)
     )
@@
       (effects (font (size 1.27 1.27)) hide)
     )
+    (property "Description" "125mW" (at 81.915 85.09 0)
+      (effects (font (size 1.27 1.27)) hide)
+    )
+    (property "JLCPCB" "C25611" (at 81.915 85.09 0)
+      (effects (font (size 1.27 1.27)) hide)
+    )
     (pin "1")
     (pin "2")
@@
       (effects (font (size 1.27 1.27)))
     )
-    (property "Footprint" "" (at 106.68 69.85 0)
+    (property "Footprint" "Resistor_SMD:R_0805_2012Metric" (at 106.68 69.85 0)
       (effects (font (size 1.27 1.27)) hide)
     )
@@
       (effects (font (size 1.27 1.27)) hide)
     )
+    (property "Description" "125mW" (at 106.68 69.85 0)
+      (effects (font (size 1.27 1.27)) hide)
+    )
+    (property "JLCPCB" "C4328" (at 106.68 69.85 0)
+      (effects (font (size 1.27 1.27)) hide)
+    )

Commit message: cleaned up footprint assignment
Parts:
- D18: Extended Part - -> (none); MFR.Part # B5819W -> (none)
Changed lines of the file:
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@@
-      (effects (font (size 1.27 1.27)) hide)
-    )
-    (property "MFR.Part #" "B5819W" (at 102.235 33.655 0)
-      (effects (font (size 1.27 1.27)) hide)
-    )
-    (property "LCSC Part #" "" (at 102.235 33.655 0)
-      (effects (font (size 1.27 1.27)) hide)
-    )
-    (property "Extended Part" "-" (at 102.235 33.655 0)
-      (effects (font (size 1.27 1.27)) hide)
-    )
-    (property "JLCPCB Part #" "" (at 102.235 33.655 0)
       (effects (font (size 1.27 1.27)) hide)
     )
@@
       (effects (font (size 1.27 1.27)) hide)
     )
-    (property "JLCPCB Part #" "" (at 29.845 83.185 0)
-      (effects (font (size 1.27 1.27)) hide)
-    )
     (property "JLCPCB" "C128987" (at 29.845 83.185 0)
       (effects (font (size 1.27 1.27)) hide)
@@
       (effects (font (size 1.27 1.27)) hide)
     )
-    (property "JLCPCB Part #" "" (at 29.845 38.735 0)
-      (effects (font (size 1.27 1.27)) hide)
-    )

Commit message: added resistor and capacitor, cleaned up TODOs
Parts:
- renumbered R46 to R47, R47 to R48, R48 to R49, U8 to U9
Changed lines of the file:
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@@
         )
         (path "/b4513875-4c57-4720-bcc5-43ead67fe18f/98dcce4c-cc8c-420d-bfb6-73762da3b881"
-          (reference "#PWR074") (unit 1)
+          (reference "#PWR076") (unit 1)
         )
       )
@@
         )
         (path "/b4513875-4c57-4720-bcc5-43ead67fe18f/98dcce4c-cc8c-420d-bfb6-73762da3b881"
-          (reference "#PWR072") (unit 1)
+          (reference "#PWR074") (unit 1)
         )
       )
@@
         )
         (path "/b4513875-4c57-4720-bcc5-43ead67fe18f/98dcce4c-cc8c-420d-bfb6-73762da3b881"
-          (reference "#PWR071") (unit 1)
+          (reference "#PWR073") (unit 1)
         )
       )
@@
   (symbol (lib_id "Device:R_Small") (at 87.63 78.105 90) (unit 1)
     (in_bom yes) (on_board yes) (dnp no)
-    (property "Reference" "R47" (at 87.63 74.295 90)
+    (property "Reference" "R48" (at 87.63 74.295 90)
       (effects (font (size 1.27 1.27)))
     )
@@
       (project "KLST_PANDA"
         (path "/b4513875-4c57-4720-bcc5-43ead67fe18f/98dcce4c-cc8c-420d-bfb6-73762da3b881"
-          (reference "R47") (unit 1)
+          (reference "R48") (unit 1)
         )
       )
@@
   (symbol (lib_id "Amplifier_Operational:TLV9001IDCK") (at 98.425 80.645 0) (unit 1)
     (in_bom yes) (on_board yes) (dnp no) (fields_autoplaced)
-    (property "Reference" "U8" (at 114.3 77.2161 0)
+    (property "Reference" "U9" (at 114.3 77.2161 0)
       (effects (font (size 1.27 1.27)))
     )
@@
       (project "KLST_PANDA"
         (path "/b4513875-4c57-4720-bcc5-43ead67fe18f/98dcce4c-cc8c-420d-bfb6-73762da3b881"
-          (reference "U8") (unit 1)
+          (reference "U9") (unit 1)
         )
       )
@@
   (symbol (lib_id "power:+3.3V") (at 98.425 66.04 0) (unit 1)
     (in_bom yes) (on_board yes) (dnp no) (fields_autoplaced)
-    (property "Reference" "#PWR073" (at 98.425 69.85 0)
+    (property "Reference" "#PWR075" (at 98.425 69.85 0)
       (effects (font (size 1.27 1.27)) hide)
     )
@@
       (project "KLST_PANDA"
         (path "/b4513875-4c57-4720-bcc5-43ead67fe18f/98dcce4c-cc8c-420d-bfb6-73762da3b881"
-          (reference "#PWR073") (unit 1)
+          (reference "#PWR075") (unit 1)
         )
       )
@@
   (symbol (lib_id "Device:R_Small") (at 81.915 85.09 0) (mirror y) (unit 1)
     (in_bom yes) (on_board yes) (dnp no)
-    (property "Reference" "R46" (at 80.645 83.82 0)
+    (property "Reference" "R47" (at 80.645 83.82 0)
       (effects (font (size 1.27 1.27)) (justify left))
     )
@@
       (project "KLST_PANDA"
         (path "/b4513875-4c57-4720-bcc5-43ead67fe18f/98dcce4c-cc8c-420d-bfb6-73762da3b881"
-          (reference "R46") (unit 1)
+          (reference "R47") (unit 1)
         )
       )
@@
   (symbol (lib_id "Device:R_Small") (at 106.68 69.85 90) (unit 1)
     (in_bom yes) (on_board yes) (dnp no)
-    (property "Reference" "R48" (at 106.68 66.04 90)
+    (property "Reference" "R49" (at 106.68 66.04 90)
       (effects (font (size 1.27 1.27)))
     )
@@
       (project "KLST_PANDA"
         (path "/b4513875-4c57-4720-bcc5-43ead67fe18f/98dcce4c-cc8c-420d-bfb6-73762da3b881"
-          (reference "R48") (unit 1)
-        )
-      )
+          (reference "R49") (unit 1)
+        )
+      )

Commit message: started updating PCB
Parts:
- renumbered J3 to J11, J3 to J12
Changed lines of the file:
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@@
   (symbol (lib_id "power:GND") (at 98.425 93.345 0) (unit 1)
     (in_bom yes) (on_board yes) (dnp no) (fields_autoplaced)
-    (property "Reference" "#PWR03" (at 98.425 99.695 0)
+    (property "Reference" "#PWR076" (at 98.425 99.695 0)
       (effects (font (size 1.27 1.27)) hide)
     )
@@
     (instances
       (project "KLST_PANDA"
-        (path "/b4513875-4c57-4720-bcc5-43ead67fe18f"
-          (reference "#PWR03") (unit 1)
-        )
-        (path "/b4513875-4c57-4720-bcc5-43ead67fe18f/f33ecd0b-aa1f-4f6b-afec-a5b478ff75fd"
-          (reference "#PWR02") (unit 1)
-        )
         (path "/b4513875-4c57-4720-bcc5-43ead67fe18f/98dcce4c-cc8c-420d-bfb6-73762da3b881"
           (reference "#PWR076") (unit 1)
@@
   (symbol (lib_id "power:GND") (at 36.83 90.17 0) (mirror y) (unit 1)
     (in_bom yes) (on_board yes) (dnp no) (fields_autoplaced)
-    (property "Reference" "#PWR03" (at 36.83 96.52 0)
+    (property "Reference" "#PWR074" (at 36.83 96.52 0)
       (effects (font (size 1.27 1.27)) hide)
     )
@@
     (instances
       (project "KLST_PANDA"
-        (path "/b4513875-4c57-4720-bcc5-43ead67fe18f"
-          (reference "#PWR03") (unit 1)
-        )
-        (path "/b4513875-4c57-4720-bcc5-43ead67fe18f/f33ecd0b-aa1f-4f6b-afec-a5b478ff75fd"
-          (reference "#PWR02") (unit 1)
-        )
         (path "/b4513875-4c57-4720-bcc5-43ead67fe18f/98dcce4c-cc8c-420d-bfb6-73762da3b881"
           (reference "#PWR074") (unit 1)
@@
   (symbol (lib_id "power:GND") (at 36.83 45.72 0) (mirror y) (unit 1)
     (in_bom yes) (on_board yes) (dnp no) (fields_autoplaced)
-    (property "Reference" "#PWR03" (at 36.83 52.07 0)
+    (property "Reference" "#PWR073" (at 36.83 52.07 0)
       (effects (font (size 1.27 1.27)) hide)
     )
@@
     (instances
       (project "KLST_PANDA"
-        (path "/b4513875-4c57-4720-bcc5-43ead67fe18f"
-          (reference "#PWR03") (unit 1)
-        )
-        (path "/b4513875-4c57-4720-bcc5-43ead67fe18f/f33ecd0b-aa1f-4f6b-afec-a5b478ff75fd"
-          (reference "#PWR02") (unit 1)
-        )
         (path "/b4513875-4c57-4720-bcc5-43ead67fe18f/98dcce4c-cc8c-420d-bfb6-73762da3b881"
           (reference "#PWR073") (unit 1)
@@
       )
       (project "KLST_PANDA"
-        (path "/b4513875-4c57-4720-bcc5-43ead67fe18f/8093d0e6-fdc1-46b4-b622-445b9f3a15e0/8f837d10-8dfd-4ab5-9b60-26a38e53480d"
-          (reference "D8") (unit 1)
-        )
-        (path "/b4513875-4c57-4720-bcc5-43ead67fe18f/8093d0e6-fdc1-46b4-b622-445b9f3a15e0/91fd47dd-a581-4f6b-aa29-abb0b8099e11"
-          (reference "D9") (unit 1)
-        )
         (path "/b4513875-4c57-4720-bcc5-43ead67fe18f/98dcce4c-cc8c-420d-bfb6-73762da3b881"
           (reference "D14") (unit 1)
@@
   (symbol (lib_id "Connector_Audio:AudioJack4_SwitchTR1") (at 29.845 83.185 0) (mirror x) (unit 1)
     (in_bom yes) (on_board yes) (dnp no)
-    (property "Reference" "J3" (at 20.955 80.645 0)
+    (property "Reference" "J12" (at 20.955 80.645 0)
       (effects (font (size 1.27 1.27)) (justify right))
     )
@@
     (instances
       (project "KLST_PANDA"
-        (path "/b4513875-4c57-4720-bcc5-43ead67fe18f/88042be3-8ae4-47d6-9c31-0a9af833bdb2"
-          (reference "J3") (unit 1)
-        )
         (path "/b4513875-4c57-4720-bcc5-43ead67fe18f/98dcce4c-cc8c-420d-bfb6-73762da3b881"
           (reference "J12") (unit 1)
@@
   (symbol (lib_id "Connector_Audio:AudioJack4_SwitchTR1") (at 29.845 38.735 0) (mirror x) (unit 1)
     (in_bom yes) (on_board yes) (dnp no)
-    (property "Reference" "J3" (at 20.955 36.195 0)
+    (property "Reference" "J11" (at 20.955 36.195 0)
       (effects (font (size 1.27 1.27)) (justify right))
     )
@@
     (instances
       (project "KLST_PANDA"
-        (path "/b4513875-4c57-4720-bcc5-43ead67fe18f/88042be3-8ae4-47d6-9c31-0a9af833bdb2"
-          (reference "J3") (unit 1)
-        )
         (path "/b4513875-4c57-4720-bcc5-43ead67fe18f/98dcce4c-cc8c-420d-bfb6-73762da3b881"
           (reference "J11") (unit 1)
