File: KLST_PANDA/external_memory.kicad_sch (KiCad schematic)
At the start: 16 parts, among them IC2 S70KL1282

Commit message: resolved TODOs
Parts:
- IC2: footprint S70KL1282:BGA24C100P5X5_600X800X100 -> BGA24C100P5X5_600X800X100
Other:
- note removed: "@TODO(check if 33R are necessary as used in MB1520)"
Changed lines of the file:
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@@
-    (effects (font (size 1.27 1.27)) (justify left bottom))
-  )
-  (text "@TODO(check if 33R are necessary as used in MB1520)"
-    (at 20.955 24.13 0)
     (effects (font (size 1.27 1.27)) (justify left bottom))
   )
@@
   (symbol (lib_id "S70KL1282:S70KL1282") (at 66.04 38.735 0) (unit 1)
     (in_bom yes) (on_board yes) (dnp no) (fields_autoplaced)
-    (property "Reference" "IC2" (at 82.55 32.385 0)
+    (property "Reference" "IC2" (at 82.55 31.75 0)
       (effects (font (size 1.27 1.27)))
     )
-    (property "Value" "S70KL1282" (at 82.55 34.925 0)
+    (property "Value" "S70KL1282" (at 82.55 34.29 0)
       (effects (font (size 1.27 1.27)))
     )
-    (property "Footprint" "S70KL1282:BGA24C100P5X5_600X800X100" (at 107.95 48.895 0)
+    (property "Footprint" "BGA24C100P5X5_600X800X100" (at 107.95 48.895 0)
       (effects (font (size 1.27 1.27)) (justify left) hide)
     )
@@
         )
         (path "/b4513875-4c57-4720-bcc5-43ead67fe18f/f33ecd0b-aa1f-4f6b-afec-a5b478ff75fd"
-          (reference "IC2") (unit 1)
-        )
-      )
+          (reference "U11") (unit 1)
+        )
+      )

Commit message: started spec'ing components
Parts:
- C1, C2, C3: JLCPCB (none) -> C1525; LCSC C1525 -> (none)
- IC2: footprint BGA24C100P5X5_600X800X100 -> S70KL1282:BGA24C100P5X5_600X800X100
- R1: footprint Resistor_SMD:R_0603_1608Metric -> Resistor_SMD:R_0402_1005Metric; JLCPCB (none) -> C25744
- R3: JLCPCB (none) -> C125766; LCSC C125766 -> (none)
Changed lines of the file:
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@@
       (effects (font (size 1.27 1.27)) hide)
     )
-    (property "LCSC" "C125766" (at 109.22 56.515 0)
+    (property "LCSC" "" (at 109.22 56.515 0)
+      (effects (font (size 1.27 1.27)) hide)
+    )
+    (property "JLCPCB" "C125766" (at 109.22 56.515 0)
       (effects (font (size 1.27 1.27)) hide)
     )
@@
       (effects (font (size 1.27 1.27)) hide)
     )
-    (property "LCSC" "C125766" (at 53.34 41.275 0)
+    (property "LCSC" "" (at 53.34 41.275 0)
+      (effects (font (size 1.27 1.27)) hide)
+    )
+    (property "JLCPCB" "C125766" (at 53.34 41.275 0)
       (effects (font (size 1.27 1.27)) hide)
     )
@@
       (effects (font (size 1.27 1.27)) hide)
     )
-    (property "LCSC" "C125766" (at 53.34 66.675 0)
+    (property "LCSC" "" (at 53.34 66.675 0)
+      (effects (font (size 1.27 1.27)) hide)
+    )
+    (property "JLCPCB" "C125766" (at 53.34 66.675 0)
       (effects (font (size 1.27 1.27)) hide)
     )
@@
       (effects (font (size 1.27 1.27)) hide)
     )
-    (property "LCSC" "C1525" (at 107.95 78.105 0)
+    (property "LCSC" "" (at 107.95 78.105 0)
       (effects (font (size 1.27 1.27)) hide)
     )
     (property "Extended Part" "-" (at 107.95 78.105 0)
+      (effects (font (size 1.27 1.27)) hide)
+    )
+    (property "JLCPCB" "C1525" (at 107.95 78.105 0)
+      (effects (font (size 1.27 1.27)) hide)
+    )
+    (property "Description" "16V" (at 107.95 78.105 0)
       (effects (font (size 1.27 1.27)) hide)
     )
@@
       (effects (font (size 1.27 1.27)) hide)
     )
-    (property "LCSC" "C1525" (at 130.81 78.105 0)
+    (property "LCSC" "" (at 130.81 78.105 0)
       (effects (font (size 1.27 1.27)) hide)
     )
@@
       (effects (font (size 1.27 1.27)) hide)
     )
+    (property "JLCPCB" "C1525" (at 130.81 78.105 0)
+      (effects (font (size 1.27 1.27)) hide)
+    )
+    (property "Description" "16V" (at 130.81 78.105 0)
+      (effects (font (size 1.27 1.27)) hide)
+    )
     (pin "1")
     (pin "2")
@@
       (effects (font (size 1.27 1.27)) hide)
     )
-    (property "LCSC" "C125766" (at 109.22 46.355 0)
+    (property "LCSC" "" (at 109.22 46.355 0)
+      (effects (font (size 1.27 1.27)) hide)
+    )
+    (property "JLCPCB" "C125766" (at 109.22 46.355 0)
       (effects (font (size 1.27 1.27)) hide)
     )
@@
       (effects (font (size 1.27 1.27)) hide)
     )
-    (property "LCSC" "C125766" (at 109.22 61.595 0)
+    (property "LCSC" "" (at 109.22 61.595 0)
+      (effects (font (size 1.27 1.27)) hide)
+    )
+    (property "JLCPCB" "C125766" (at 109.22 61.595 0)
       (effects (font (size 1.27 1.27)) hide)
     )
@@
       (effects (font (size 1.27 1.27)) hide)
     )
-    (property "LCSC" "C125766" (at 109.22 48.895 0)
+    (property "LCSC" "" (at 109.22 48.895 0)
+      (effects (font (size 1.27 1.27)) hide)
+    )
+    (property "JLCPCB" "C125766" (at 109.22 48.895 0)
       (effects (font (size 1.27 1.27)) hide)
     )
@@
       (effects (font (size 1.27 1.27)) hide)
     )
-    (property "LCSC" "C1525" (at 119.38 78.105 0)
+    (property "LCSC" "" (at 119.38 78.105 0)
       (effects (font (size 1.27 1.27)) hide)
     )
@@
       (effects (font (size 1.27 1.27)) hide)
     )
+    (property "JLCPCB" "C1525" (at 119.38 78.105 0)
+      (effects (font (size 1.27 1.27)) hide)
+    )
+    (property "Description" "16V" (at 119.38 78.105 0)
+      (effects (font (size 1.27 1.27)) hide)
+    )
     (pin "1")
     (pin "2")
@@
       (effects (font (size 1.27 1.27)) hide)
     )
-    (property "LCSC" "C125766" (at 109.22 59.055 0)
+    (property "LCSC" "" (at 109.22 59.055 0)
+      (effects (font (size 1.27 1.27)) hide)
+    )
+    (property "JLCPCB" "C125766" (at 109.22 59.055 0)
       (effects (font (size 1.27 1.27)) hide)
     )
@@
       (effects (font (size 1.27 1.27)) (justify right))
     )
-    (property "Footprint" "Resistor_SMD:R_0603_1608Metric" (at 62.23 33.655 0)
+    (property "Footprint" "Resistor_SMD:R_0402_1005Metric" (at 62.23 33.655 0)
       (effects (font (size 1.27 1.27)) hide)
     )
@@
       (effects (font (size 1.27 1.27)) hide)
     )
+    (property "JLCPCB" "C25744" (at 62.23 33.655 0)
+      (effects (font (size 1.27 1.27)) hide)
+    )
     (pin "1")
     (pin "2")
@@
       (effects (font (size 1.27 1.27)) hide)
     )
-    (property "LCSC" "C125766" (at 109.22 38.735 0)
+    (property "LCSC" "" (at 109.22 38.735 0)
+      (effects (font (size 1.27 1.27)) hide)
+    )
+    (property "JLCPCB" "C125766" (at 109.22 38.735 0)
       (effects (font (size 1.27 1.27)) hide)
     )
@@
       (effects (font (size 1.27 1.27)))
     )
-    (property "Footprint" "BGA24C100P5X5_600X800X100" (at 107.95 48.895 0)
+    (property "Footprint" "S70KL1282:BGA24C100P5X5_600X800X100" (at 107.95 48.895 0)
       (effects (font (size 1.27 1.27)) (justify left) hide)
     )
@@
       (effects (font (size 1.27 1.27)) hide)
     )
-    (property "LCSC" "C125766" (at 109.22 51.435 0)
+    (property "LCSC" "" (at 109.22 51.435 0)
+      (effects (font (size 1.27 1.27)) hide)
+    )
+    (property "JLCPCB" "C125766" (at 109.22 51.435 0)
       (effects (font (size 1.27 1.27)) hide)
     )
@@
       (effects (font (size 1.27 1.27)) hide)
     )
-    (property "LCSC" "C125766" (at 109.22 53.975 0)
+    (property "LCSC" "" (at 109.22 53.975 0)
+      (effects (font (size 1.27 1.27)) hide)
+    )
+    (property "JLCPCB" "C125766" (at 109.22 53.975 0)
       (effects (font (size 1.27 1.27)) hide)
     )
@@
       (effects (font (size 1.27 1.27)) hide)
     )
-    (property "LCSC" "C125766" (at 53.34 51.435 0)
-      (effects (font (size 1.27 1.27)) hide)
-    )
+    (property "LCSC" "" (at 53.34 51.435 0)
+      (effects (font (size 1.27 1.27)) hide)
+    )
+    (property "JLCPCB" "C125766" (at 53.34 51.435 0)
+      (effects (font (size 1.27 1.27)) hide)
+    )

Commit message: assigned footprints
Parts:
- IC2: JLCPCB (none) -> C7428856
- R3: footprint Resistor_SMD:R_0603_1608Metric -> Resistor_SMD:R_0402_1005Metric; JLCPCB C125766 -> C138002
Changed lines of the file:
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@@
       (effects (font (size 1.27 1.27)) (justify right top))
     )
-    (property "Footprint" "Resistor_SMD:R_0603_1608Metric" (at 109.22 56.515 0)
+    (property "Footprint" "Resistor_SMD:R_0402_1005Metric" (at 109.22 56.515 0)
       (effects (font (size 1.27 1.27)) hide)
     )
@@
       (effects (font (size 1.27 1.27)) hide)
     )
-    (property "JLCPCB" "C125766" (at 109.22 56.515 0)
+    (property "JLCPCB" "C138002" (at 109.22 56.515 0)
+      (effects (font (size 1.27 1.27)) hide)
+    )
+    (property "Description" "62.5mW" (at 109.22 56.515 0)
       (effects (font (size 1.27 1.27)) hide)
     )
@@
       (effects (font (size 1.27 1.27)) (justify right top))
     )
-    (property "Footprint" "Resistor_SMD:R_0603_1608Metric" (at 53.34 41.275 0)
+    (property "Footprint" "Resistor_SMD:R_0402_1005Metric" (at 53.34 41.275 0)
       (effects (font (size 1.27 1.27)) hide)
     )
@@
       (effects (font (size 1.27 1.27)) hide)
     )
-    (property "JLCPCB" "C125766" (at 53.34 41.275 0)
+    (property "JLCPCB" "C138002" (at 53.34 41.275 0)
+      (effects (font (size 1.27 1.27)) hide)
+    )
+    (property "Description" "62.5mW" (at 53.34 41.275 0)
       (effects (font (size 1.27 1.27)) hide)
     )
@@
       (effects (font (size 1.27 1.27)) (justify right top))
     )
-    (property "Footprint" "Resistor_SMD:R_0603_1608Metric" (at 53.34 66.675 0)
+    (property "Footprint" "Resistor_SMD:R_0402_1005Metric" (at 53.34 66.675 0)
       (effects (font (size 1.27 1.27)) hide)
     )
@@
       (effects (font (size 1.27 1.27)) hide)
     )
-    (property "JLCPCB" "C125766" (at 53.34 66.675 0)
+    (property "JLCPCB" "C138002" (at 53.34 66.675 0)
+      (effects (font (size 1.27 1.27)) hide)
+    )
+    (property "Description" "62.5mW" (at 53.34 66.675 0)
       (effects (font (size 1.27 1.27)) hide)
     )
@@
       (effects (font (size 1.27 1.27)) (justify right top))
     )
-    (property "Footprint" "Resistor_SMD:R_0603_1608Metric" (at 109.22 46.355 0)
+    (property "Footprint" "Resistor_SMD:R_0402_1005Metric" (at 109.22 46.355 0)
       (effects (font (size 1.27 1.27)) hide)
     )
@@
       (effects (font (size 1.27 1.27)) hide)
     )
-    (property "JLCPCB" "C125766" (at 109.22 46.355 0)
+    (property "JLCPCB" "C138002" (at 109.22 46.355 0)
+      (effects (font (size 1.27 1.27)) hide)
+    )
+    (property "Description" "62.5mW" (at 109.22 46.355 0)
       (effects (font (size 1.27 1.27)) hide)
     )
@@
       (effects (font (size 1.27 1.27)) (justify right top))
     )
-    (property "Footprint" "Resistor_SMD:R_0603_1608Metric" (at 109.22 61.595 0)
+    (property "Footprint" "Resistor_SMD:R_0402_1005Metric" (at 109.22 61.595 0)
       (effects (font (size 1.27 1.27)) hide)
     )
@@
       (effects (font (size 1.27 1.27)) hide)
     )
-    (property "JLCPCB" "C125766" (at 109.22 61.595 0)
+    (property "JLCPCB" "C138002" (at 109.22 61.595 0)
+      (effects (font (size 1.27 1.27)) hide)
+    )
+    (property "Description" "62.5mW" (at 109.22 61.595 0)
       (effects (font (size 1.27 1.27)) hide)
     )
@@
       (effects (font (size 1.27 1.27)) (justify right top))
     )
-    (property "Footprint" "Resistor_SMD:R_0603_1608Metric" (at 109.22 48.895 0)
+    (property "Footprint" "Resistor_SMD:R_0402_1005Metric" (at 109.22 48.895 0)
       (effects (font (size 1.27 1.27)) hide)
     )
@@
       (effects (font (size 1.27 1.27)) hide)
     )
-    (property "JLCPCB" "C125766" (at 109.22 48.895 0)
+    (property "JLCPCB" "C138002" (at 109.22 48.895 0)
+      (effects (font (size 1.27 1.27)) hide)
+    )
+    (property "Description" "62.5mW" (at 109.22 48.895 0)
       (effects (font (size 1.27 1.27)) hide)
     )
@@
       (effects (font (size 1.27 1.27)) (justify right top))
     )
-    (property "Footprint" "Resistor_SMD:R_0603_1608Metric" (at 109.22 59.055 0)
+    (property "Footprint" "Resistor_SMD:R_0402_1005Metric" (at 109.22 59.055 0)
       (effects (font (size 1.27 1.27)) hide)
     )
@@
       (effects (font (size 1.27 1.27)) hide)
     )
-    (property "JLCPCB" "C125766" (at 109.22 59.055 0)
+    (property "JLCPCB" "C138002" (at 109.22 59.055 0)
+      (effects (font (size 1.27 1.27)) hide)
+    )
+    (property "Description" "62.5mW" (at 109.22 59.055 0)
       (effects (font (size 1.27 1.27)) hide)
     )
@@
       (effects (font (size 1.27 1.27)) hide)
     )
+    (property "Description" "62.5mW" (at 62.23 33.655 0)
+      (effects (font (size 1.27 1.27)) hide)
+    )
     (pin "1")
     (pin "2")
@@
       (effects (font (size 1.27 1.27)) (justify right top))
     )
-    (property "Footprint" "Resistor_SMD:R_0603_1608Metric" (at 109.22 38.735 0)
+    (property "Footprint" "Resistor_SMD:R_0402_1005Metric" (at 109.22 38.735 0)
       (effects (font (size 1.27 1.27)) hide)
     )
@@
       (effects (font (size 1.27 1.27)) hide)
     )
-    (property "JLCPCB" "C125766" (at 109.22 38.735 0)
+    (property "JLCPCB" "C138002" (at 109.22 38.735 0)
+      (effects (font (size 1.27 1.27)) hide)
+    )
+    (property "Description" "62.5mW" (at 109.22 38.735 0)
       (effects (font (size 1.27 1.27)) hide)
     )
@@
       (effects (font (size 1.27 1.27)) (justify left) hide)
     )
-    (property "Description" "DRAM Chip DDR SDRAM 128Mbit 16Mx8 3V/3.3V 24-Pin Fortified BGA T/R" (at 107.95 53.975 0)
+    (property "Description" "S70KL1282GABHV020" (at 107.95 53.975 0)
       (effects (font (size 1.27 1.27)) (justify left) hide)
     )
@@
     (property "Manufacturer_Part_Number" "S70KL1282GABHV020" (at 107.95 61.595 0)
       (effects (font (size 1.27 1.27)) (justify left) hide)
+    )
+    (property "JLCPCB" "C7428856" (at 66.04 38.735 0)
+      (effects (font (size 1.27 1.27)) hide)
     )
     (pin "A2")
@@
       (effects (font (size 1.27 1.27)) (justify right top))
     )
-    (property "Footprint" "Resistor_SMD:R_0603_1608Metric" (at 109.22 51.435 0)
+    (property "Footprint" "Resistor_SMD:R_0402_1005Metric" (at 109.22 51.435 0)
       (effects (font (size 1.27 1.27)) hide)
     )
@@
       (effects (font (size 1.27 1.27)) hide)
     )
-    (property "JLCPCB" "C125766" (at 109.22 51.435 0)
+    (property "JLCPCB" "C138002" (at 109.22 51.435 0)
+      (effects (font (size 1.27 1.27)) hide)
+    )
+    (property "Description" "62.5mW" (at 109.22 51.435 0)
       (effects (font (size 1.27 1.27)) hide)
     )
@@
       (effects (font (size 1.27 1.27)) (justify right top))
     )
-    (property "Footprint" "Resistor_SMD:R_0603_1608Metric" (at 109.22 53.975 0)
+    (property "Footprint" "Resistor_SMD:R_0402_1005Metric" (at 109.22 53.975 0)
       (effects (font (size 1.27 1.27)) hide)
     )
@@
       (effects (font (size 1.27 1.27)) hide)
     )
-    (property "JLCPCB" "C125766" (at 109.22 53.975 0)
+    (property "JLCPCB" "C138002" (at 109.22 53.975 0)
+      (effects (font (size 1.27 1.27)) hide)
+    )
+    (property "Description" "62.5mW" (at 109.22 53.975 0)
       (effects (font (size 1.27 1.27)) hide)
     )
@@
       (effects (font (size 1.27 1.27)) (justify right top))
     )
-    (property "Footprint" "Resistor_SMD:R_0603_1608Metric" (at 53.34 51.435 0)
+    (property "Footprint" "Resistor_SMD:R_0402_1005Metric" (at 53.34 51.435 0)
       (effects (font (size 1.27 1.27)) hide)
     )
@@
       (effects (font (size 1.27 1.27)) hide)
     )
-    (property "JLCPCB" "C125766" (at 53.34 51.435 0)
-      (effects (font (size 1.27 1.27)) hide)
-    )
+    (property "JLCPCB" "C138002" (at 53.34 51.435 0)
+      (effects (font (size 1.27 1.27)) hide)
+    )
+    (property "Description" "62.5mW" (at 53.34 51.435 0)
+      (effects (font (size 1.27 1.27)) hide)
+    )

Commit message: cleaned up footprint assignment
Parts:
- C1, C2, C3: Extended Part - -> (none)
- IC2: Height 1 -> (none); Manufacturer_Name Infinion -> (none); Manufacturer_Part_Number S70KL1282GABHV020 -> (none)
Changed lines of the file:
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@@
-      (effects (font (size 1.27 1.27)) hide)
-    )
-    (property "LCSC" "" (at 109.22 56.515 0)
       (effects (font (size 1.27 1.27)) hide)
     )
@@
       (effects (font (size 1.27 1.27)) hide)
     )
-    (property "LCSC" "" (at 53.34 41.275 0)
-      (effects (font (size 1.27 1.27)) hide)
-    )
     (property "JLCPCB" "C138002" (at 53.34 41.275 0)
       (effects (font (size 1.27 1.27)) hide)
@@
     )
     (property "Datasheet" "~" (at 53.34 66.675 0)
-      (effects (font (size 1.27 1.27)) hide)
-    )
-    (property "LCSC" "" (at 53.34 66.675 0)
       (effects (font (size 1.27 1.27)) hide)
     )
@@
       (effects (font (size 1.27 1.27)) hide)
     )
-    (property "LCSC" "" (at 107.95 78.105 0)
-      (effects (font (size 1.27 1.27)) hide)
-    )
-    (property "Extended Part" "-" (at 107.95 78.105 0)
-      (effects (font (size 1.27 1.27)) hide)
-    )
     (property "JLCPCB" "C1525" (at 107.95 78.105 0)
       (effects (font (size 1.27 1.27)) hide)
@@
       (effects (font (size 1.27 1.27)) hide)
     )
-    (property "LCSC" "" (at 130.81 78.105 0)
-      (effects (font (size 1.27 1.27)) hide)
-    )
-    (property "Extended Part" "-" (at 130.81 78.105 0)
-      (effects (font (size 1.27 1.27)) hide)
-    )
     (property "JLCPCB" "C1525" (at 130.81 78.105 0)
       (effects (font (size 1.27 1.27)) hide)
@@
     )
     (property "Datasheet" "~" (at 109.22 46.355 0)
-      (effects (font (size 1.27 1.27)) hide)
-    )
-    (property "LCSC" "" (at 109.22 46.355 0)
       (effects (font (size 1.27 1.27)) hide)
     )
@@
       (effects (font (size 1.27 1.27)) hide)
     )
-    (property "LCSC" "" (at 109.22 61.595 0)
-      (effects (font (size 1.27 1.27)) hide)
-    )
     (property "JLCPCB" "C138002" (at 109.22 61.595 0)
       (effects (font (size 1.27 1.27)) hide)
@@
     )
     (property "Datasheet" "~" (at 109.22 48.895 0)
-      (effects (font (size 1.27 1.27)) hide)
-    )
-    (property "LCSC" "" (at 109.22 48.895 0)
       (effects (font (size 1.27 1.27)) hide)
     )
@@
       (effects (font (size 1.27 1.27)) hide)
     )
-    (property "LCSC" "" (at 119.38 78.105 0)
-      (effects (font (size 1.27 1.27)) hide)
-    )
-    (property "Extended Part" "-" (at 119.38 78.105 0)
-      (effects (font (size 1.27 1.27)) hide)
-    )
     (property "JLCPCB" "C1525" (at 119.38 78.105 0)
       (effects (font (size 1.27 1.27)) hide)
@@
     )
     (property "Datasheet" "~" (at 109.22 59.055 0)
-      (effects (font (size 1.27 1.27)) hide)
-    )
-    (property "LCSC" "" (at 109.22 59.055 0)
       (effects (font (size 1.27 1.27)) hide)
     )
@@
     )
     (property "Datasheet" "~" (at 109.22 38.735 0)
-      (effects (font (size 1.27 1.27)) hide)
-    )
-    (property "LCSC" "" (at 109.22 38.735 0)
       (effects (font (size 1.27 1.27)) hide)
     )
@@
     )
     (property "Description" "S70KL1282GABHV020" (at 107.95 53.975 0)
-      (effects (font (size 1.27 1.27)) (justify left) hide)
-    )
-    (property "Height" "1" (at 95.25 43.815 0)
-      (effects (font (size 1.27 1.27)) (justify left) hide)
-    )
-    (property "Manufacturer_Name" "Infinion" (at 107.95 59.055 0)
-      (effects (font (size 1.27 1.27)) (justify left) hide)
-    )
-    (property "Manufacturer_Part_Number" "S70KL1282GABHV020" (at 107.95 61.595 0)
       (effects (font (size 1.27 1.27)) (justify left) hide)
     )
@@
       (effects (font (size 1.27 1.27)) hide)
     )
-    (property "LCSC" "" (at 109.22 51.435 0)
-      (effects (font (size 1.27 1.27)) hide)
-    )
     (property "JLCPCB" "C138002" (at 109.22 51.435 0)
       (effects (font (size 1.27 1.27)) hide)
@@
       (effects (font (size 1.27 1.27)) hide)
     )
-    (property "LCSC" "" (at 109.22 53.975 0)
-      (effects (font (size 1.27 1.27)) hide)
-    )
     (property "JLCPCB" "C138002" (at 109.22 53.975 0)
       (effects (font (size 1.27 1.27)) hide)
@@
       (effects (font (size 1.27 1.27)) hide)
     )
-    (property "LCSC" "" (at 53.34 51.435 0)
-      (effects (font (size 1.27 1.27)) hide)
-    )

Commit message: started updating PCB
Parts:
- renumbered C1 to C54, C2 to C55, C3 to C56, R3 to R60, R3 to R61, R3 to R62, R1 to R63, R3 to R64, R3 to R65, R3 to R66, R3 to R67, R3 to R68, R3 to R69, R3 to R70, R3 to R71, IC2 to U12
