File: KLST_PANDA/sd_card.kicad_sch (KiCad schematic)
At the start: 9 parts, among them J1 Micro_SD_Card_Det_Hirose_DM3AT

Commit message: started updating PCB
Parts:
- renumbered C3 to C30
Changed lines of the file:
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@@
   (symbol (lib_id "power:+3.3V") (at 125.095 23.495 0) (unit 1)
     (in_bom yes) (on_board yes) (dnp no) (fields_autoplaced)
-    (property "Reference" "#PWR021" (at 125.095 27.305 0)
+    (property "Reference" "#PWR040" (at 125.095 27.305 0)
       (effects (font (size 1.27 1.27)) hide)
     )
@@
     (instances
       (project "KLST_PANDA"
-        (path "/b4513875-4c57-4720-bcc5-43ead67fe18f/88042be3-8ae4-47d6-9c31-0a9af833bdb2"
-          (reference "#PWR021") (unit 1)
-        )
         (path "/b4513875-4c57-4720-bcc5-43ead67fe18f/52cda7d1-da0e-43fc-963f-d09ac6e0ff74"
           (reference "#PWR040") (unit 1)
@@
       )
       (project "KLST_PANDA"
-        (path "/b4513875-4c57-4720-bcc5-43ead67fe18f/f08ee185-46fd-4c64-8c0d-73017bc497ee/7936a5e0-5a04-43e4-aa84-42432289d154"
+        (path "/b4513875-4c57-4720-bcc5-43ead67fe18f/52cda7d1-da0e-43fc-963f-d09ac6e0ff74"
           (reference "#PWR039") (unit 1)
         )
-        (path "/b4513875-4c57-4720-bcc5-43ead67fe18f/52cda7d1-da0e-43fc-963f-d09ac6e0ff74"
-          (reference "#PWR039") (unit 1)
-        )
       )
     )
@@
   (symbol (lib_id "power:+3.3V") (at 24.765 23.495 0) (unit 1)
     (in_bom yes) (on_board yes) (dnp no) (fields_autoplaced)
-    (property "Reference" "#PWR021" (at 24.765 27.305 0)
+    (property "Reference" "#PWR038" (at 24.765 27.305 0)
       (effects (font (size 1.27 1.27)) hide)
     )
@@
     (instances
       (project "KLST_PANDA"
-        (path "/b4513875-4c57-4720-bcc5-43ead67fe18f/88042be3-8ae4-47d6-9c31-0a9af833bdb2"
-          (reference "#PWR021") (unit 1)
-        )
         (path "/b4513875-4c57-4720-bcc5-43ead67fe18f/52cda7d1-da0e-43fc-963f-d09ac6e0ff74"
           (reference "#PWR038") (unit 1)
@@
   (symbol (lib_id "power:GND") (at 161.29 92.71 0) (unit 1)
     (in_bom yes) (on_board yes) (dnp no)
-    (property "Reference" "#PWR07" (at 161.29 99.06 0)
+    (property "Reference" "#PWR041" (at 161.29 99.06 0)
       (effects (font (size 1.27 1.27)) hide)
     )
@@
     (instances
       (project "KLST_PANDA"
-        (path "/b4513875-4c57-4720-bcc5-43ead67fe18f"
-          (reference "#PWR07") (unit 1)
-        )
         (path "/b4513875-4c57-4720-bcc5-43ead67fe18f/52cda7d1-da0e-43fc-963f-d09ac6e0ff74"
           (reference "#PWR041") (unit 1)
@@
   (symbol (lib_id "Device:C_Small") (at 127 75.565 0) (unit 1)
     (in_bom yes) (on_board yes) (dnp no)
-    (property "Reference" "C3" (at 129.3368 74.3966 0)
+    (property "Reference" "C30" (at 129.3368 74.3966 0)
       (effects (font (size 1.27 1.27)) (justify left))
     )
@@
     (instances
       (project "KLST_PANDA"
-        (path "/b4513875-4c57-4720-bcc5-43ead67fe18f"
-          (reference "C3") (unit 1)
-        )
-        (path "/b4513875-4c57-4720-bcc5-43ead67fe18f/d68846c2-d235-4363-b980-eab3c53b4a55"
-          (reference "C6") (unit 1)
-        )
         (path "/b4513875-4c57-4720-bcc5-43ead67fe18f/52cda7d1-da0e-43fc-963f-d09ac6e0ff74"
           (reference "C30") (unit 1)
@@
       )
       (project "KLST_PANDA"
-        (path "/b4513875-4c57-4720-bcc5-43ead67fe18f/f08ee185-46fd-4c64-8c0d-73017bc497ee/7936a5e0-5a04-43e4-aa84-42432289d154"
-          (reference "R62") (unit 1)
-        )
         (path "/b4513875-4c57-4720-bcc5-43ead67fe18f/52cda7d1-da0e-43fc-963f-d09ac6e0ff74"
           (reference "R12") (unit 1)
