File: KLST_CATERPILLAR/buttons_keys.kicad_sch (KiCad schematic)
At the start: 0 parts

Commit message: reduced modules
Other:
- removed sheet MECHANICAL_KEY_00
- removed sheet MECHANICAL_KEY_01
Changed lines of the file:
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@@
-		)
-	)
-	(global_label "_MECH_BUTTON_00"
-		(shape input)
-		(at 42.545 35.56 180)
-		(fields_autoplaced yes)
-		(effects
-			(font
-				(size 1.27 1.27)
-			)
-			(justify right)
-		)
-		(property "Intersheetrefs" "${INTERSHEET_REFS}"
-			(at 21.9198 35.56 0)
-			(effects
-				(font
-					(size 1.27 1.27)
-				)
-				(justify right)
-				(hide yes)
-			)
-		)
-	)
-	(global_label "_MECH_BUTTON_01"
-		(shape input)
-		(at 42.545 46.99 180)
-		(fields_autoplaced yes)
-		(effects
-			(font
-				(size 1.27 1.27)
-			)
-			(justify right)
-		)
-		(property "Intersheetrefs" "${INTERSHEET_REFS}"
-			(at 21.9198 46.99 0)
-			(effects
-				(font
-					(size 1.27 1.27)
-				)
-				(justify right)
-				(hide yes)
-			)
 		)
 	)
@@
 				(justify right)
 				(hide yes)
-			)
-		)
-	)
-	(sheet
-		(at 42.545 33.02)
-		(size 34.29 5.08)
-		(fields_autoplaced yes)
-		(stroke
-			(width 0.1524)
-			(type solid)
-		)
-		(fill
-			(color 0 0 0 0.0000)
-		)
-		(property "Sheetname" "MECHANICAL_KEY_00"
-			(at 42.545 32.3084 0)
-			(effects
-				(font
-					(size 1.27 1.27)
-				)
-				(justify left bottom)
-			)
-		)
-		(property "Sheetfile" "mechanical_key.kicad_sch"
-			(at 42.545 38.6846 0)
-			(effects
-				(font
-					(size 1.27 1.27)
-				)
-				(justify left top)
-			)
-		)
-		(pin "KEY" input
-			(at 42.545 35.56 180)
-			(effects
-				(font
-					(size 1.27 1.27)
-				)
-				(justify left)
-			)
-		)
-		(instances
-			(project "KLST_CATERPILLAR"
-				(path "/b4513875-4c57-4720-bcc5-43ead67fe18f/f08ee185-46fd-4c64-8c0d-73017bc497ee"
-					(page "21")
-				)
 			)
 		)
@@
 				)
 			)
-		)
-	)
-	(sheet
-		(at 42.545 44.45)
-		(size 34.29 5.08)
-		(fields_autoplaced yes)
-		(stroke
-			(width 0.1524)
-			(type solid)
-		)
-		(fill
-			(color 0 0 0 0.0000)
-		)
-		(property "Sheetname" "MECHANICAL_KEY_01"
-			(at 42.545 43.7384 0)
-			(effects
-				(font
-					(size 1.27 1.27)
-				)
-				(justify left bottom)
-			)
-		)
-		(property "Sheetfile" "mechanical_key.kicad_sch"
-			(at 42.545 50.1146 0)
-			(effects
-				(font
-					(size 1.27 1.27)
-				)
-				(justify left top)
-			)
-		)
-		(pin "KEY" input
-			(at 42.545 46.99 180)
-			(effects
-				(font
-					(size 1.27 1.27)
-				)
-				(justify left)
-			)
-		)
-		(instances
-			(project "KLST_CATERPILLAR"
-				(path "/b4513875-4c57-4720-bcc5-43ead67fe18f/f08ee185-46fd-4c64-8c0d-73017bc497ee"
-					(page "22")
-				)
-			)
