File: KLST_CATERPILLAR/IDC_serial.kicad_sch (KiCad schematic)
At the start: 2 parts, among them J13 UART

Commit message: reduced modules
Parts:
- J13: footprint Connector_IDC:IDC-Header_2x03_P2.54mm_Horizontal -> Connector_IDC:IDC-Header_2x03_P2.54mm_Vertical_SMD; JLCPCB C146629 -> C720733
Other:
- note removed: "@TODO(maybe replace THT with SMD connector e.g C720733 )"
Changed lines of the file:
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@@
 		)
 	)
-	(text "@TODO(maybe replace THT with SMD connector e.g C720733 )"
-		(exclude_from_sim no)
-		(at 121.92 123.19 0)
+	(text_box "@TODO(replaced THT with SMD connector C720733. check with footprint)"
+		(exclude_from_sim no)
+		(at 103.505 119.38 0)
+		(size 113.665 40.005)
+		(stroke
+			(width -0.0001)
+			(type default)
+		)
+		(fill
+			(type color)
+			(color 255 0 0 1)
+		)
 		(effects
 			(font
-				(size 1.27 1.27)
-			)
-			(justify left bottom)
+				(size 5.08 5.08)
+			)
+			(justify left top)
 		)
 	)
@@
 					(unit 1)
 				)
-				(path "/b4513875-4c57-4720-bcc5-43ead67fe18f/8093d0e6-fdc1-46b4-b622-445b9f3a15e0/91fd47dd-a581-4f6b-aa29-abb0b8099e11"
-					(reference "D10")
-					(unit 1)
-				)
 			)
 		)
@@
 					(unit 1)
 				)
-				(path "/b4513875-4c57-4720-bcc5-43ead67fe18f/8093d0e6-fdc1-46b4-b622-445b9f3a15e0/91fd47dd-a581-4f6b-aa29-abb0b8099e11"
-					(reference "#PWR058")
-					(unit 1)
-				)
 			)
 		)
@@
 					(unit 1)
 				)
-				(path "/b4513875-4c57-4720-bcc5-43ead67fe18f/8093d0e6-fdc1-46b4-b622-445b9f3a15e0/91fd47dd-a581-4f6b-aa29-abb0b8099e11"
-					(reference "#PWR057")
-					(unit 1)
-				)
 			)
 		)
@@
 			)
 		)
-		(property "Footprint" "Connector_IDC:IDC-Header_2x03_P2.54mm_Horizontal"
+		(property "Footprint" "Connector_IDC:IDC-Header_2x03_P2.54mm_Vertical_SMD"
 			(at 148.59 101.6 0)
 			(effects
@@
 			)
 		)
-		(property "JLCPCB" "C146629"
+		(property "JLCPCB" "C720733"
 			(at 148.59 101.6 0)
 			(effects
@@
 					(unit 1)
 				)
-				(path "/b4513875-4c57-4720-bcc5-43ead67fe18f/8093d0e6-fdc1-46b4-b622-445b9f3a15e0/91fd47dd-a581-4f6b-aa29-abb0b8099e11"
-					(reference "J6")
-					(unit 1)
-				)

Commit message: added test points, replaced unavailable components
Parts:
- J13: JLCPCB C720733 -> C492445
Changed lines of the file:
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@@
-		)
-	)
-	(text_box "@TODO(replaced THT with SMD connector C720733. check with footprint)"
-		(exclude_from_sim no)
-		(at 103.505 119.38 0)
-		(size 113.665 40.005)
-		(stroke
-			(width -0.0001)
-			(type default)
-		)
-		(fill
-			(type color)
-			(color 255 0 0 1)
-		)
-		(effects
-			(font
-				(size 5.08 5.08)
-			)
-			(justify left top)
 		)
 	)
@@
 			)
 		)
-		(property "JLCPCB" "C720733"
-			(at 148.59 101.6 0)
-			(effects
+		(property "JLCPCB" "C492445"
+			(at 148.59 101.6 0)
+			(effects
