File: KLST_CATERPILLAR/testpoints.kicad_sch (KiCad schematic)
At the start: 0 parts

Commit message: added test points, replaced unavailable components
Parts:
- added TP1: TP_AUDIO_CODEC_I2C_SCL, KLST:TestPoint_Pad_D1.5mm, symbol Connector:TestPoint_Small
- added TP10: TP_CARD_SDMMC_CMD, KLST:TestPoint_Pad_D1.5mm, symbol Connector:TestPoint_Small
- added TP11: TP_CARD_SDMMC_CK, KLST:TestPoint_Pad_D1.5mm, symbol Connector:TestPoint_Small
- added TP12: TP_CARD_SDMMC_D0, KLST:TestPoint_Pad_D1.5mm, symbol Connector:TestPoint_Small
- added TP13: TP_CARD_SDMMC_D1, KLST:TestPoint_Pad_D1.5mm, symbol Connector:TestPoint_Small
- added TP14: TP_USB_DEVICE_HOST_N, KLST:TestPoint_Pad_D1.5mm, symbol Connector:TestPoint_Small
- added TP15: TP_USB_DEVICE_HOST_P, KLST:TestPoint_Pad_D1.5mm, symbol Connector:TestPoint_Small
- added TP16: TP_AUDIO_MIC_CLK, KLST:TestPoint_Pad_D1.5mm, symbol Connector:TestPoint_Small
- added TP17: TP_AUDIO_MIC_DATA, KLST:TestPoint_Pad_D1.5mm, symbol Connector:TestPoint_Small
- added TP2: TP_AUDIO_CODEC_I2C_SCA, KLST:TestPoint_Pad_D1.5mm, symbol Connector:TestPoint_Small
- added TP3: TP_AUDIO_CODEC_SAI_MCLK, KLST:TestPoint_Pad_D1.5mm, symbol Connector:TestPoint_Small
- added TP4: TP_AUDIO_CODEC_SAI_FS, KLST:TestPoint_Pad_D1.5mm, symbol Connector:TestPoint_Small
- added TP5: TP_AUDIO_CODEC_SAI_SCK, KLST:TestPoint_Pad_D1.5mm, symbol Connector:TestPoint_Small
- added TP6: TP_AUDIO_CODEC_SAI_SD_OUT, KLST:TestPoint_Pad_D1.5mm, symbol Connector:TestPoint_Small
- added TP7: TP_AUDIO_CODEC_SAI_SD_IN, KLST:TestPoint_Pad_D1.5mm, symbol Connector:TestPoint_Small
- added TP8: TP_CARD_SDMMC_D2, KLST:TestPoint_Pad_D1.5mm, symbol Connector:TestPoint_Small
- added TP9: TP_CARD_SDMMC_D3, KLST:TestPoint_Pad_D1.5mm, symbol Connector:TestPoint_Small
Connections:
- new net _AUDIO_CODEC_I2C_SCL: TP1.1
- new net _AUDIO_CODEC_I2C_SDA: TP2.1
- new net _AUDIO_CODEC_SAI_FS: TP4.1
- new net _AUDIO_CODEC_SAI_MCLK: TP3.1
- new net _AUDIO_CODEC_SAI_SCK: TP5.1
- new net _AUDIO_CODEC_SAI_SD_IN: TP7.1
- new net _AUDIO_CODEC_SAI_SD_OUT: TP6.1
- new net _AUDIO_MIC_CLK: TP16.1
- new net _AUDIO_MIC_DATA: TP17.1
- new net _CARD_SDMMC_CK: TP11.1
- new net _CARD_SDMMC_CMD: TP10.1
- new net _CARD_SDMMC_D0: TP12.1
- new net _CARD_SDMMC_D1: TP13.1
- new net _CARD_SDMMC_D2: TP8.1
- new net _CARD_SDMMC_D3: TP9.1
- new net _USB_DEVICE_HOST_N: TP14.1
- new net _USB_DEVICE_HOST_P: TP15.1
Other:
- note added: "AUDIO CODEC"
- note added: "ON-BOARD MICROPHONE"
- note added: "SD CARD"
- note added: "USB"
